File: ACW_First/24_to_5.kicad_sch (KiCad schematic)
At the start: 20 parts, among them U2 MP1584EN

Commit message: okokok
Changed lines of the file:
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@@
-	)
-	(bus_entry
-		(at 247.65 66.04)
-		(size -2.54 2.54)
-		(stroke
-			(width 0)
-			(type default)
-		)
 	)
 	(bus_entry
