File: ACW_First/ACW_First.kicad_pcb (KiCad board)
At the start: 2 copper layers, 132 parts, among them J1 Screw_Terminal_01x02, J2 RELAYIOPIN, J3 3.8VDC, J4 5VDC, J5 12VDC, J6 STMRX/TX PINS, J7 Conn_01x02_Socket, J8 Conn_01x02_Pin, J9 24VDCPINS, K1 SRD-05VDC-SL-C, Q1 S8050, U1 MP1584EN, U2 MP1584EN, U3 MP1584EN, U4 PC817, U5 HT7133-1_C15060, U6 V9881D, U7 CT817C, U8 CT817C

Commit message: okok
Parts:
- added H1: MountingHole, MountingHole:MountingHole_3.2mm_M3, F.Cu at (602.4, 21.0)
- added H2: MountingHole, MountingHole:MountingHole_3.2mm_M3, F.Cu at (602.4, 79.7)
- added H3: MountingHole, MountingHole:MountingHole_3.2mm_M3, F.Cu at (533.3, 21.0)
- added H4: MountingHole, MountingHole:MountingHole_3.2mm_M3, F.Cu at (533.3, 79.7)
- added J10: Conn_01x04_Pin, Connector_PinHeader_2.54mm:PinHeader_1x04_P2.54mm_Vertical, F.Cu at (547.4, 20.0)
- added J11: 24VDC, Connector_PinSocket_2.54mm:PinSocket_1x02_P2.54mm_Vertical, B.Cu at (612.6, 128.2)
- added J12: Conn_01x02_Pin, Connector_PinSocket_2.54mm:PinSocket_1x02_P2.54mm_Vertical, F.Cu at (610.4, 169.5)
- added J13: Conn_01x04_Socket, Connector_PinSocket_2.54mm:PinSocket_1x04_P2.54mm_Vertical, B.Cu at (537.8, 119.3)
- added J14: Conn_01x02_Pin, Connector_PinSocket_2.54mm:PinSocket_1x02_P2.54mm_Vertical, F.Cu at (607.6, 172.3)
- C25, C26, C27, C28, C30, C31, C33, C34, C35, C36, C37, C38, C39, C40, D10, D11, D12, D13, D14, D6, D9, R20, R21, R22, R23, R26, R27, R28, R29, R30, R31, R32, R33, R34, R36, R37, R38, R39, R40, R41, R42, R43, TP1, TP2, U5, U6, U7, U8, Z1: moved to B.Cu
- J2: value RELAYIOPIN -> Conn_01x03_Pin; footprint Connector_PinSocket_2.54mm:PinSocket_1x02_P2.54mm_Vertical -> Connector_PinHeader_2.54mm:PinHeader_1x03_P2.54mm_Vertical; moved to B.Cu
- J6: value STMRX/TX PINS -> Screw_Terminal_01x02; footprint Connector_PinSocket_2.54mm:PinSocket_1x02_P2.54mm_Vertical -> TerminalBlock_MetzConnect:TerminalBlock_MetzConnect_Type101_RT01602HBWC_1x02_P5.08mm_Horizontal
- J7: value Conn_01x02_Socket -> Screw_Terminal_01x04; footprint Connector_PinSocket_2.54mm:PinSocket_1x02_P2.54mm_Vertical -> TerminalBlock_MetzConnect:TerminalBlock_MetzConnect_Type101_RT01604HBWC_1x04_P5.08mm_Horizontal
- J9: value 24VDCPINS -> Conn_01x03_Socket; footprint Connector_PinHeader_2.54mm:PinHeader_1x02_P2.54mm_Vertical -> Connector_PinSocket_2.54mm:PinSocket_1x03_P2.54mm_Vertical
- Q1: footprint Package_TO_SOT_THT:TO-92_Inline -> Package_TO_SOT_SMD:SOT-23; moved to B.Cu
- U4: footprint Package_DIP:DIP-4_W7.62mm -> Custom_Library:SOP254P975X460-4N; moved to B.Cu
- Y1: footprint Crystal:Crystal_C26-LF_D2.1mm_L6.5mm_Horizontal -> Crystal:Crystal_SMD_5032-4Pin_5.0x3.2mm; moved to B.Cu
- moved R36 555.4 mm to (571.8, 27.6), turned to 0 degrees
- moved U6 538.5 mm to (562.9, 42.9), turned to -90 degrees
- moved R34 529.8 mm to (565.2, 51.8), turned to 0 degrees
- moved C33 518.5 mm to (578.4, 39.6), turned to 180 degrees
- moved C29 517.8 mm to (557.2, 77.2), turned to 180 degrees
- moved C37 515.3 mm to (580.4, 31.4), turned to 180 degrees
- moved C31 512.9 mm to (574.7, 48.8), turned to 180 degrees
- moved C38 511.7 mm to (575.4, 27.0), turned to 180 degrees
- moved C39 509.8 mm to (572.6, 25.1), turned to 180 degrees
- moved R33 509.3 mm to (578.4, 41.9)
- moved C30 508.6 mm to (567.7, 32.0), turned to 90 degrees
- moved R35 507.9 mm to (546.0, 66.0)
- moved C40 506.1 mm to (569.7, 31.8), turned to -90 degrees
- moved R32 505.3 mm to (574.7, 41.9)
- moved R31 497.2 mm to (568.9, 53.9)
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Connections:
- C10 pad 1: /24VDC to 5VDC/5VDC -> /5VDC
- C15 pad 1: /24VDC to 5VDC/5VDC -> /5VDC
- C25 pad 1: Load -> /PZEM/CT2
- C25 pad 2: Net-(U6-IAP) -> Net-(U6-VDD5)
- C26 pad 1: Load -> /PZEM/CT2
- C26 pad 2: Net-(U6-IAN) -> Net-(U6-VDCIN)
- C27 pad 1: Net-(U6-IAP) -> Net-(U6-VDD5)
- C27 pad 2: Net-(U6-IAN) -> Net-(U6-VDCIN)
- C28 pad 1: Net-(U6-UP) -> Net-(U6-REF)
- C28 pad 2: Load -> /PZEM/CT2
- C29 pad 2: LO -> /PZEM/L
- C30 pad 1: Net-(U6-REF) -> Net-(U6-UP)
- C30 pad 2: Load -> /PZEM/CT2
- C33 pad 2: Net-(U6-VDCIN) -> Net-(U6-IAN)
- C35 pad 1: Net-(U6-DVCC) -> Net-(U6-VSS)
- C36 pad 1: Net-(U6-LDO33) -> Net-(U6-P1.3/RXD5/INT0/CFx/SP/PLLDIV/WAKEUP2)
- C38 pad 2: Net-(U6-DVCC) -> Net-(U6-VSS)
- C39 pad 2: Net-(U6-LDO33) -> Net-(U6-P1.3/RXD5/INT0/CFx/SP/PLLDIV/WAKEUP2)
- C40 pad 1: Net-(U6-RSTn) -> Net-(U6-MODE1)
- C40 pad 2: Load -> /PZEM/CT2
- D11 pad 1: Load -> /PZEM/CT2
- D8 pad 2: /24VDC to 5VDC/5VDC -> /5VDC
- D9 pad 1: 5 VDC -> /Relay/5V
- F1 pad 1: /24VDC to 12VDC/24VDC -> Net-(D2-A)
- F1 pad 2: Net-(D2-A) -> /24VDC
- F2 pad 1: /24VDC to 12VDC/24VDC -> /24VDC
- F3 pad 1: LO -> /Relay/NO
- F4 pad 1: /LIVE to 24V/L -> /Live
- J1 pad 1: Load -> /Neutral
- J1 pad 2: LI -> /Live
- J2 pad 1: unconnected-(J2-Pin_1-Pad1) -> GND
- J2 pad 2: /Relay/IO_PIN -> /5VDC
- J4 pad 2: /24VDC to 5VDC/5VDC -> /5VDC
- J6 pad 1: /PZEM/U8/2OUT -> /Relay/COM
- J6 pad 2: /PZEM/U7/4OUT -> /Relay/NO
- J7 pad 1: /LIVE to 24V/N -> /PZEM/CT1
- J7 pad 2: /LIVE to 24V/L -> /PZEM/CT2
- J8 pad 1: /24VDC to 12VDC/24VDC -> /LIVE to 24V/24VDC
- J9 pad 2: /24VDC to 12VDC/24VDC -> /Relay/5V
- K1 pad A1: 5 VDC -> /Relay/5V
- K1 pad COM: LI -> /Relay/COM
- K1 pad NO: Net-(C24-Pad1) -> Net-(K1-PadNO)
- L2 pad 2: /24VDC to 5VDC/5VDC -> /5VDC
- PS1 pad 2: /LIVE to 24V/N -> /Neutral
- PS1 pad 4: /24VDC to 12VDC/24VDC -> /LIVE to 24V/24VDC
- R13 pad 2: /24VDC to 5VDC/5VDC -> /5VDC
- R14 pad 1: /24VDC to 5VDC/5VDC -> /5VDC
- R2 pad 1: /24VDC to 12VDC/24VDC -> /24VDC
- R23 pad 2: 5 VDC -> /Relay/5V
- R24 pad 1: /Relay/N -> Net-(K1-PadNO)
- R25 pad 1: Load -> /PZEM/CT2
- R25 pad 2: Load -> /PZEM/CT1
- R26 pad 1: Load -> /PZEM/CT1
- R26 pad 2: Net-(U6-IAP) -> Net-(U6-VDD5)
- R27 pad 1: Load -> /PZEM/CT2
- R27 pad 2: Net-(U6-IAN) -> Net-(U6-VDCIN)
- R28 pad 1: Net-(U6-UP) -> Net-(U6-REF)
- R28 pad 2: LO -> /PZEM/L
- R29 pad 1: Load -> /PZEM/CT2
- R29 pad 2: Net-(U6-UP) -> Net-(U6-REF)
- R30 pad 1: LO -> /PZEM/L
- R32 pad 2: Net-(U6-VDCIN) -> Net-(U6-IAN)
- R33 pad 1: Net-(U6-VDCIN) -> Net-(U6-IAN)
- R34 pad 1: Net-(U6-MODE1) -> Net-(U6-RSTn)
- R36 pad 1: Net-(U6-RSTn) -> Net-(U6-MODE1)
- R36 pad 2: Net-(U6-LDO33) -> Net-(U6-P1.3/RXD5/INT0/CFx/SP/PLLDIV/WAKEUP2)
- R37 pad 2: Net-(U6-P2.4/RXD2) -> Net-(U6-P0.1/TDI)
- R39 pad 1: /24VDC to 5VDC/5VDC -> /PZEM/5VDC
- R40 pad 1: /24VDC to 5VDC/5VDC -> /PZEM/5VDC
- R41 pad 1: /24VDC to 5VDC/5VDC -> /PZEM/5VDC
- R42 pad 1: /24VDC to 5VDC/5VDC -> /PZEM/5VDC
- R43 pad 1: /24VDC to 12VDC/24VDC -> /LIVE to 24V/24VDC
- R9 pad 1: /24VDC to 12VDC/24VDC -> /24VDC
- RV2 pad 2: /Relay/N -> Net-(K1-PadNO)
- RV3 pad 2: /LIVE to 24V/N -> /Neutral
- TP2 pad 1: /24VDC to 12VDC/24VDC -> /LIVE to 24V/24VDC
- TP4 pad 1: /24VDC to 5VDC/5VDC -> /5VDC
- U4 pad 1: Net-(R20-Pad2) -> /Relay/5V
- U4 pad 2: GND -> Net-(R21-Pad1)
- U4 pad 3: Net-(R21-Pad1) -> GND
- U4 pad 4: 5 VDC -> Net-(R20-Pad2)
- U6 pad 11: unconnected-(U6-P1.3/RXD5/INT0/CFx/SP/PLLDIV/WAKEUP2-Pad11) -> Net-(U6-P1.3/RXD5/INT0/CFx/SP/PLLDIV/WAKEUP2)
- U6 pad 12: Load -> Net-(U6-VSS)
- U6 pad 13: Net-(U6-DVCC) -> /PZEM/CT2
- U6 pad 14: Net-(U6-LDO33) -> unconnected-(U6-LDO33-Pad14)
- U6 pad 16: Net-(U6-P2.5/TXD2) -> unconnected-(U6-P2.5/TXD2-Pad16)
- U6 pad 17: Net-(U6-P2.4/RXD2) -> unconnected-(U6-P2.4/RXD2-Pad17)
- U6 pad 18: Net-(U6-P2.0/T2/OSC) -> unconnected-(U6-P2.0/T2/OSC-Pad18)
- U6 pad 2: Net-(U6-IAP) -> Net-(U5-Vout)
- U6 pad 21: Net-(U6-CTO) -> Net-(U6-CTI)
- U6 pad 23: Net-(U5-Vout) -> Net-(U6-VDD5)
- U6 pad 5: Net-(U6-IBN) -> Net-(U6-IBP)
- U6 pad 7: unconnected-(U6-P0.0/TDO-Pad7) -> Net-(U6-P0.0/TDO)
- U6 pad 8: unconnected-(U6-P0.1/TDI-Pad8) -> Net-(U6-P0.1/TDI)
- U6 pad 9: unconnected-(U6-P0.2/WAKEUP3/TMS-Pad9) -> Net-(U6-P0.2/WAKEUP3/TMS)
- U7 pad 2: Net-(U6-P2.5/TXD2) -> Net-(U6-P0.2/WAKEUP3/TMS)
- U8 pad 3: Net-(U6-P2.0/T2/OSC) -> Net-(U6-P0.0/TDO)
- U8 pad 4: Net-(U6-P2.4/RXD2) -> Net-(U6-P0.1/TDI)
- Y1 pad 1: Net-(U6-CTI) -> Net-(U6-IBP)
- Y1 pad 2: Net-(U6-CTO) -> Net-(U6-IBN)
Routing:
- net (no net): track 0.00 -> 244.6 mm
- net /5VDC: track 0.00 -> 142.5 mm
- net /24VDC to 12VDC/24VDC: track 139.0 -> 0.00 mm, vias 2 -> 0
- net /PZEM/CT2: track 0.00 -> 116.9 mm, vias 0 -> 5
- net AGND: track 0.00 -> 72.4 mm, vias 0 -> 1
- net /24VDC to 12VDC/12VDC: track 55.5 -> 120.9 mm, vias 0 -> 1
- net /24VDC to 5VDC/5VDC: track 61.2 -> 0.00 mm, vias 2 -> 0
- net /Relay/5V: track 0.00 -> 57.0 mm, vias 0 -> 1
- net Net-(D10-K): track 0.00 -> 54.4 mm, vias 0 -> 1
- net GND: track 576.0 -> 628.0 mm, vias 15 -> 21
- net Net-(D2-K): track 65.5 -> 17.8 mm, vias 3 -> 0
- net /PZEM/L: track 0.00 -> 46.4 mm
- net /LIVE to 24V/N: track 43.9 -> 0.00 mm
- net /24VDC: track 0.00 -> 41.2 mm
- net Net-(U5-Vout): track 0.00 -> 41.2 mm, vias 0 -> 4
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Other:
- board outline added: 354 x 274.5 mm
- board text removed: "C1"

Commit message: okok
Parts:
- D6, D9, Q1, R21, R22, R23, TP1, TP2: moved to F.Cu
- F3: footprint Fuse:Fuseholder_Clip-5x20mm_Littelfuse_100_Inline_P20.50x4.60mm_D1.30mm_Horizontal -> Fuse:Fuseholder_Cylinder-5x20mm_Schurter_0031_8201_Horizontal_Open
- R25: moved to B.Cu
- moved R22 48.7 mm to (571.4, 79.6), turned to 90 degrees
- moved R21 46.7 mm to (568.2, 81.9), turned to 0 degrees
- moved Q1 41.4 mm to (572.3, 75.7), turned to 0 degrees
- moved U4 39.1 mm to (569.6, 78.0)
- moved D9 25.7 mm to (566.2, 68.6)
- moved R23 24.9 mm to (570.8, 66.5)
- moved D6 24.9 mm to (570.9, 70.3)
- moved R35 23.1 mm to (522.9, 66.0)
- moved R20 21.9 mm to (580.9, 60.4), turned to -90 degrees
- moved Y1 21.9 mm to (566.0, 49.9)
- moved TP2 20.5 mm to (589.4, 20.4), turned to 0 degrees
- moved H3 18.8 mm to (514.5, 21.6)
- moved C32 11.8 mm to (556.4, 77.6)
- moved C29 11.2 mm to (546.0, 76.0)
- moved R25 9.27 mm to (527.0, 65.8)
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Routing:
- net GND: track 628.0 -> 683.5 mm
- net /Relay/5V: track 57.0 -> 92.9 mm
- net Net-(C29-Pad1): track 37.4 -> 67.1 mm
- net AGND: track 72.4 -> 93.7 mm, vias 1 -> 3
- net Net-(D10-K): track 54.4 -> 75.5 mm
- net Net-(R20-Pad2): track 2.68 -> 22.9 mm
- net Net-(D10-A): track 26.4 -> 44.6 mm, vias 0 -> 1
- net /Relay/NO: track 21.1 -> 38.9 mm
- net /PZEM/CT2: track 116.9 -> 100.6 mm, vias 5 -> 4
- net /Relay/IO_PIN: track 30.2 -> 43.6 mm, vias 1 -> 0
- net /PZEM/CT1: track 26.7 -> 17.3 mm, vias 1 -> 0
- net Net-(R21-Pad1): track 3.79 -> 12.0 mm, vias 0 -> 1
- net Net-(U6-VDD5): track 36.7 -> 44.7 mm, vias 2 -> 0
- net /PZEM/L: track 46.4 -> 53.9 mm
- net /Relay/COM: track 36.2 -> 43.5 mm, vias 2 -> 0
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Other:
- board size 354 x 274.5 mm -> 119.2 x 164.5 mm

Commit message: add firstlevel & secondlevevl pcb
Parts:
- added H1: MountingHole, MountingHole:MountingHole_3.2mm_M3, F.Cu at (753.9, 79.6)
- added H2: MountingHole, MountingHole:MountingHole_3.2mm_M3, F.Cu at (753.9, 137.1)
- added H3: MountingHole, MountingHole:MountingHole_3.2mm_M3, F.Cu at (663.0, 79.6)
- added H4: MountingHole, MountingHole:MountingHole_3.2mm_M3, F.Cu at (668.1, 137.1)
- D11, D12, D13, R31: moved to F.Cu
- moved C18 185.0 mm to (698.4, 114.3)
- moved C19 185.0 mm to (698.4, 112.0)
- moved C2 184.0 mm to (752.6, 126.0), turned to -90 degrees
- moved TP3 183.9 mm to (748.1, 134.3), turned to 180 degrees
- moved R17 183.5 mm to (701.4, 116.6)
- moved R16 176.5 mm to (700.9, 106.8), turned to 0 degrees
- moved L3 176.0 mm to (694.3, 119.3)
- moved R7 175.6 mm to (753.7, 117.5), turned to 0 degrees
- moved U3 175.3 mm to (694.0, 106.2)
- moved L1 175.1 mm to (744.5, 126.3), turned to 0 degrees
- moved C17 174.5 mm to (699.4, 101.9), turned to 0 degrees
- moved C20 173.7 mm to (694.0, 102.2)
- moved C16 173.2 mm to (700.1, 98.6), turned to 0 degrees
- moved TP4 172.6 mm to (723.2, 136.9), turned to 180 degrees
- moved C4 171.5 mm to (750.3, 117.5), turned to 0 degrees
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Connections:
- J13 pad 2: unconnected-(J13-Pin_2-Pad2) -> /5VDC
- J13 pad 3: unconnected-(J13-Pin_3-Pad3) -> Net-(J13-Pin_3)
- J13 pad 4: unconnected-(J13-Pin_4-Pad4) -> Net-(J13-Pin_4)
- J14 pad 1: unconnected-(J14-Pin_1-Pad1) -> Net-(J13-Pin_3)
- J14 pad 2: unconnected-(J14-Pin_2-Pad2) -> Net-(J13-Pin_4)
Routing:
- net (no net): track 244.6 -> 0.00 mm
- net GND: track 683.5 -> 796.4 mm, vias 21 -> 17
- net Net-(U5-Vout): track 41.2 -> 115.2 mm, vias 4 -> 7
- net /5VDC: track 142.5 -> 202.8 mm, vias 0 -> 1
- net /24VDC to 12VDC/1.65V: track 66.2 -> 29.8 mm, vias 2 -> 0
- net Net-(D10-A): track 44.6 -> 11.2 mm, vias 1 -> 0
- net /24VDC to 12VDC/12VDC: track 120.9 -> 149.4 mm, vias 1 -> 2
- net Net-(D12-A): track 2.50 -> 30.3 mm, vias 0 -> 1
- net Net-(U6-P1.3/RXD5/INT0/CFx/SP/PLLDIV/WAKEUP2): track 32.2 -> 6.06 mm
- net /5VDC to 3.8VDC/3.8VDC: track 47.6 -> 73.6 mm, vias 2 -> 3
- net /PZEM/U8/1OUT: track 22.8 -> 46.2 mm, vias 2 -> 3
- net Net-(D10-K): track 75.5 -> 52.3 mm
- net Net-(U3-FB): track 28.7 -> 6.22 mm
- net Net-(D13-A): track 2.64 -> 24.2 mm, vias 0 -> 1
- net Net-(D5-K): track 26.5 -> 46.8 mm, vias 0 -> 2
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Other:
- board size 119.2 x 164.5 mm -> 246 x 122.6 mm

Commit message: okok
Parts:
- D3, D5, D7, R14, R15, R16, R18, R19: moved to B.Cu
- moved C23 59.2 mm to (709.4, 82.8), turned to -90 degrees
- moved TP5 53.4 mm to (708.6, 89.3), turned to 180 degrees
- moved C22 51.9 mm to (714.8, 86.2), turned to 0 degrees
- moved R15 42.3 mm to (715.8, 131.5), turned to -90 degrees
- moved D8 40.9 mm to (715.0, 129.7), turned to -90 degrees
- moved R14 40.0 mm to (713.5, 131.5), turned to 90 degrees
- moved C21 38.9 mm to (714.3, 95.5), turned to 0 degrees
- moved C16 29.1 mm to (715.6, 123.3)
- moved L3 26.5 mm to (716.0, 104.2)
- moved D7 25.2 mm to (710.9, 109.2), turned to 90 degrees
- moved C17 24.1 mm to (714.9, 120.4)
- moved C20 23.9 mm to (716.3, 110.6)
- moved U3 22.7 mm to (714.6, 115.7)
- moved R16 21.8 mm to (720.2, 117.1), turned to -90 degrees
- moved R18 21.6 mm to (710.9, 101.4), turned to 90 degrees
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Routing:
- net /5VDC to 3.8VDC/3.8VDC: track 73.6 -> 112.4 mm, vias 3 -> 2
- net Net-(U3-FB): track 6.22 -> 20.3 mm, vias 0 -> 1
- net /5VDC to 3.8VDC/COMP INPUT: track 20.5 -> 9.84 mm, vias 2 -> 0
- net GND: track 796.4 -> 806.3 mm, vias 17 -> 18
- net /PZEM/U7/4OUT: track 46.3 -> 38.7 mm, vias 0 -> 1
- net /24VDC: track 42.2 -> 34.7 mm
- net Net-(D3-K): track 40.9 -> 47.5 mm, vias 2 -> 3
- net Net-(D8-K): track 14.4 -> 20.2 mm
- net /24VDC to 5VDC/COMP INPUT: track 22.4 -> 17.6 mm
- net Net-(D5-K): track 46.8 -> 51.4 mm
- net Net-(D7-K): track 25.0 -> 21.1 mm, vias 2 -> 1
- net /24VDC to 5VDC/1.65V: track 36.2 -> 32.7 mm
- net /5VDC to 3.8VDC/1.65V: track 18.1 -> 21.5 mm, vias 0 -> 1
- net /5VDC: track 202.8 -> 205.1 mm, vias 1 -> 3
- net /24VDC to 12VDC/1.65V: track 29.8 -> 27.6 mm
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
Commit message: okokok
Routing:
- net Net-(D3-K): vias 3 -> 2
Changed lines of the file:
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@@
-	)
-	(via
-		(at 740.97 119.39)
-		(size 0.6)
-		(drill 0.3)
-		(layers "F.Cu" "B.Cu")
-		(net "Net-(D3-K)")
 	)
 	(via

Commit message: revisi
Parts:
- removed J7: Screw_Terminal_01x04, TerminalBlock_MetzConnect:TerminalBlock_MetzConnect_Type101_RT01604HBWC_1x04_P5.08mm_Horizontal
- removed U4: PC817, Custom_Library:SOP254P975X460-4N
- added BT101: Battery_Cell, Battery:BatteryHolder_Keystone_500, F.Cu at (600.2, 159.4)
- added C101: 100nf, Capacitor_SMD:C_0603_1608Metric, F.Cu at (614.5, 187.5)
- added C102: 2.2uf, Capacitor_SMD:C_0603_1608Metric, F.Cu at (595.8, 188.4)
- added C103: 100nf, Capacitor_SMD:C_0603_1608Metric, B.Cu at (563.2, 162.7)
- added C104: 100nf, Capacitor_SMD:C_0603_1608Metric, B.Cu at (597.7, 188.3)
- added C105: 100nf, Capacitor_SMD:C_0603_1608Metric, B.Cu at (609.0, 188.3)
- added C106: 22pf, Capacitor_SMD:C_0603_1608Metric, F.Cu at (607.9, 169.0)
- added C107: 22pf, Capacitor_SMD:C_0603_1608Metric, F.Cu at (598.8, 169.0)
- added C108: 100nf, Capacitor_SMD:C_0603_1608Metric, F.Cu at (609.0, 177.0)
- added C109: 100nf, Capacitor_SMD:C_0603_1608Metric, B.Cu at (553.8, 162.8)
- added C110: 100nf, Capacitor_SMD:C_0603_1608Metric, B.Cu at (601.7, 173.6)
- added C111: 100nf, Capacitor_SMD:C_0603_1608Metric, B.Cu at (579.1, 162.1)
- added C112: 1uf, Capacitor_SMD:C_0603_1608Metric, B.Cu at (626.2, 158.3)
- added C113: 1uf, Capacitor_SMD:C_0603_1608Metric, B.Cu at (627.2, 167.9)
- added C114: 1uf, Capacitor_SMD:C_0603_1608Metric, B.Cu at (607.8, 156.7)
- added C115: 1uf, Capacitor_SMD:C_0603_1608Metric, B.Cu at (594.0, 211.8)
- added C116: 1uf, Capacitor_SMD:C_0603_1608Metric, B.Cu at (591.8, 211.8)
- added D101: LED, LED_SMD:LED_0603_1608Metric, F.Cu at (613.9, 169.3)
- added D102: LED, LED_SMD:LED_0603_1608Metric, F.Cu at (616.4, 169.3)
- added H1: MountingHole, MountingHole:MountingHole_3.2mm_M3, F.Cu at (630.7, 155.0)
- added H2: MountingHole, MountingHole:MountingHole_3.2mm_M3, F.Cu at (630.7, 212.5)
- added H3: MountingHole, MountingHole:MountingHole_3.2mm_M3, F.Cu at (539.8, 155.0)
- added H4: MountingHole, MountingHole:MountingHole_3.2mm_M3, F.Cu at (544.8, 212.5)
- added J101: Conn_01x02_Male, TerminalBlock_MetzConnect:TerminalBlock_MetzConnect_Type101_RT01602HBWC_1x02_P5.08mm_Horizontal, F.Cu at (583.0, 211.8)
- added J102: Conn_STLink, Connector_JST:JST_XH_S4B-XH-A_1x04_P2.50mm_Horizontal, F.Cu at (630.8, 181.0)
- added J103: Conn_01x04_Female, Connector_JST:JST_XH_S4B-XH-A_1x04_P2.50mm_Horizontal, F.Cu at (631.0, 195.3)
- added J104: Conn_01x02_Pin, Connector_PinHeader_2.54mm:PinHeader_1x02_P2.54mm_Vertical, F.Cu at (590.7, 153.3)
- added J105: Conn_01x02_Pin, Connector_PinHeader_2.54mm:PinHeader_1x02_P2.54mm_Vertical, F.Cu at (586.1, 153.2)
- added J106: Conn_01x02_Pin, Connector_PinHeader_2.54mm:PinHeader_1x02_P2.54mm_Vertical, F.Cu at (533.7, 182.8)
- added J107: Conn_01x02_Pin, Connector_PinHeader_2.54mm:PinHeader_1x02_P2.54mm_Vertical, F.Cu at (533.7, 162.1)
- added J108: Conn_01x02_Pin, Connector_PinHeader_2.54mm:PinHeader_1x02_P2.54mm_Vertical, F.Cu at (533.7, 201.9)
- added PS101: RKZ-1212S_P, Custom_Library:CONV_RKZ-1212S_P, F.Cu at (581.0, 190.6)
- added R101: 10k, Resistor_SMD:R_0603_1608Metric, F.Cu at (614.6, 182.7)
- added R102: 10k, Resistor_SMD:R_0603_1608Metric, F.Cu at (614.6, 177.1)
- added R103: 100, Resistor_SMD:R_0603_1608Metric, B.Cu at (621.4, 183.0)
- added R104: 100, Resistor_SMD:R_0603_1608Metric, B.Cu at (621.4, 179.9)
- added R105: 100, Resistor_SMD:R_0603_1608Metric, F.Cu at (624.0, 208.9)
- added R106: 100, Resistor_SMD:R_0603_1608Metric, F.Cu at (616.3, 208.9)
- added R107: 220, Resistor_SMD:R_0603_1608Metric, F.Cu at (613.9, 173.1)
- added R108: 220, Resistor_SMD:R_0603_1608Metric, F.Cu at (616.4, 173.1)
- added R109: 100, Resistor_SMD:R_0603_1608Metric, F.Cu at (611.2, 209.2)
- added R110: 100, Resistor_SMD:R_0603_1608Metric, F.Cu at (613.7, 209.1)
- added R111: 100, Resistor_SMD:R_0603_1608Metric, F.Cu at (583.6, 157.2)
- added R112: 100, Resistor_SMD:R_0603_1608Metric, F.Cu at (586.1, 157.2)
- added R113: 100, Resistor_SMD:R_0603_1608Metric, B.Cu at (587.8, 178.2)
- added R114: 100, Resistor_SMD:R_0603_1608Metric, B.Cu at (623.7, 191.5)
- added R115: 100, Resistor_SMD:R_0603_1608Metric, B.Cu at (623.7, 193.4)
- added R116: 10k, Resistor_SMD:R_0603_1608Metric, B.Cu at (579.8, 168.4)
- added R117: LDR07, OptoDevice:R_LDR_5.1x4.3mm_P3.4mm_Vertical, F.Cu at (576.6, 153.9)
- added R118: 220, Resistor_SMD:R_0603_1608Metric, B.Cu at (580.3, 158.4)
- added R119: 4.7k, Resistor_SMD:R_0603_1608Metric, B.Cu at (632.2, 169.2)
- added R120: 4.7k, Resistor_SMD:R_0603_1608Metric, B.Cu at (629.1, 170.1)
- added R121: 4.7k, Resistor_SMD:R_0603_1608Metric, B.Cu at (632.2, 167.3)
- added R122: 4.7k, Resistor_SMD:R_0603_1608Metric, B.Cu at (624.4, 167.9)
- added R123: 4.7k, Resistor_SMD:R_0603_1608Metric, B.Cu at (620.9, 167.9)
- added R124: 220, Resistor_SMD:R_0603_1608Metric, B.Cu at (591.4, 191.0)
- added R125: 10k, Resistor_SMD:R_0603_1608Metric, B.Cu at (586.9, 198.1)
- added R126: 4.7k, Resistor_SMD:R_0603_1608Metric, B.Cu at (598.5, 207.6)
- added R127: 10k, Resistor_SMD:R_0603_1608Metric, B.Cu at (600.2, 207.6)
- added R128: 10k, Resistor_SMD:R_0603_1608Metric, B.Cu at (602.0, 207.7)
- added R129: 4.7k, Resistor_SMD:R_0603_1608Metric, B.Cu at (576.1, 203.2)
- added SW101: SW_Push, Library:Pushbutton_3x4x2mm_2P_SMD, F.Cu at (616.3, 182.5)
- added SW102: SW_Push, Library:Pushbutton_3x4x2mm_2P_SMD, F.Cu at (616.3, 177.2)
- added U101: A7600_Pinout, Connector_PinHeader_2.54mm:PinHeader_1x07_P2.54mm_Vertical, F.Cu at (608.7, 213.9)
- added U102: STM32F401CCUx, Package_DFN_QFN:QFN-48-1EP_7x7mm_P0.5mm_EP5.6x5.6mm, F.Cu at (603.8, 182.0)
- added U103: AMS1117-3.3, Package_TO_SOT_SMD:SOT-223, B.Cu at (558.5, 165.1)
- added U104: MCP6002-I_SN, Custom_Library:SOIC127P600X175-8N, B.Cu at (584.5, 164.0)
- added U105: DS3231M, Package_SO:SOIC-16W_7.5x10.3mm_P1.27mm, B.Cu at (618.2, 157.8)
- added U106: AT24C512-SSHM, Custom_Library:SOIC127P600X175-8N, B.Cu at (628.8, 163.1)
- added U107: PC817, Custom_Library:SOP254P975X460-4N, B.Cu at (592.7, 200.7)
- added U108: LM358PSR, Custom_Library:SOIC127P780X200-8N, B.Cu at (582.8, 205.9)
- added Y101: 8Mhz, Crystal:Crystal_SMD_5032-4Pin_5.0x3.2mm, F.Cu at (603.6, 168.8)
- D14, R43: moved to F.Cu
- U1: value MP1584EN -> PC817; footprint Custom_Footprints:SOIC127P600X170-9N -> Custom_Library:SOP254P975X460-4N; moved to B.Cu
- moved U1 177.9 mm to (570.0, 73.2)
- moved R21 15.4 mm to (573.5, 67.5), turned to 180 degrees
- moved R22 12.2 mm to (570.2, 67.5), turned to 0 degrees
- moved Q1 11.2 mm to (573.7, 64.5)
- moved R23 9.59 mm to (574.4, 75.4), turned to 0 degrees
- moved H4 8.62 mm to (516.5, 79.5)
- moved D9 6.88 mm to (572.2, 72.0), turned to 180 degrees
- moved C32 6.68 mm to (556.8, 71.2)
- moved D6 5.22 mm to (570.3, 75.5), turned to 0 degrees
- moved D11 4.06 mm to (555.3, 65.0)
- moved R31 4.01 mm to (558.7, 65.0)
- moved H3 3.53 mm to (516.5, 22.0)
- moved R20 0.06 mm to (581.7, 61.2)
Connections:
- C25 pad 1: /PZEM/CT2 -> /Neutral
- C26 pad 1: /PZEM/CT2 -> /Neutral
- C28 pad 2: /PZEM/CT2 -> /Neutral
- C29 pad 2: /PZEM/L -> /Live_OutPZEM
- C30 pad 2: /PZEM/CT2 -> /Neutral
- C40 pad 2: /PZEM/CT2 -> /Neutral
- D11 pad 1: /PZEM/CT2 -> /Neutral
- J6 pad 1: /Relay/COM -> /Relay/NO
- J6 pad 2: /Relay/NO -> /Neutral
- J8 pad 1: /LIVE to 24V/24VDC -> /24VDC
- K1 pad COM: /Relay/COM -> /Live_OutPZEM
- K1 pad NO: Net-(K1-PadNO) -> Net-(C24-Pad1)
- PS1 pad 4: /LIVE to 24V/24VDC -> /24VDC
- R24 pad 1: Net-(K1-PadNO) -> /Neutral
- R25 pad 1: /PZEM/CT2 -> /Neutral
- R25 pad 2: /PZEM/CT1 -> /Live
- R26 pad 1: /PZEM/CT1 -> /Live
- R27 pad 1: /PZEM/CT2 -> /Neutral
- R28 pad 2: /PZEM/L -> /Live_OutPZEM
- R29 pad 1: /PZEM/CT2 -> /Neutral
- R30 pad 1: /PZEM/L -> /Live_OutPZEM
- R43 pad 1: /LIVE to 24V/24VDC -> /24VDC
- RV2 pad 2: Net-(K1-PadNO) -> /Neutral
- TP2 pad 1: /LIVE to 24V/24VDC -> /24VDC
- U1 pad 1: Net-(D3-K) -> Net-(R20-Pad2)
- U1 pad 2: /24VDC to 12VDC/1.65V -> GND
- U1 pad 3: /24VDC to 12VDC/COMP INPUT -> Net-(R21-Pad1)
- U1 pad 4: Net-(U1-FB) -> /Relay/5V
- U6 pad 13: /PZEM/CT2 -> /Neutral
Routing:
- net GND: track 806.3 -> 1331.2 mm, vias 18 -> 35
- net /Neutral: track 25.3 -> 261.3 mm, vias 0 -> 4
- net +3.3V: track 0.00 -> 235.7 mm, vias 0 -> 11
- net +5V: track 0.00 -> 111.9 mm, vias 0 -> 2
- net /Live_OutPZEM: track 0.00 -> 101.2 mm, vias 0 -> 2
- net /3.8V: track 0.00 -> 91.4 mm
- net /PZEM/CT2: track 90.8 -> 0.00 mm, vias 2 -> 0
- net /PZEM/L: track 51.4 -> 0.00 mm, vias 2 -> 0
- net +12V: track 0.00 -> 49.5 mm
- net IGND: track 0.00 -> 43.2 mm, vias 0 -> 3
- net /SCL_RTC: track 0.00 -> 40.5 mm, vias 0 -> 4
- net /SWDIO: track 0.00 -> 40.3 mm, vias 0 -> 3
- net /Relay/COM: track 39.8 -> 0.00 mm
- net /SDA_RTC: track 0.00 -> 39.2 mm, vias 0 -> 4
- net Net-(U102-PB14): track 0.00 -> 38.7 mm, vias 0 -> 2
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Other:
- board size 246 x 122.6 mm -> 246 x 198 mm
