File: ACW_First/ACW_First.kicad_pcb (KiCad board)
At the start: 2 copper layers, 246 x 198 mm, 215 parts, among them J1 Screw_Terminal_01x02, J10 Conn_01x04_Pin, J101 Conn_01x02_Male, J102 Conn_STLink, J103 Conn_01x04_Female, J104 Conn_01x02_Pin, J105 Conn_01x02_Pin, J106 Conn_01x02_Pin, J107 Conn_01x02_Pin, J108 Conn_01x02_Pin, J11 24VDC, J12 Conn_01x02_Pin, J13 Conn_01x04_Socket, J14 Conn_01x02_Pin, J2 Conn_01x03_Pin, J3 3.8VDC, J4 5VDC, J5 12VDC, J6 Screw_Terminal_01x02, J8 Conn_01x02_Pin, J9 Conn_01x03_Socket, K1 SRD-05VDC-SL-C, Q1 S8050, SW101 SW_Push, SW102 SW_Push, U1 PC817, U101 A7600_Pinout, U102 STM32F401CCUx, U103 AMS1117-3.3, U104 MCP6002-I_SN, U105 DS3231M, U106 AT24C512-SSHM, U107 PC817, U108 LM358PSR, U2 MP1584EN, U3 MP1584EN, U5 HT7133-1_C15060, U6 V9881D, U7 CT817C, U8 CT817C, Y101 8Mhz

Commit message: okok
Parts:
- removed C10: 470µF, Capacitor_SMD:CP_Elec_8x10.5
- removed C11: 10µF, Capacitor_SMD:CP_Elec_5x5.4
- removed C12, C14, C15, C17, C20, C23, C3, C7: 100nF, Capacitor_SMD:C_0603_1608Metric
- removed C13: 10µF, Capacitor_SMD:CP_Elec_6.3x5.4
- removed C16: 10µF, Capacitor_Tantalum_SMD:CP_EIA-3528-21_Kemet-B
- removed C18, C4, C8: 220pF, Capacitor_SMD:C_0603_1608Metric
- removed C19, C5, C9: NS, Capacitor_SMD:C_0603_1608Metric
- removed C2: 22µF, Capacitor_SMD:CP_Elec_6.3x5.4
- removed C21, C22: 330µF, Capacitor_SMD:CP_Elec_8x10.5
- removed C6: 220µF, Capacitor_SMD:CP_Elec_8x10.5
- removed D3, D4, D5, D7, D8: SS34, Diode_SMD:D_SMA
- removed F2: Resettable Fuse/2A, Fuse:Fuse_1812_4532Metric_Pad1.30x3.40mm_HandSolder
- removed the H1 at (630.7, 155.0)
- removed the H1 at (753.9, 79.6)
- removed the H2 at (630.7, 212.5)
- removed the H2 at (753.9, 137.1)
- removed the H3 at (663.0, 79.6)
- removed the H3 at (539.8, 155.0)
- removed the H4 at (668.1, 137.1)
- removed the H4 at (544.8, 212.5)
- removed J104, J105, J106, J107, J108: Conn_01x02_Pin, Connector_PinHeader_2.54mm:PinHeader_1x02_P2.54mm_Vertical
- removed J12, J14: Conn_01x02_Pin, Connector_PinSocket_2.54mm:PinSocket_1x02_P2.54mm_Vertical
- removed J3: 3.8VDC, Connector_PinHeader_2.54mm:PinHeader_1x02_P2.54mm_Vertical
- removed J4: 5VDC, Connector_PinHeader_2.54mm:PinHeader_1x02_P2.54mm_Vertical
- removed J5: 12VDC, Connector_PinHeader_2.54mm:PinHeader_1x02_P2.54mm_Vertical
- removed L1: 22µH, Inductor_SMD:L_7.3x7.3_H4.5
- removed L2: 10µH, Inductor_SMD:L_Bourns-SRR1005
- removed L3: 10µH, Inductor_SMD:L_7.3x7.3_H4.5
- removed R10: 11KΩ, Resistor_SMD:R_0603_1608Metric
- removed R11, R5: 40.2KΩ, Resistor_SMD:R_0603_1608Metric
- removed R12, R17: 68.1KΩ, Resistor_SMD:R_0603_1608Metric
- removed R13: 210KΩ, Resistor_SMD:R_0603_1608Metric
- removed R14: 20KΩ, Resistor_SMD:R_0603_1608Metric
- removed R15: 10KΩ, Resistor_SMD:R_0603_1608Metric
- removed R16, R4, R8: 200KΩ, Resistor_SMD:R_0603_1608Metric
- removed R18: 150KΩ, Capacitor_SMD:C_0603_1608Metric
- removed R19: 40.2KΩ, Capacitor_SMD:C_0603_1608Metric
- removed R2: 149KΩ/1%, Resistor_SMD:R_0603_1608Metric
- removed R3: 11KΩ/1%, Resistor_SMD:R_0603_1608Metric
- removed R6: 562KΩ, Resistor_SMD:R_0603_1608Metric
- removed R7: 68.1KΩ/1%, Resistor_SMD:R_0603_1608Metric
- removed R9: 149KΩ, Resistor_SMD:R_0603_1608Metric
- removed TP3: 12VTP, TestPoint:TestPoint_Pad_D1.5mm
- removed TP4: 5VTP, TestPoint:TestPoint_Pad_D1.5mm
- removed TP5: 3.8VTP, TestPoint:TestPoint_Pad_D1.5mm
- removed U2, U3: MP1584EN, Custom_Footprints:SOIC127P600X170-9N
- added C42: 10µF, Capacitor_SMD:CP_Elec_5x5.4, F.Cu at (752.2, 108.0)
- added C43: 100nF, Capacitor_SMD:C_0603_1608Metric, F.Cu at (752.9, 112.2)
- added C44: 220pF, Capacitor_SMD:C_0603_1608Metric, F.Cu at (750.0, 119.2)
- added C45: 100nF, Capacitor_SMD:C_0603_1608Metric, F.Cu at (742.6, 107.8)
- added C46: NS, Capacitor_SMD:C_0603_1608Metric, F.Cu at (750.0, 117.1)
- added C47: 22µF, Capacitor_SMD:CP_Elec_6.3x5.4, F.Cu at (752.3, 127.7)
- added C48: 220µF, Capacitor_SMD:CP_Elec_8x10.5, F.Cu at (731.6, 96.9)
- added C49: 10µF, Capacitor_SMD:CP_Elec_6.3x5.4, F.Cu at (733.1, 105.6)
- added C50: 100nF, Capacitor_SMD:C_0603_1608Metric, F.Cu at (732.5, 110.4)
- added C51: 220pF, Capacitor_SMD:C_0603_1608Metric, F.Cu at (732.9, 116.7)
- added C52: 100nF, Capacitor_SMD:C_0603_1608Metric, F.Cu at (724.0, 108.6)
- added C53: NS, Capacitor_SMD:C_0603_1608Metric, F.Cu at (732.9, 114.7)
- added C54: 470µF, Capacitor_SMD:CP_Elec_8x10.5, F.Cu at (733.7, 127.2)
- added C55: 100nF, Capacitor_SMD:C_0603_1608Metric, F.Cu at (730.4, 133.9)
- added C56: 10µF, Capacitor_Tantalum_SMD:CP_EIA-3528-21_Kemet-B, F.Cu at (715.3, 125.1)
- added C57: 100nF, Capacitor_SMD:C_0603_1608Metric, F.Cu at (714.6, 122.1)
- added C58: 220pF, Capacitor_SMD:C_0603_1608Metric, F.Cu at (708.8, 121.8)
- added C59: 100nF, Capacitor_SMD:C_0603_1608Metric, F.Cu at (716.0, 112.3)
- added C60: NS, Capacitor_SMD:C_0603_1608Metric, F.Cu at (710.8, 125.0)
- added C61: 330µF, Capacitor_SMD:CP_Elec_8x10.5, F.Cu at (714.0, 97.2)
- added C62: 330µF, Capacitor_SMD:CP_Elec_8x10.5, F.Cu at (714.5, 87.9)
- added C63: 100nF, Capacitor_SMD:C_0603_1608Metric, F.Cu at (709.1, 84.5)
- added D16: SS34, Diode_SMD:D_SMA, B.Cu at (737.7, 127.6)
- added D17: SS34, Diode_SMD:D_SMA, F.Cu at (725.0, 103.7)
- added D18: SS34, Diode_SMD:D_SMA, B.Cu at (719.8, 128.3)
- added D19: SS34, Diode_SMD:D_SMA, F.Cu at (714.8, 131.3)
- added D20: SS34, Diode_SMD:D_SMA, B.Cu at (710.7, 110.8)
- added F6: Resettable Fuse/2A, Fuse:Fuse_1812_4532Metric_Pad1.30x3.40mm_HandSolder, F.Cu at (734.5, 88.6)
- added H101: MountingHole, MountingHole:MountingHole_3.2mm_M3, F.Cu at (725.8, 208.5)
- added H102: MountingHole, MountingHole:MountingHole_3.2mm_M3, F.Cu at (717.0, 250.7)
- added H103: MountingHole, MountingHole:MountingHole_3.2mm_M3, F.Cu at (518.7, 235.8)
- added H104: MountingHole, MountingHole:MountingHole_3.2mm_M3, F.Cu at (513.7, 178.3)
- added H5: MountingHole, MountingHole:MountingHole_3.2mm_M3, F.Cu at (753.9, 79.6)
- added H6: MountingHole, MountingHole:MountingHole_3.2mm_M3, F.Cu at (753.9, 137.1)
- added H7: MountingHole, MountingHole:MountingHole_3.2mm_M3, F.Cu at (658.2, 79.6)
- added H8: MountingHole, MountingHole:MountingHole_3.2mm_M3, F.Cu at (658.2, 137.1)
- added L4: 22µH, Inductor_SMD:L_7.3x7.3_H4.5, F.Cu at (744.1, 128.0)
- added L5: 10µH, Inductor_SMD:L_Bourns-SRR1005, F.Cu at (723.2, 128.0)
- added L6: 10µH, Inductor_SMD:L_7.3x7.3_H4.5, F.Cu at (715.8, 105.9)
- added R44: 149KΩ/1%, Resistor_SMD:R_0603_1608Metric, F.Cu at (743.4, 91.0)
- added R45: 11KΩ/1%, Resistor_SMD:R_0603_1608Metric, F.Cu at (740.5, 91.1)
- added R46: 200KΩ, Resistor_SMD:R_0603_1608Metric, F.Cu at (752.9, 114.0)
- added R47: 68.1KΩ/1%, Resistor_SMD:R_0603_1608Metric, F.Cu at (753.4, 119.2)
- added R48: 40.2KΩ, Resistor_SMD:R_0603_1608Metric, F.Cu at (741.2, 118.9)
- added R49: 562KΩ, Resistor_SMD:R_0603_1608Metric, F.Cu at (744.0, 118.9)
- added R50: 149KΩ, Resistor_SMD:R_0603_1608Metric, F.Cu at (728.6, 88.9)
- added R51: 11KΩ, Resistor_SMD:R_0603_1608Metric, F.Cu at (725.5, 89.0)
- added R52: 200KΩ, Resistor_SMD:R_0603_1608Metric, F.Cu at (732.5, 112.6)
- added R53: 68.1KΩ, Resistor_SMD:R_0603_1608Metric, F.Cu at (736.5, 116.7)
- added R54: 40.2KΩ, Resistor_SMD:R_0603_1608Metric, F.Cu at (725.0, 118.9)
- added R55: 210KΩ, Resistor_SMD:R_0603_1608Metric, F.Cu at (727.8, 118.9)
- added R56: 20KΩ, Resistor_SMD:R_0603_1608Metric, B.Cu at (713.2, 133.3)
- added R57: 10KΩ, Resistor_SMD:R_0603_1608Metric, B.Cu at (715.4, 133.3)
- added R58: 200KΩ, Resistor_SMD:R_0603_1608Metric, B.Cu at (719.9, 118.8)
- added R59: 68.1KΩ, Resistor_SMD:R_0603_1608Metric, F.Cu at (708.8, 125.0)
- added R60: 40.2KΩ, Capacitor_SMD:C_0603_1608Metric, B.Cu at (708.7, 103.1)
- added R61: 150KΩ, Capacitor_SMD:C_0603_1608Metric, B.Cu at (710.6, 103.1)
- added TP6: 12VTP, TestPoint:TestPoint_Pad_D1.5mm, F.Cu at (747.6, 136.0)
- added TP7: 5VTP, TestPoint:TestPoint_Pad_D1.5mm, F.Cu at (728.3, 137.0)
- added TP8: 3.8VTP, TestPoint:TestPoint_Pad_D1.5mm, F.Cu at (708.5, 90.9)
- added U10: MP1584EN, Custom_Footprints:SOIC127P600X170-9N, F.Cu at (725.7, 112.6)
- added U11: MP1584EN, Custom_Footprints:SOIC127P600X170-9N, F.Cu at (714.4, 117.4)
- added U9: MP1584EN, Custom_Footprints:SOIC127P600X170-9N, F.Cu at (743.7, 112.2)
- J102, J103: footprint Connector_JST:JST_XH_S4B-XH-A_1x04_P2.50mm_Horizontal -> Connector_JST:JST_XH_B4B-XH-A_1x04_P2.50mm_Vertical
- U103: moved to F.Cu
- moved C109 155.1 mm to (706.3, 134.9), turned to 0 degrees
- moved U103 149.3 mm to (704.2, 132.7)
- moved C103 145.4 mm to (706.3, 136.5), turned to 0 degrees
- moved R113 121.1 mm to (670.7, 89.9), turned to 90 degrees
- moved U104 118.1 mm to (675.6, 88.8)
- moved C115 115.1 mm to (674.1, 129.1)
- moved C116 115.1 mm to (671.9, 129.1)
- moved R126 114.1 mm to (677.8, 125.7), turned to 0 degrees
- moved J101 113.2 mm to (666.9, 135.7)
- moved U108 113.2 mm to (664.5, 127.6)
- moved U107 112.6 mm to (672.7, 121.5)
- moved R129 112.4 mm to (658.5, 126.8)
- moved R127 111.5 mm to (677.8, 127.5), turned to 180 degrees
- moved R128 109.0 mm to (677.8, 129.3), turned to 180 degrees
- moved R125 108.6 mm to (664.2, 121.8)
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- renumbered C1 to C41, D2 to D15, F1 to F5
Connections:
- net /A7600_PWRKY renamed /Controller/A7600_PWRKY
- net /A7600_RXD renamed /Controller/A7600_RXD
- net /A7600_SLEEP renamed /Controller/A7600_SLEEP
- net /A7600_TXD renamed /Controller/A7600_TXD
- net /BOOT0 renamed /Controller/BOOT0
- net /DEBUG_RXD renamed /Controller/DEBUG_RXD
- net /DEBUG_TXD renamed /Controller/DEBUG_TXD
- net /Dimm_Circuit/Dim_Output+ renamed /Controller/Dimm_Circuit/Dim_Output+
- net /Dimm_Circuit/Dim_Output- renamed /Controller/Dimm_Circuit/Dim_Output-
- net /LDR_Output renamed /Controller/LDR_Output
- net /NRST renamed /Controller/NRST
- net /PC13 renamed /Controller/PC13
- net /PH0 renamed /Controller/PH0
- net /PH1 renamed /Controller/PH1
- net /PWM_Input renamed /Controller/PWM_Input
- net /SCL_RTC renamed /Controller/SCL_RTC
- net /SDA_RTC renamed /Controller/SDA_RTC
- net /SWCLK renamed /Controller/SWCLK
- net /SWDIO renamed /Controller/SWDIO
- net GND renamed -12VDC
- C103 pad 1: +5V -> 5VDC
- J103 pad 4: +5V -> 5VDC
- J13 pad 2: /5VDC -> 5VDC
- J13 pad 3: Net-(J13-Pin_3) -> /PZEM_TXD
- J13 pad 4: Net-(J13-Pin_4) -> /PZEM_RXD
- J2 pad 2: /5VDC -> 5VDC
- J2 pad 3: Net-(J12-Pin_1) -> /RELAY_DATA
- PS101 pad 1: +12V -> 12VDC
- U101 pad 5: /3.8V -> 3.8VDC
- U103 pad 3: +5V -> 5VDC
Routing:
- net -12VDC: track 1331.2 -> 1069.6 mm
- net 5VDC: track 0.00 -> 222.7 mm, vias 0 -> 3
- net /5VDC: track 205.1 -> 0.00 mm, vias 3 -> 0
- net 12VDC: track 0.00 -> 151.6 mm
- net /24VDC to 12VDC/12VDC: track 149.4 -> 0.00 mm, vias 2 -> 0
- net /5VDC to 3.8VDC/3.8VDC: track 112.4 -> 0.00 mm, vias 2 -> 0
- net +5V: track 111.9 -> 0.00 mm, vias 2 -> 0
- net /3.8V: track 91.4 -> 0.00 mm
- net 3.8VDC: track 0.00 -> 89.7 mm, vias 0 -> 2
- net /RELAY_DATA: track 36.2 -> 103.3 mm
- net Net-(D5-K): track 51.4 -> 0.00 mm, vias 2 -> 0
- net +12V: track 49.5 -> 0.00 mm
- net Net-(D3-K): track 47.5 -> 0.00 mm, vias 2 -> 0
- net /PZEM_RXD: track 3.10 -> 46.4 mm, vias 0 -> 2
- net /PZEM_TXD: track 3.11 -> 41.4 mm
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Other:
- board size 246 x 198 mm -> 246 x 122.6 mm

Commit message: okok
Parts:
- removed D6: LED_Red, LED_SMD:LED_0805_2012Metric
- removed R23: 1KΩ, Resistor_SMD:R_0603_1608Metric
- Q1, R21, R22: moved to B.Cu
- R114, R115, R34: moved to F.Cu
- U1: footprint Custom_Library:SOP254P975X460-4N -> Custom_Footprints:SOP-4_L6.4-W4.6-P2.54-LS10.2-TL
- moved H101 246.7 mm to (566.1, 20.5)
- moved H102 234.4 mm to (567.4, 70.2)
- moved H103 196.4 mm to (499.5, 40.3)
- moved H104 128.7 mm to (496.3, 50.7)
- moved R111 74.8 mm to (737.5, 96.9)
- moved R112 70.3 mm to (734.9, 96.9)
- moved C107 53.2 mm to (725.7, 102.7), turned to 180 degrees
- moved Y101 45.3 mm to (720.1, 110.2)
- moved C106 44.7 mm to (725.7, 104.6), turned to 180 degrees
- moved R102 41.1 mm to (727.1, 115.8)
- moved R120 41.1 mm to (738.7, 108.7)
- moved C103 41.1 mm to (744.6, 151.2)
- moved C104 41.1 mm to (714.6, 128.5)
- moved C105 41.1 mm to (721.5, 127.0)
- moved C109 41.1 mm to (744.7, 149.6)
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Connections:
- BT101 pad 2: -12VDC -> GND
- C101 pad 1: -12VDC -> GND
- C102 pad 1: -12VDC -> GND
- C103 pad 2: -12VDC -> GND
- C104 pad 1: -12VDC -> GND
- C105 pad 1: -12VDC -> GND
- C106 pad 1: -12VDC -> GND
- C107 pad 1: -12VDC -> GND
- C108 pad 1: -12VDC -> GND
- C109 pad 2: -12VDC -> GND
- C110 pad 1: -12VDC -> GND
- C111 pad 2: -12VDC -> GND
- C112 pad 2: -12VDC -> GND
- C113 pad 2: -12VDC -> GND
- C114 pad 2: -12VDC -> GND
- C41 pad 2: -12VDC -> GND
- C42 pad 2: -12VDC -> GND
- C43 pad 2: -12VDC -> GND
- C46 pad 2: -12VDC -> GND
- C47 pad 2: -12VDC -> GND
- C48 pad 2: -12VDC -> GND
- C49 pad 2: -12VDC -> GND
- C50 pad 2: -12VDC -> GND
- C53 pad 2: -12VDC -> GND
- C54 pad 2: -12VDC -> GND
- C55 pad 2: -12VDC -> GND
- C56 pad 2: -12VDC -> GND
- C57 pad 2: -12VDC -> GND
- C60 pad 2: -12VDC -> GND
- C61 pad 2: -12VDC -> GND
- C62 pad 2: -12VDC -> GND
- C63 pad 1: -12VDC -> GND
- D101 pad 1: -12VDC -> GND
- D102 pad 1: -12VDC -> GND
- D14 pad 1: -12VDC -> GND
- D16 pad 2: -12VDC -> GND
- D18 pad 2: -12VDC -> GND
- D20 pad 2: -12VDC -> GND
- J10 pad 1: -12VDC -> GND
- J102 pad 1: -12VDC -> GND
- J103 pad 1: -12VDC -> GND
- J11 pad 2: -12VDC -> GND
- J13 pad 1: -12VDC -> GND
- J2 pad 1: -12VDC -> GND
- J8 pad 2: -12VDC -> GND
- J9 pad 1: -12VDC -> GND
- PS1 pad 3: -12VDC -> GND
- PS101 pad 2: -12VDC -> GND
- Q1 pad 1: -12VDC -> GND
- R102 pad 2: -12VDC -> GND
- R117 pad 2: -12VDC -> GND
- R119 pad 2: -12VDC -> GND
- R120 pad 2: -12VDC -> GND
- R121 pad 2: -12VDC -> GND
- R22 pad 1: -12VDC -> GND
- R38 pad 1: Net-(U5-Vout) -> Net-(U7-ANODE)
- R38 pad 2: Net-(U7-ANODE) -> Net-(U5-Vout)
- R45 pad 2: -12VDC -> GND
- R46 pad 2: -12VDC -> GND
- R47 pad 2: -12VDC -> GND
- R48 pad 2: -12VDC -> GND
- R51 pad 2: -12VDC -> GND
- R52 pad 2: -12VDC -> GND
- R53 pad 2: -12VDC -> GND
- R54 pad 2: -12VDC -> GND
- R57 pad 2: -12VDC -> GND
- R58 pad 2: -12VDC -> GND
- R59 pad 2: -12VDC -> GND
- R60 pad 2: -12VDC -> GND
- SW101 pad 1: -12VDC -> GND
- TP1 pad 1: -12VDC -> GND
- U1 pad 2: -12VDC -> GND
- U10 pad 5: -12VDC -> GND
- U10 pad 9: -12VDC -> GND
- U101 pad 1: -12VDC -> GND
- U101 pad 6: -12VDC -> GND
- U102 pad 23: -12VDC -> GND
- U102 pad 35: -12VDC -> GND
- U102 pad 47: -12VDC -> GND
- U102 pad 49: -12VDC -> GND
- U102 pad 8: AGND -> GND
- U103 pad 1: -12VDC -> GND
- U104 pad 4: -12VDC -> GND
- U105 pad 10: -12VDC -> GND
- U105 pad 11: -12VDC -> GND
- U105 pad 12: -12VDC -> GND
- U105 pad 13: -12VDC -> GND
- U105 pad 5: -12VDC -> GND
- U105 pad 6: -12VDC -> GND
- U105 pad 7: -12VDC -> GND
- U105 pad 8: -12VDC -> GND
- U105 pad 9: -12VDC -> GND
- U106 pad 4: -12VDC -> GND
- U106 pad 7: -12VDC -> GND
- U107 pad 2: -12VDC -> GND
- U11 pad 5: -12VDC -> GND
- U11 pad 9: -12VDC -> GND
- U7 pad 3: -12VDC -> GND
- U9 pad 5: -12VDC -> GND
- U9 pad 9: -12VDC -> GND
Routing:
- net -12VDC: track 1069.6 -> 0.00 mm, vias 35 -> 0
- net GND: track 0.00 -> 1040.2 mm, vias 0 -> 28
- net /PZEM_RXD: track 46.4 -> 2.52 mm, vias 2 -> 0
- net /Neutral: track 261.3 -> 301.4 mm, vias 4 -> 1
- net /PZEM_TXD: track 41.4 -> 2.59 mm
- net Net-(U5-Vout): track 112.4 -> 78.2 mm, vias 7 -> 4
- net /Relay/IO_PIN: track 45.1 -> 14.6 mm, vias 0 -> 1
- net Net-(D9-A): track 48.6 -> 18.7 mm
- net /PZEM/U8/1OUT: track 46.2 -> 21.3 mm, vias 3 -> 1
- net /PZEM/5VDC: track 37.0 -> 14.0 mm, vias 1 -> 0
- net Net-(R20-Pad2): track 27.8 -> 7.03 mm
- net Net-(C24-Pad1): track 42.3 -> 62.7 mm
- net Net-(D12-A): track 30.3 -> 12.7 mm
- net Net-(U102-PA3): track 20.2 -> 36.2 mm, vias 2 -> 0
- net Net-(U102-PA2): track 22.1 -> 36.4 mm, vias 2 -> 0
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Other:
- board size 246 x 122.6 mm -> 284.4 x 137.3 mm
- board text added: "3.3V"
- board text added: "5V"
- board text added: "CLK"
- board text added: "DIO"
- board text added: "G"
- board text added: "GND"
- board text added: "L"
- board text added: "N"
- board text added: "P"
- board text added: "RX"
- board text added: "S"
- board text added: "TX"
- board text added: "VCC"
