File: ACW_First/ACW_First.kicad_pcb (KiCad board)
At the start: 2 copper layers, 284.4 x 137.3 mm, 204 parts, among them J1 Screw_Terminal_01x02, J10 Conn_01x04_Pin, J101 Conn_01x02_Male, J102 Conn_STLink, J103 Conn_01x04_Female, J11 24VDC, J13 Conn_01x04_Socket, J2 Conn_01x03_Pin, J6 Screw_Terminal_01x02, J8 Conn_01x02_Pin, J9 Conn_01x03_Socket, K1 SRD-05VDC-SL-C, Q1 S8050, SW101 SW_Push, SW102 SW_Push, U1 PC817, U10 MP1584EN, U101 A7600_Pinout, U102 STM32F401CCUx, U103 AMS1117-3.3, U104 MCP6002-I_SN, U105 DS3231M, U106 AT24C512-SSHM, U107 PC817, U108 LM358PSR, U11 MP1584EN, U5 HT7133-1_C15060, U6 V9881D, U7 CT817C, U8 CT817C, U9 MP1584EN, Y101 8Mhz

Commit message: fix
Parts:
- moved R58 107.2 mm to (661.6, 42.5), turned to -90 degrees
- moved R59 106.2 mm to (659.7, 42.6), turned to -90 degrees
- moved BT1 102.0 mm to (629.9, 26.3)
- moved C10 102.0 mm to (680.2, 39.8)
- moved C12 102.0 mm to (718.4, 50.5)
- moved C13 102.0 mm to (708.8, 50.3)
- moved C14 102.0 mm to (699.3, 48.1)
- moved C17 102.0 mm to (682.3, 54.8)
- moved C18 102.0 mm to (719.1, 54.8)
- moved C19 102.0 mm to (654.9, 54.0)
- moved C20 102.0 mm to (639.3, 56.4)
- moved C22 102.0 mm to (716.3, 59.6)
- moved C24 102.0 mm to (675.0, 64.4)
- moved C25 102.0 mm to (680.8, 64.7)
- moved C26 102.0 mm to (716.2, 61.8)
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- renumbered BT101 to BT1, C24 to C1, C61 to C10, C108 to C11, C42 to C12, C45 to C13, C49 to C14, C52 to C15, C50 to C16, C59 to C17, C43 to C18, C101 to C19, C29 to C2, C102 to C20, C53 to C21, C46 to C22, C51 to C23, C58 to C24, C57 to C25, C44 to C26, C54 to C27, C56 to C28, C47 to C29, C32 to C3, C60 to C30, C55 to C31, C34 to C32, C37 to C33, C35 to C34, C38 to C35, C39 to C36, C36 to C37, C30 to C38, C40 to C39, C63 to C4, C27 to C40, C28 to C41, C33 to C42, C31 to C43, C26 to C44, C25 to C45, C114 to C46, C113 to C47, C112 to C48, C111 to C49, C62 to C5, C110 to C50, C105 to C51, C104 to C52, C115 to C53, C116 to C54, C109 to C55, C103 to C56, C107 to C6, C106 to C7, C48 to C8, C41 to C9, D12 to D1, D19 to D10, D10 to D11, D20 to D12, D16 to D13, D18 to D14, D13 to D2, D14 to D3, D11 to D4, D9 to D5, D101 to D6, D102 to D7, D17 to D8, D15 to D9, F4 to F1, F3 to F2, F5 to F3, F6 to F4, H3 to H1, H5 to H10, H8 to H11, H6 to H12, H101 to H2, H1 to H3, H103 to H4, H104 to H5, H102 to H6, H4 to H7, H2 to H8, H7 to H9, J8 to J1, J13 to J10, J2 to J11, J10 to J2, J9 to J3, J1 to J4, J6 to J5, J102 to J6, J103 to J7, J101 to J8, J11 to J9, L6 to L1, L4 to L2, L5 to L3, PS101 to PS2, R24 to R1, R112 to R10, R45 to R11, R44 to R12, R107 to R13, R108 to R14, R102 to R15, R101 to R16, R52 to R17, R46 to R18, R115 to R19, R43 to R2, R114 to R20, R47 to R21, R53 to R22, R55 to R23, R48 to R24, R49 to R25, R54 to R26, R59 to R27, R105 to R28, R106 to R29, R31 to R3, R109 to R30, R110 to R31, R42 to R32, R40 to R33, R41 to R34, R39 to R35, R20 to R36, R36 to R37, R37 to R38, R38 to R39, R34 to R4, R21 to R40, R22 to R41, R29 to R42, R28 to R43, R30 to R44, R33 to R45, R32 to R46, R27 to R47, R26 to R48, R25 to R49, R35 to R5, R118 to R50, R121 to R51, R113 to R52, R122 to R53, R116 to R54, R119 to R55, R123 to R56, R120 to R57, R103 to R58, R104 to R59, R50 to R6, R61 to R60, R60 to R61, R124 to R62, R58 to R63, R125 to R64, R126 to R65, R129 to R66, R127 to R67, R128 to R68, R56 to R69, R111 to R7, R57 to R70, R51 to R8, R117 to R9, RV3 to RV1, SW102 to SW1, SW101 to SW2, TH2 to TH1, TP8 to TP3, TP6 to TP4, TP7 to TP5, U102 to U1, U6 to U10, U5 to U11, U105 to U12, U106 to U13, U104 to U14, U107 to U15, U108 to U16, U10 to U2, U9 to U3, U11 to U4, U101 to U5, U103 to U6, U8 to U7, U7 to U8, U1 to U9, Y101 to Y1, Y1 to Y2
Routing:
- net GND: track 1040.2 -> 1059.2 mm
- net +3.3V: track 225.2 -> 212.6 mm
- net /Controller/SCL_RTC: track 32.7 -> 24.0 mm
- net /Controller/SDA_RTC: track 33.1 -> 25.2 mm
- net Net-(U102-PB6): track 13.7 -> 20.0 mm
- net Net-(U6-P0.1/TDI): track 17.3 -> 13.5 mm
- net AGND: track 99.4 -> 102.6 mm
- net Net-(U102-PB7): track 14.5 -> 16.8 mm
- net /Relay/5V: track 85.4 -> 83.4 mm
- net /Neutral: track 301.4 -> 300.0 mm
- net Net-(C24-Pad1): track 62.7 -> 64.1 mm
- net Net-(C24-Pad2): track 9.95 -> 8.89 mm
- net /Controller/PWM_Input: track 18.8 -> 18.2 mm
- net /RELAY_DATA: track 103.7 -> 103.3 mm, vias 2 -> 0
- added copper zone on B.Cu, net AGND
- added copper zone on B.Cu, net GND
- added copper zone on F.Cu, net GND
- added copper zone on B.Cu, net IGND
Other:
- board size 284.4 x 137.3 mm -> 212.3 x 65.1 mm

Commit message: okok
Parts:
- C47, C49, C50, C51, C52, C53, C54, R50, R51, R52, R53, R54, R55, R56, R57, R58, R59, R62, R64, R65, R66, R67, R68, U13, U14, U16: moved to F.Cu
- J6: value Conn_STLink -> Conn_01x03_Pin; footprint Connector_JST:JST_XH_B4B-XH-A_1x04_P2.50mm_Vertical -> Connector_JST:JST_XH_B3B-XH-A_1x03_P2.50mm_Vertical
- J7: value Conn_01x04_Female -> Conn_01x03_Socket; footprint Connector_JST:JST_XH_B4B-XH-A_1x04_P2.50mm_Vertical -> Connector_JST:JST_XH_B3B-XH-A_1x03_P2.50mm_Vertical
- L3: footprint Inductor_SMD:L_Bourns-SRR1005 -> Inductor_SMD:L_7.3x7.3_H4.5
- R42: value 750Ω -> 100Ω
- U15: footprint Custom_Library:SOP254P975X460-4N -> Custom_Footprints:SOP-4_L6.4-W4.6-P2.54-LS10.2-TL; moved to F.Cu
- moved J8 152.8 mm to (745.5, 181.7)
- moved PS2 135.3 mm to (677.3, 182.9), turned to 180 degrees
- moved SW1 131.1 mm to (708.4, 164.1), turned to 90 degrees
- moved R15 125.0 mm to (694.0, 162.4), turned to -90 degrees
- moved SW2 124.8 mm to (704.9, 164.1), turned to 90 degrees
- moved R16 121.6 mm to (699.2, 162.4), turned to 90 degrees
- moved R66 116.7 mm to (672.5, 175.8), turned to 90 degrees
- moved C19 116.3 mm to (696.9, 162.4), turned to 90 degrees
- moved R65 115.3 mm to (692.9, 172.8)
- moved C53 115.3 mm to (689.2, 176.2)
- moved C54 115.3 mm to (687.0, 176.2)
- moved R64 115.3 mm to (679.3, 168.9)
- moved R68 115.3 mm to (692.9, 176.3)
- moved U16 115.3 mm to (679.7, 174.6), turned to 180 degrees
- moved R67 115.3 mm to (692.9, 174.5)
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Connections:
- C41 pad 1: Net-(U6-REF) -> Net-(U10-REF)
- R42 pad 1: /Neutral -> Net-(U10-REF)
- R42 pad 2: Net-(U6-REF) -> /Neutral
- R43 pad 1: Net-(U6-REF) -> Net-(U10-REF)
- U10 pad 24: Net-(U6-REF) -> Net-(U10-REF)
Routing:
- net GND: track 1059.2 -> 1416.1 mm, vias 28 -> 33
- net /Controller/Dimm_Circuit/Dim_Output-: track 19.0 -> 99.9 mm, vias 0 -> 1
- net /Controller/Dimm_Circuit/Dim_Output+: track 21.4 -> 80.9 mm, vias 0 -> 1
- net 12VDC: track 151.6 -> 95.2 mm
- net 3.8VDC: track 91.0 -> 127.4 mm, vias 2 -> 5
- net /Controller/BOOT0: track 9.96 -> 39.3 mm, vias 2 -> 5
- net Net-(PS2-+VOUT): track 15.5 -> 37.2 mm
- net 5VDC: track 233.1 -> 214.9 mm
- net Net-(U1-PB14): track 36.5 -> 20.0 mm
- net Net-(U10-REF): track 0.00 -> 15.4 mm, vias 0 -> 2
- net Net-(U6-REF): track 15.3 -> 0.00 mm, vias 2 -> 0
- net /Controller/NRST: track 23.8 -> 38.3 mm, vias 2 -> 4
- net /Controller/SCL_RTC: track 24.0 -> 37.9 mm, vias 4 -> 2
- net /Controller/PWM_Input: track 18.2 -> 31.3 mm, vias 3 -> 2
- net Net-(U1-PA2): track 36.4 -> 24.9 mm
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- removed copper zone on B.Cu, net IGND
Other:
- board size 212.3 x 65.1 mm -> 239.4 x 70.1 mm
- board text removed: "3.3V"
- board text removed: "5V"
- board text removed: "CLK"
- board text removed: "DIO"
- board text removed: "G"
- board text removed: "GND"
- board text removed: "P"
- board text removed: "RX"
- board text removed: "S"
- board text removed: "TX"
- board text removed: "VCC"

Commit message: okok
Routing:
- net GND: track 1416.1 -> 1536.9 mm
- net /RELAY_DATA: track 103.2 -> 102.0 mm
- added copper zone on F.Cu, net IGND
Changed lines of the file:
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@@
 		(tags "capacitor")
 		(property "Reference" "C47"
-			(at 20.48 4.82 180)
+			(at 2.15 0.03 180)
 			(layer "F.SilkS")
 			(effects
@@
 		(tags "resistor")
 		(property "Reference" "R51"
-			(at -0.8288 16.46 180)
+			(at -2.49 0.81 270)
 			(layer "F.SilkS")
 			(effects
@@
 			(at -3.54 -0.06 0)
 			(layer "F.SilkS")
-			(hide yes)
 			(effects
 				(font
@@
 		(tags "resistor")
 		(property "Reference" "R56"
-			(at 3.025 -0.05 90)
+			(at 3.09 -0.03 90)
 			(layer "F.SilkS")
 			(effects
@@
 			(at -3.43 -0.28 0)
 			(layer "F.SilkS")
-			(hide yes)
 			(effects
 				(font
@@
 		(tags "resistor")
 		(property "Reference" "R57"
-			(at -22.005 -9.41 90)
+			(at 2.49 0.39 270)
 			(layer "F.SilkS")
 			(effects
@@
 		(tags "resistor")
 		(property "Reference" "R55"
-			(at -0.237258 1.77 90)
+			(at 0.81 -2.6 180)
 			(layer "F.SilkS")
 			(effects
@@
 	(gr_poly
 		(pts
-			(xy 670.574996 117.275004) (xy 670.6 117.25) (xy 670.6 117.54) (xy 734.05 117.54) (xy 734.04 117.55)
-			(xy 734.04 117.38) (xy 734.04 117.264998)
-		)
-		(stroke
-			(width 0.2)
-			(type solid)
-		)
-		(fill yes)
-		(layer "B.Cu")
-		(net "GND")
-	)
-	(gr_poly
-		(pts
 			(xy 525.81 151.301292) (xy 523.05 154.061292) (xy 523.05 156.391292) (xy 523.32 156.661292) (xy 525.86 156.661292)
 			(xy 526.24 156.281292) (xy 526.24 151.401292) (xy 526.14 151.301292)
@@
 	)
 	(segment
+		(start 743.93672 117.88328)
+		(end 742.233318 117.88328)
+		(width 1.5)
+		(layer "F.Cu")
+		(net "GND")
+	)
+	(segment
 		(start 689.22 132.58328)
 		(end 691.36 132.58328)
@@
 	)
 	(segment
-		(start 742.32 117.88328)
-		(end 697.27672 117.88328)
-		(width 1.5)
-		(layer "F.Cu")
-		(net "GND")
-	)
-	(segment
 		(start 721.84 134.37328)
 		(end 721.3 134.91328)
@@
 	)
 	(segment
-		(start 743.085019 118.648299)
-		(end 742.32 117.88328)
-		(width 1.5)
-		(layer "F.Cu")
-		(net "GND")
-	)
-	(segment
 		(start 705.84 135.52)
 		(end 706.19 135.52)
@@
 	)
 	(segment
+		(start 742.233318 117.88328)
+		(end 697 117.88328)
+		(width 1.5)
+		(layer "F.Cu")
+		(net "GND")
+	)
+	(segment
 		(start 660.78 137.08)
 		(end 660.78 137.41)
@@
 	)
 	(segment
-		(start 743.93672 117.88328)
-		(end 742.32 117.88328)
-		(width 1.5)
-		(layer "F.Cu")
-		(net "GND")
-	)
-	(segment
 		(start 720.45 163.68828)
 		(end 719.825 163.06328)
@@
 	)
 	(segment
-		(start 743.085019 118.734981)
-		(end 743.085019 118.648299)
-		(width 1.5)
-		(layer "F.Cu")
-		(net "GND")
-	)
-	(segment
 		(start 748.825001 155.06828)
 		(end 747.335 153.578279)
@@
 	)
 	(segment
+		(start 743.085019 118.734981)
+		(end 742.233318 117.88328)
+		(width 1.5)
+		(layer "F.Cu")
+		(net "GND")
+	)
+	(segment
 		(start 732.86 156.55328)
 		(end 732.86 158.25328)
@@
 	)
 	(segment
-		(start 687.635 129.973096)
-		(end 690.752316 126.85578)
-		(width 0.5)
+		(start 742.13328 117.63328)
+		(end 696.5 117.63328)
+		(width 1)
 		(layer "B.Cu")
 		(net "GND")
 	)
 	(segment
-		(start 733.83 117.88328)
-		(end 733.33 117.38328)
+		(start 687.635 129.973096)
+		(end 690.752316 126.85578)
 		(width 0.5)
 		(layer "B.Cu")
@@
 	)
 	(segment
+		(start 748.13328 117.63328)
+		(end 760 129.5)
+		(width 1)
+		(layer "B.Cu")
+		(net "GND")
+	)
+	(segment
 		(start 721.37 177.45328)
 		(end 723.41 175.41328)
@@
 	)
 	(segment
+		(start 743.085019 119.91328)
+		(end 743.085019 118.585019)
+		(width 1)
+		(layer "B.Cu")
+		(net "GND")
+	)
+	(segment
 		(start 741.335 175.12828)
 		(end 741.335 174.28328)
@@
 	)
 	(segment
-		(start 743.085019 118.711199)
-		(end 742.2571 117.88328)
-		(width 1.5)
-		(layer "B.Cu")
-		(net "GND")
-	)
-	(segment
 		(start 726.71 166.35328)
 		(end 728.68 168.32328)
@@
 	)
 	(segment
+		(start 760 129.5)
+		(end 760 176.5)
+		(width 1)
+		(layer "B.Cu")
+		(net "GND")
+	)
+	(segment
 		(start 737.335 167.76328)
 		(end 737.335 125.62828)
@@
 	)
 	(segment
+		(start 743.085019 118.585019)
+		(end 743.085019 118.548261)
+		(width 1)
+		(layer "B.Cu")
+		(net "GND")
+	)
+	(segment
 		(start 678.61328 155.47328)
 		(end 682.03328 155.47328)
@@
 	)
 	(segment
-		(start 733.33 117.38328)
-		(end 725.1 117.38328)
-		(width 0.5)
+		(start 743.085019 118.585019)
+		(end 742.13328 117.63328)
+		(width 1)
 		(layer "B.Cu")
 		(net "GND")
@@
 	)
 	(segment
-		(start 743.085019 119.91328)
-		(end 743.085019 118.711199)
-		(width 1.5)
-		(layer "B.Cu")
-		(net "GND")
-	)
-	(segment
 		(start 731.16 176.36328)
 		(end 731.92 175.60328)
@@
 	)
 	(segment
+		(start 743.085019 118.548261)
+		(end 744 117.63328)
+		(width 1)
+		(layer "B.Cu")
+		(net "GND")
+	)
+	(segment
 		(start 690.752316 126.85578)
 		(end 691.36 126.85578)
@@
 	)
 	(segment
+		(start 659.61 127.98328)
+		(end 659.61 145.05)
+		(width 0.5)
+		(layer "B.Cu")
+		(net "GND")
+	)
+	(segment
 		(start 742.49 173.07328)
 		(end 741.415 173.07328)
@@
 	)
 	(segment
+		(start 742.13328 117.63328)
+		(end 744 117.63328)
+		(width 1)
+		(layer "B.Cu")
+		(net "GND")
+	)
+	(segment
 		(start 675.11 125.00328)
 		(end 675.44 124.67328)
@@
 	)
 	(segment
+		(start 744 117.63328)
+		(end 748.13328 117.63328)
+		(width 1)
+		(layer "B.Cu")
+		(net "GND")
+	)
+	(segment
 		(start 746.36 173.07328)
 		(end 746.4 173.07328)
@@
 	)
 	(segment
+		(start 662.27 125.32328)
+		(end 659.61 127.98328)
+		(width 0.5)
+		(layer "B.Cu")
+		(net "GND")
+	)
+	(segment
 		(start 693.0125 151.55828)
 		(end 694.6525 149.91828)
@@
 	)
 	(segment
-		(start 742.2571 117.88328)
-		(end 733.83 117.88328)
-		(width 1.5)
-		(layer "B.Cu")
-		(net "GND")
-	)
-	(segment
 		(start 718.96 176.57328)
 		(end 719.025 176.57328)
@@
 	)
 	(segment
-		(start 669.2 118.08)
-		(end 731.22 118.08)
+		(start 730.156739 118.5)
+		(end 731.610019 119.95328)
 		(width 0.3)
 		(layer "B.Cu")
@@
 	(segment
 		(start 665.68 121.6)
-		(end 669.2 118.08)
+		(end 668.78 118.5)
 		(width 0.3)
 		(layer "B.Cu")
@@
 	)
 	(segment
-		(start 731.22 118.08)
-		(end 731.610019 118.470019)
-		(width 0.3)
-		(layer "B.Cu")
-		(net "/RELAY_DATA")
-	)
-	(segment
-		(start 731.610019 118.470019)
-		(end 731.610019 119.95328)
+		(start 668.78 118.5)
+		(end 730.156739 118.5)
 		(width 0.3)
 		(layer "B.Cu")
@@
 	)
 	(zone
+		(net "IGND")
+		(layer "F.Cu")
+		(name "IGND")
+		(hatch edge 0.5)
+		(priority 6)
+		(connect_pads
+			(clearance 0.1)
+		)
+		(min_thickness 0.25)
+		(fill yes
+			(thermal_gap 0.5)
+			(thermal_bridge_width 0.5)
+			(island_removal_mode 0)
+		)
+		(polygon
+			(pts
+				(xy 670 168.5) (xy 697 168.5) (xy 697.5 169) (xy 697.5 179) (xy 696.5 180) (xy 684.5 180) (xy 679 183.5)
+				(xy 679 185) (xy 678 186) (xy 673 186) (xy 669 179.5) (xy 669 169.5)
+			)
+		)
+	)
+	(zone
 		(net "GND")
 		(layer "F.Cu")
@@
 		(net "GND")
 		(layer "F.Cu")
-		(name "GND_2")
+		(name "GND_4")
 		(hatch edge 0.5)
-		(priority 4)
+		(priority 7)
 		(connect_pads
-			(clearance 0)
+			(clearance 0.1)
 		)
 		(min_thickness 0.25)
@@
 		(polygon
 			(pts
-				(xy 714.78 178.21828) (xy 712.955 176.39328) (xy 712.955 172.34328) (xy 716.305 168.99328) (xy 716.305 162.61828)
-				(xy 716.705 162.21828) (xy 723.53 162.21828) (xy 724.18 161.56828) (xy 724.18 151.69328) (xy 725.53 150.34328)
-				(xy 732.205 150.34328) (xy 733.23 151.36828) (xy 733.23 154.39328) (xy 733.705 154.86828) (xy 740.38 154.86828)
-				(xy 741.78 156.26828) (xy 741.78 176.06828) (xy 739.63 178.21828) (xy 723.58 178.21828)
+				(xy 693.5 119) (xy 731 119) (xy 731.5 119.5) (xy 731.5 124.5) (xy 730.5 125.5) (xy 727.5 125.5)
+				(xy 724 122) (xy 693.5 122) (xy 693 121.5) (xy 693 119.5)
 			)
 		)
@@
 	(zone
 		(net "GND")
-		(layer "B.Cu")
-		(name "GND")
+		(layer "F.Cu")
+		(name "GND_2")
 		(hatch edge 0.5)
-		(priority 1)
+		(priority 4)
 		(connect_pads
 			(clearance 0)
@@
 		(polygon
 			(pts
-				(xy 596.15 117.66) (xy 597.12 118.63) (xy 597.12 122.26) (xy 596.17 123.21) (xy 571.52 123.21) (xy 568.18 126.55)
-				(xy 568.18 129.09) (xy 566.76 130.51) (xy 549.94 130.51) (xy 547.86 128.43) (xy 547.86 117.67) (xy 547.87 117.66)
-				(xy 548.6 117.66)
+				(xy 714.78 178.21828) (xy 712.955 176.39328) (xy 712.955 172.34328) (xy 716.305 168.99328) (xy 716.305 162.61828)
+				(xy 716.705 162.21828) (xy 723.53 162.21828) (xy 724.18 161.56828) (xy 724.18 151.69328) (xy 725.53 150.34328)
+				(xy 732.205 150.34328) (xy 733.23 151.36828) (xy 733.23 154.39328) (xy 733.705 154.86828) (xy 740.38 154.86828)
+				(xy 741.78 156.26828) (xy 741.78 176.06828) (xy 739.63 178.21828) (xy 723.58 178.21828)
 			)
 		)
@@
 		(net "GND")
 		(layer "B.Cu")
-		(name "GND_4")
+		(name "GND")
 		(hatch edge 0.5)
-		(priority 6)
+		(priority 1)
 		(connect_pads
 			(clearance 0)
@@
 		(polygon
 			(pts
-				(xy 693.805 118.04328) (xy 693.805 122.39328) (xy 696.08 124.66828) (xy 709.155 124.66828) (xy 710.755 123.06828)
-				(xy 725.83 123.06828) (xy 728.105 125.34328) (xy 731.755 125.34328) (xy 734.68 122.41828) (xy 734.68 118.84328)
-				(xy 733.63 117.79328) (xy 694.055 117.79328)
+				(xy 596.15 117.66) (xy 597.12 118.63) (xy 597.12 122.26) (xy 596.17 123.21) (xy 571.52 123.21) (xy 568.18 126.55)
+				(xy 568.18 129.09) (xy 566.76 130.51) (xy 549.94 130.51) (xy 547.86 128.43) (xy 547.86 117.67) (xy 547.87 117.66)
+				(xy 548.6 117.66)
 			)
 		)

Commit message: okok
Parts:
- moved C30 0.25 mm to (714.2, 165.9)
Routing:
- net GND: track 1536.9 -> 1151.2 mm, vias 33 -> 31
- net AGND: track 102.6 -> 105.4 mm, vias 1 -> 2
- net Net-(PS2-+VOUT): track 37.2 -> 35.6 mm
- net /Power/COMP INPUT for 3.8VDC: track 10.5 -> 9.92 mm
- net 3.8VDC: vias 5 -> 3
- net /Controller/SCL_RTC: vias 2 -> 1
- added copper zone on F.Cu, net (none)
- added copper zone on F.Cu, net AGND
Other:
- outline, holes or cut-outs redrawn
