File: ACW_First/ACW_First.kicad_sch (KiCad schematic)
At the start: 8 parts, among them J1 Screw_Terminal_01x02, J2 RELAYIOPIN, J3 3.8VDC, J4 5VDC, J5 12VDC, J6 STMRX/TX PINS, J7 Conn_01x02_Socket, J9 24VDCPINS

Commit message: okok
Parts:
- removed J2: RELAYIOPIN, Connector_PinSocket_2.54mm:PinSocket_1x02_P2.54mm_Vertical, symbol Connector:Conn_01x02_Socket
- removed J6: STMRX/TX PINS, Connector_PinSocket_2.54mm:PinSocket_1x02_P2.54mm_Vertical, symbol Connector:Conn_01x02_Socket
- removed J7: Conn_01x02_Socket, Connector_PinSocket_2.54mm:PinSocket_1x02_P2.54mm_Vertical, symbol Connector:Conn_01x02_Socket
- removed J9: 24VDCPINS, Connector_PinHeader_2.54mm:PinHeader_1x02_P2.54mm_Vertical, symbol Connector:Conn_01x02_Pin
- added H1, H2, H3, H4: MountingHole, MountingHole:MountingHole_3.2mm_M3, symbol Mechanical:MountingHole
- added J10: Conn_01x04_Pin, Connector_PinHeader_2.54mm:PinHeader_1x04_P2.54mm_Vertical, symbol Connector:Conn_01x04_Pin
- added J11: 24VDC, Connector_PinSocket_2.54mm:PinSocket_1x02_P2.54mm_Vertical, symbol Connector:Conn_01x02_Socket
- added J12, J14: Conn_01x02_Pin, Connector_PinSocket_2.54mm:PinSocket_1x02_P2.54mm_Vertical, symbol Connector:Conn_01x02_Pin
- added J13: Conn_01x04_Socket, Connector_PinSocket_2.54mm:PinSocket_1x04_P2.54mm_Vertical, symbol Connector:Conn_01x04_Socket
- added J2: Conn_01x03_Pin, Connector_PinHeader_2.54mm:PinHeader_1x03_P2.54mm_Vertical, symbol Connector:Conn_01x03_Pin
- added J6: Screw_Terminal_01x02, TerminalBlock_MetzConnect:TerminalBlock_MetzConnect_Type101_RT01602HBWC_1x02_P5.08mm_Horizontal, symbol Connector:Screw_Terminal_01x02
- added J7: Screw_Terminal_01x04, TerminalBlock_MetzConnect:TerminalBlock_MetzConnect_Type101_RT01604HBWC_1x04_P5.08mm_Horizontal, symbol Connector:Screw_Terminal_01x04
- added J8: Conn_01x02_Pin, Connector_PinHeader_2.54mm:PinHeader_1x02_P2.54mm_Vertical, symbol Connector:Conn_01x02_Pin
- added J9: Conn_01x03_Socket, Connector_PinSocket_2.54mm:PinSocket_1x03_P2.54mm_Vertical, symbol Connector:Conn_01x03_Socket
Connections:
- net PZEM/RX: now also J10.4 (Pin_4)
- net PZEM/TX: now also J10.3 (Pin_3)
- net Relay/IO_PIN: now also J9.3 (Pin_3)
- net 24VDC to 5VDC/5VDC renamed 5VDC
- net 5VDC: now also J2.2 (Pin_2)
- net LI renamed Live
- net N renamed Neutral
- new net: J12.1 (Pin_1), J2.3 (Pin_3)
- new net -24VDC: J11.2 (Pin_2)
- new net 24VDC: J11.1 (Pin_1)
- new net GND: J10.1 (Pin_1), J13.1 (Pin_1), J2.1 (Pin_1), J9.1 (Pin_1)
- new net LIVE to 24V/-24VDC: J8.2 (Pin_2)
- new net LIVE to 24V/24VDC: J8.1 (Pin_1)
- new net PZEM/5VDC: J10.2 (Pin_2)
- new net PZEM/CT1: J7.1 (Pin_1)
- new net PZEM/CT2: J7.2 (Pin_2)
- new net PZEM/L: J7.4 (Pin_4)
- new net PZEM/N: J7.3 (Pin_3)
- new net Relay/5V: J9.2 (Pin_2)
- new net Relay/COM: J6.1 (Pin_1)
- new net Relay/NO: J6.2 (Pin_2)
- no-connect marks 0 -> 1
Other:
- sheet PZEM ports: added CT1, CT2; removed CT
- sheet Relay ports: added 5V, COM, NO; removed LI, LO

Commit message: add firstlevel & secondlevevl pcb
Connections:
- net 5VDC: now also J13.2 (Pin_2)
- net at J13.3 (Pin_3): now also J14.1 (Pin_1)
- net at J13.4 (Pin_4): now also J14.2 (Pin_2)
Changed lines of the file:
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@@
+	(wire
+		(pts
+			(xy 43.18 237.49) (xy 57.15 237.49)
+		)
+		(stroke
+			(width 0)
+			(type default)
+		)
+	)
 	(wire
 		(pts
@@
 	(wire
 		(pts
+			(xy 43.18 240.03) (xy 57.15 240.03)
+		)
+		(stroke
+			(width 0)
+			(type default)
+		)
+	)
+	(wire
+		(pts
 			(xy 175.26 53.34) (xy 175.26 111.76)
 		)
@@
 		(pts
 			(xy 52.07 224.79) (xy 52.07 219.71)
+		)
+		(stroke
+			(width 0)
+			(type default)
+		)
+	)
+	(wire
+		(pts
+			(xy 43.18 242.57) (xy 48.26 242.57)
 		)
 		(stroke
@@
 		(effects
 			(font
+				(size 1.27 1.27)
+			)
+			(justify left bottom)
+		)
+	)
+	(label "5VDC"
+		(at 48.26 242.57 0)
+		(effects
+			(font

Commit message: okokok
Parts:
- removed J3: 3.8VDC, Connector_PinHeader_2.54mm:PinHeader_1x02_P2.54mm_Vertical, symbol Connector:Conn_01x02_Pin
- removed J4: 5VDC, Connector_PinHeader_2.54mm:PinHeader_1x02_P2.54mm_Vertical, symbol Connector:Conn_01x02_Pin
- removed J5: 12VDC, Connector_PinHeader_2.54mm:PinHeader_1x02_P2.54mm_Vertical, symbol Connector:Conn_01x02_Pin
- removed J7: Screw_Terminal_01x04, TerminalBlock_MetzConnect:TerminalBlock_MetzConnect_Type101_RT01604HBWC_1x04_P5.08mm_Horizontal, symbol Connector:Screw_Terminal_01x04
Connections:
- net Relay/COM is gone; now on net Relay/NO: J6.1 (Pin_1)
- net Relay/NO: no longer J6.2 (Pin_2)
- new net Neutral_OutPZEM: J6.2 (Pin_2)
Other:
- sheet LIVE to 24V renamed Power
- removed sheet 24VDC to 12VDC
- removed sheet 24VDC to 5VDC
- removed sheet 5VDC to 3.8VDC
- sheet Power: file LIVE_to_24V.kicad_sch -> Power.kicad_sch
- sheet Relay ports: added NeutralInput; removed none
- moved on the sheet: J10, J6, J8

Commit message: revisi
Connections:
- net Power/-24VDC is gone; now on net -24VDC: J8.2 (Pin_2)
- net Power/24VDC is gone; now on net 24VDC: J8.1 (Pin_1)
Other:
- added sheet Controller (Controller.kicad_sch)
- sheet Power ports: added 3.8VDC, 5VDC; removed none
- moved on the sheet: J10, J8

Commit message: okok
Parts:
- removed J12, J14: Conn_01x02_Pin, Connector_PinSocket_2.54mm:PinSocket_1x02_P2.54mm_Vertical, symbol Connector:Conn_01x02_Pin
- added H5, H6, H7, H8: MountingHole, MountingHole:MountingHole_3.2mm_M3, symbol Mechanical:MountingHole
Connections:
- net RELAY_DATA: now reaches J2.3 (Pin_3)
- net PZEM_TXD: now reaches J13.3 (Pin_3)
- net PZEM_RXD: now reaches J13.4 (Pin_4)
Other:
- sheet Controller ports: added PZEM_RXD, PZEM_TXD, RELAY_DATA; removed none
- sheet Power ports: added none; removed 3.8VDC, 5VDC

Commit message: okok
Connections:
- net -24VDC is gone; now on net GND: J11.2 (Pin_2), J8.2 (Pin_2)
- no-connect marks 1 -> 0
Other:
- sheet Power ports: added none; removed -24VDC
- moved on the sheet: J11, J13, J2, J8

Commit message: fix
Parts:
- renumbered J9 to J1, J11 to J2, J8 to J3, J13 to J4, J2 to J5, J1 to J6, J10 to J7, J6 to J8
Changed lines of the file:
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@@
 		(dnp no)
 		(fields_autoplaced yes)
-		(property "Reference" "#PWR06"
+		(property "Reference" "#PWR04"
 			(at 81.28 217.17 0)
 			(hide yes)
@@
 			(project "ACW_First"
 				(path "/f90a1fa2-4579-4163-be1b-3b1c72ac9515"
-					(reference "#PWR06")
+					(reference "#PWR04")
 					(unit 1)
 				)
@@
 		(in_pos_files yes)
 		(dnp no)
-		(property "Reference" "J11"
+		(property "Reference" "J2"
 			(at 32.004 214.63 0)
 			(show_name no)
@@
 			(project "ACW_First"
 				(path "/f90a1fa2-4579-4163-be1b-3b1c72ac9515"
-					(reference "J11")
+					(reference "J2")
 					(unit 1)
 				)
@@
 		(dnp no)
 		(fields_autoplaced yes)
-		(property "Reference" "J2"
+		(property "Reference" "J5"
 			(at 73.025 222.25 0)
 			(show_name no)
@@
 			(project "ACW_First"
 				(path "/f90a1fa2-4579-4163-be1b-3b1c72ac9515"
-					(reference "J2")
+					(reference "J5")
 					(unit 1)
 				)
@@
 		(dnp no)
 		(fields_autoplaced yes)
-		(property "Reference" "#PWR02"
+		(property "Reference" "#PWR01"
 			(at 25.4 64.77 0)
 			(hide yes)
@@
 			(project "ACW_First"
 				(path "/f90a1fa2-4579-4163-be1b-3b1c72ac9515"
-					(reference "#PWR02")
+					(reference "#PWR01")
 					(unit 1)
 				)
@@
 		(in_pos_files yes)
 		(dnp no)
-		(property "Reference" "J13"
+		(property "Reference" "J4"
 			(at 67.564 193.548 0)
 			(show_name no)
@@
 			(project "ACW_First"
 				(path "/f90a1fa2-4579-4163-be1b-3b1c72ac9515"
-					(reference "J13")
+					(reference "J4")
 					(unit 1)
 				)
@@
 		(dnp no)
 		(fields_autoplaced yes)
-		(property "Reference" "#PWR09"
+		(property "Reference" "#PWR02"
 			(at 53.34 208.28 0)
 			(hide yes)
@@
 			(project "ACW_First"
 				(path "/f90a1fa2-4579-4163-be1b-3b1c72ac9515"
-					(reference "#PWR09")
+					(reference "#PWR02")
 					(unit 1)
 				)
@@
 		(in_pos_files yes)
 		(dnp no)
-		(property "Reference" "#PWR08"
+		(property "Reference" "#PWR03"
 			(at 53.34 226.06 0)
 			(hide yes)
@@
 			(project "ACW_First"
 				(path "/f90a1fa2-4579-4163-be1b-3b1c72ac9515"
-					(reference "#PWR08")
+					(reference "#PWR03")
 					(unit 1)
 				)
@@
 		(in_pos_files yes)
 		(dnp no)
-		(property "Reference" "J1"
+		(property "Reference" "J6"
 			(at 99.314 27.686 90)
 			(show_name no)
@@
 			(project "ACW_First"
 				(path "/f90a1fa2-4579-4163-be1b-3b1c72ac9515"
-					(reference "J1")
+					(reference "J6")
 					(unit 1)
 				)
@@
 		(in_pos_files yes)
 		(dnp no)
-		(property "Reference" "J6"
+		(property "Reference" "J8"
 			(at 143.256 41.656 90)
 			(show_name no)
@@
 			(project "ACW_First"
 				(path "/f90a1fa2-4579-4163-be1b-3b1c72ac9515"
-					(reference "J6")
+					(reference "J8")
 					(unit 1)
 				)
@@
 		(dnp no)
 		(fields_autoplaced yes)
-		(property "Reference" "J9"
+		(property "Reference" "J1"
 			(at 17.145 45.72 0)
 			(show_name no)
@@
 			(project "ACW_First"
 				(path "/f90a1fa2-4579-4163-be1b-3b1c72ac9515"
-					(reference "J9")
+					(reference "J1")
 					(unit 1)
 				)
@@
 		(in_pos_files yes)
 		(dnp no)
-		(property "Reference" "#PWR03"
+		(property "Reference" "#PWR05"
 			(at 87.63 243.84 0)
 			(hide yes)
@@
 			(project "ACW_First"
 				(path "/f90a1fa2-4579-4163-be1b-3b1c72ac9515"
-					(reference "#PWR03")
+					(reference "#PWR05")
 					(unit 1)
 				)
@@
 		(dnp no)
 		(fields_autoplaced yes)
-		(property "Reference" "J8"
+		(property "Reference" "J3"
 			(at 40.64 196.8501 0)
 			(show_name no)
@@
 			(project "ACW_First"
 				(path "/f90a1fa2-4579-4163-be1b-3b1c72ac9515"
-					(reference "J8")
+					(reference "J3")
 					(unit 1)
 				)
@@
 		(dnp no)
 		(fields_autoplaced yes)
-		(property "Reference" "#PWR01"
+		(property "Reference" "#PWR06"
 			(at 95.25 166.37 0)
 			(hide yes)
@@
 			(project "ACW_First"
 				(path "/f90a1fa2-4579-4163-be1b-3b1c72ac9515"
-					(reference "#PWR01")
+					(reference "#PWR06")
 					(unit 1)
 				)
@@
 		(dnp no)
 		(fields_autoplaced yes)
-		(property "Reference" "J10"
+		(property "Reference" "J7"
 			(at 105.41 154.9399 0)
 			(show_name no)
@@
 			(project "ACW_First"
 				(path "/f90a1fa2-4579-4163-be1b-3b1c72ac9515"
-					(reference "J10")
-					(unit 1)
-				)
+					(reference "J7")
+					(unit 1)
+				)

Commit message: okok
Parts:
- renumbered H3 to H1, H5 to H10, H8 to H11, H6 to H12, H1 to H3, H4 to H7, H2 to H8, H7 to H9, J3 to J1, J4 to J10, J5 to J11, J7 to J2, J1 to J3, J6 to J4, J8 to J5, J2 to J9
Changed lines of the file:
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@@
 		(dnp no)
 		(fields_autoplaced yes)
-		(property "Reference" "H1"
+		(property "Reference" "H3"
 			(at 127 222.2499 0)
 			(show_name no)
@@
 			(project "ACW_First"
 				(path "/f90a1fa2-4579-4163-be1b-3b1c72ac9515"
-					(reference "H1")
+					(reference "H3")
 					(unit 1)
 				)
@@
 		(dnp no)
 		(fields_autoplaced yes)
-		(property "Reference" "H7"
+		(property "Reference" "H9"
 			(at 156.21 233.6799 0)
 			(show_name no)
@@
 			(project "ACW_First"
 				(path "/f90a1fa2-4579-4163-be1b-3b1c72ac9515"
-					(reference "H7")
+					(reference "H9")
 					(unit 1)
 				)
@@
 		(in_pos_files yes)
 		(dnp no)
-		(property "Reference" "J2"
+		(property "Reference" "J9"
 			(at 32.004 214.63 0)
 			(show_name no)
@@
 			(project "ACW_First"
 				(path "/f90a1fa2-4579-4163-be1b-3b1c72ac9515"
-					(reference "J2")
+					(reference "J9")
 					(unit 1)
 				)
@@
 		(dnp no)
 		(fields_autoplaced yes)
-		(property "Reference" "H5"
+		(property "Reference" "H10"
 			(at 156.21 223.5199 0)
 			(show_name no)
@@
 			(project "ACW_First"
 				(path "/f90a1fa2-4579-4163-be1b-3b1c72ac9515"
-					(reference "H5")
+					(reference "H10")
 					(unit 1)
 				)
@@
 		(dnp no)
 		(fields_autoplaced yes)
-		(property "Reference" "J5"
+		(property "Reference" "J11"
 			(at 73.025 222.25 0)
 			(show_name no)
@@
 			(project "ACW_First"
 				(path "/f90a1fa2-4579-4163-be1b-3b1c72ac9515"
-					(reference "J5")
+					(reference "J11")
 					(unit 1)
 				)
@@
 		(in_pos_files yes)
 		(dnp no)
-		(property "Reference" "J4"
+		(property "Reference" "J10"
 			(at 67.564 193.548 0)
 			(show_name no)
@@
 			(project "ACW_First"
 				(path "/f90a1fa2-4579-4163-be1b-3b1c72ac9515"
-					(reference "J4")
+					(reference "J10")
 					(unit 1)
 				)
@@
 		(dnp no)
 		(fields_autoplaced yes)
-		(property "Reference" "H8"
+		(property "Reference" "H11"
 			(at 156.21 238.7599 0)
 			(show_name no)
@@
 			(project "ACW_First"
 				(path "/f90a1fa2-4579-4163-be1b-3b1c72ac9515"
-					(reference "H8")
+					(reference "H11")
 					(unit 1)
 				)
@@
 		(dnp no)
 		(fields_autoplaced yes)
-		(property "Reference" "H4"
+		(property "Reference" "H7"
 			(at 127 237.4899 0)
 			(show_name no)
@@
 			(project "ACW_First"
 				(path "/f90a1fa2-4579-4163-be1b-3b1c72ac9515"
-					(reference "H4")
+					(reference "H7")
 					(unit 1)
 				)
@@
 		(dnp no)
 		(fields_autoplaced yes)
-		(property "Reference" "H6"
+		(property "Reference" "H12"
 			(at 156.21 228.5999 0)
 			(show_name no)
@@
 			(project "ACW_First"
 				(path "/f90a1fa2-4579-4163-be1b-3b1c72ac9515"
-					(reference "H6")
+					(reference "H12")
 					(unit 1)
 				)
@@
 		(in_pos_files yes)
 		(dnp no)
-		(property "Reference" "J6"
+		(property "Reference" "J4"
 			(at 99.314 27.686 90)
 			(show_name no)
@@
 			(project "ACW_First"
 				(path "/f90a1fa2-4579-4163-be1b-3b1c72ac9515"
-					(reference "J6")
+					(reference "J4")
 					(unit 1)
 				)
@@
 		(in_pos_files yes)
 		(dnp no)
-		(property "Reference" "J8"
+		(property "Reference" "J5"
 			(at 143.256 41.656 90)
 			(show_name no)
@@
 			(project "ACW_First"
 				(path "/f90a1fa2-4579-4163-be1b-3b1c72ac9515"
-					(reference "J8")
+					(reference "J5")
 					(unit 1)
 				)
@@
 		(dnp no)
 		(fields_autoplaced yes)
-		(property "Reference" "J1"
+		(property "Reference" "J3"
 			(at 17.145 45.72 0)
 			(show_name no)
@@
 			(project "ACW_First"
 				(path "/f90a1fa2-4579-4163-be1b-3b1c72ac9515"
-					(reference "J1")
+					(reference "J3")
 					(unit 1)
 				)
@@
 		(dnp no)
 		(fields_autoplaced yes)
-		(property "Reference" "H3"
+		(property "Reference" "H1"
 			(at 127 232.4099 0)
 			(show_name no)
@@
 			(project "ACW_First"
 				(path "/f90a1fa2-4579-4163-be1b-3b1c72ac9515"
-					(reference "H3")
+					(reference "H1")
 					(unit 1)
 				)
@@
 		(dnp no)
 		(fields_autoplaced yes)
-		(property "Reference" "H2"
+		(property "Reference" "H8"
 			(at 127 227.3299 0)
 			(show_name no)
@@
 			(project "ACW_First"
 				(path "/f90a1fa2-4579-4163-be1b-3b1c72ac9515"
-					(reference "H2")
+					(reference "H8")
 					(unit 1)
 				)
@@
 		(dnp no)
 		(fields_autoplaced yes)
-		(property "Reference" "J3"
+		(property "Reference" "J1"
 			(at 40.64 196.8501 0)
 			(show_name no)
@@
 			(project "ACW_First"
 				(path "/f90a1fa2-4579-4163-be1b-3b1c72ac9515"
-					(reference "J3")
+					(reference "J1")
 					(unit 1)
 				)
@@
 		(dnp no)
 		(fields_autoplaced yes)
-		(property "Reference" "J7"
+		(property "Reference" "J2"
 			(at 105.41 154.9399 0)
 			(show_name no)
@@
 			(project "ACW_First"
 				(path "/f90a1fa2-4579-4163-be1b-3b1c72ac9515"
-					(reference "J7")
-					(unit 1)
-				)
+					(reference "J2")
+					(unit 1)
+				)
