File: ACW_First/Controller.kicad_sch (KiCad schematic)
At the start: 35 parts, among them J101 Conn_01x02_Male, J102 Conn_STLink, SW101 SW_Push, SW102 SW_Push, U101 A7600_Pinout, U102 STM32F401CCUx, U103 AMS1117-3.3, Y101 8Mhz

Commit message: okok
Parts:
- added H101, H102, H103, H104: MountingHole, symbol Mechanical:MountingHole
- C101, C102, C103, C104, C105, C106, C107, C108, C109, C110, D101, D102, R101, R102, R103, R104, R105, R106, R107, R108, R109, R110, R111, R112, R113, R114, R115: KiLib_Generator (none) -> SMD_2terminal_chip_molded
- J101: KiLib_Generator (none) -> terminal_block/Metz_Connect
- J102: footprint Connector_JST:JST_XH_S4B-XH-A_1x04_P2.50mm_Horizontal -> Connector_JST:JST_XH_B4B-XH-A_1x04_P2.50mm_Vertical; KiLib_Generator (none) -> connector/JST
- U101: KiLib_Generator (none) -> connector/pin_header_socket
- U102: KiLib_Generator (none) -> package/no_lead
- Y101: KiLib_Generator (none) -> crystal_resonator_oscillator
Connections:
- net +5V renamed 5VDC
- net 3.8V renamed 3.8VDC
Other:
- sheet Connector_Sheet ports: added none; removed 12V, 3.8V, 5V, PZEM_RXD, PZEM_TXD, RELAY_DATA_PIN

Commit message: okok
Connections:
- net AGND is gone; now on net GND: U102.8 (VSSA)
- no-connect marks 1 -> 19
Changed lines of the file:
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@@
 	)
 	(junction
+		(at 146.05 147.32)
+		(diameter 0)
+		(color 0 0 0 0)
+	)
+	(junction
 		(at 228.6 31.75)
 		(diameter 0)
@@
 	)
 	(no_connect
+		(at 125.73 124.46)
+	)
+	(no_connect
+		(at 125.73 88.9)
+	)
+	(no_connect
+		(at 125.73 116.84)
+	)
+	(no_connect
+		(at 125.73 127)
+	)
+	(no_connect
 		(at 138.43 55.88)
 	)
+	(no_connect
+		(at 158.75 132.08)
+	)
+	(no_connect
+		(at 125.73 119.38)
+	)
+	(no_connect
+		(at 158.75 114.3)
+	)
+	(no_connect
+		(at 125.73 101.6)
+	)
+	(no_connect
+		(at 125.73 109.22)
+	)
+	(no_connect
+		(at 125.73 91.44)
+	)
+	(no_connect
+		(at 125.73 106.68)
+	)
+	(no_connect
+		(at 158.75 93.98)
+	)
+	(no_connect
+		(at 158.75 96.52)
+	)
+	(no_connect
+		(at 125.73 99.06)
+	)
+	(no_connect
+		(at 125.73 104.14)
+	)
+	(no_connect
+		(at 125.73 96.52)
+	)
+	(no_connect
+		(at 125.73 121.92)
+	)
+	(no_connect
+		(at 158.75 111.76)
+	)
 	(wire
 		(pts
@@
 	(wire
 		(pts
+			(xy 146.05 147.32) (xy 148.59 147.32)
+		)
+		(stroke
+			(width 0)
+			(type default)
+		)
+	)
+	(wire
+		(pts
 			(xy 158.75 104.14) (xy 171.45 104.14)
 		)
@@
 					(unit 1)
 				)
-			)
-		)
-	)
-	(symbol
-		(lib_id "power:GND")
-		(at 148.59 147.32 0)
-		(unit 1)
-		(body_style 1)
-		(exclude_from_sim no)
-		(in_bom yes)
-		(on_board yes)
-		(in_pos_files yes)
-		(dnp no)
-		(fields_autoplaced yes)
-		(property "Reference" "#PWR0112"
-			(at 148.59 153.67 0)
-			(hide yes)
-			(show_name no)
-			(do_not_autoplace no)
-			(effects
-				(font
-					(size 1.27 1.27)
-				)
-			)
-		)
-		(property "Value" "AGND"
-			(at 148.59 152.4 0)
-			(show_name no)
-			(do_not_autoplace no)
-			(effects
-				(font
-					(size 1.27 1.27)
-				)
-			)
-		)
-		(property "Footprint" ""
-			(at 148.59 147.32 0)
-			(hide yes)
-			(show_name no)
-			(do_not_autoplace no)
-			(effects
-				(font
-					(size 1.27 1.27)
-				)
-			)
-		)
-		(property "Datasheet" ""
-			(at 148.59 147.32 0)
-			(hide yes)
-			(show_name no)
-			(do_not_autoplace no)
-			(effects
-				(font
-					(size 1.27 1.27)
-				)
-			)
-		)
-		(property "Description" ""
-			(at 148.59 147.32 0)
-			(show_name no)
-			(do_not_autoplace no)
-			(effects
-				(font
-					(size 1.27 1.27)
-				)
-			)
-		)
-		(pin "1"
-		)
-		(instances
-			(project "ACW_First"
-				(path "/f90a1fa2-4579-4163-be1b-3b1c72ac9515/b1ee6347-5b28-490c-a137-9ca76f07a51b"
-					(reference "#PWR0112")
-					(unit 1)
-				)

Commit message: fix
Parts:
- renumbered C109 to C10, C110 to C11, C101 to C2, C102 to C3, C103 to C4, C104 to C5, C105 to C6, C106 to C7, C107 to C8, C108 to C9, D101 to D2, D102 to D3, H102 to H10, H103 to H11, H104 to H12, H101 to H9, J102 to J10, J101 to J9, R106 to R10, R107 to R11, R108 to R12, R109 to R13, R110 to R14, R111 to R15, R112 to R16, R113 to R17, R114 to R18, R115 to R19, R101 to R5, R102 to R6, R103 to R7, R104 to R8, R105 to R9, SW101 to SW1, SW102 to SW2, U101 to U2, U102 to U3, U103 to U4, Y101 to Y1

Commit message: okok
Parts:
- removed J10: Conn_STLink, Connector_JST:JST_XH_B4B-XH-A_1x04_P2.50mm_Vertical, symbol Connector:Conn_01x04_Male
- added J6: Conn_01x03_Pin, Connector_JST:JST_XH_B3B-XH-A_1x03_P2.50mm_Vertical, symbol Connector:Conn_01x03_Pin
- renumbered C9 to C11, C2 to C19, C3 to C20, C11 to C50, C6 to C51, C5 to C52, C10 to C55, C4 to C56, C8 to C6, D2 to D6, D3 to D7, H9 to H2, H11 to H4, H12 to H5, H10 to H6, J9 to J8, R16 to R10, R11 to R13, R12 to R14, R6 to R15, R5 to R16, R18 to R20, R9 to R28, R10 to R29, R13 to R30, R14 to R31, R17 to R52, R7 to R58, R8 to R59, R15 to R7, SW2 to SW1, SW1 to SW2, U3 to U1, U2 to U5, U4 to U6
Connections:
- net GND: now also J6.1 (Pin_1)
- net SWCLK: now also J6.2 (Pin_2)
- net SWDIO: now also J6.3 (Pin_3)
