File: ACW_First/Dimm_Circuit.kicad_sch (KiCad schematic)
At the start: 11 parts, among them U107 PC817, U108 LM358PSR

Commit message: okok
Connections:
- net GND: no longer PS101.2 (-VIN)
- net +12V renamed 12VDC
- new net -12VDC: PS101.2 (-VIN)
Changed lines of the file:
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@@
+		)
+	)
+	(global_label "-12VDC"
+		(shape input)
+		(at 67.31 64.77 270)
+		(fields_autoplaced yes)
+		(effects
+			(font
+				(size 1.27 1.27)
+			)
+			(justify right)
+		)
+		(property "Intersheetrefs" "${INTERSHEET_REFS}"
+			(at 67.31 75.3752 90)
+			(hide yes)
+			(show_name no)
+			(do_not_autoplace no)
+			(effects
+				(font
+					(size 1.27 1.27)
+				)
+				(justify right)
+			)
+		)
+	)
+	(global_label "12VDC"
+		(shape input)
+		(at 66.04 45.72 180)
+		(fields_autoplaced yes)
+		(effects
+			(font
+				(size 1.27 1.27)
+			)
+			(justify right)
+		)
+		(property "Intersheetrefs" "${INTERSHEET_REFS}"
+			(at 57.0072 45.72 0)
+			(hide yes)
+			(show_name no)
+			(do_not_autoplace no)
+			(effects
+				(font
+					(size 1.27 1.27)
+				)
+				(justify right)
+			)
 		)
 	)
@@
 		(instances
 			(project "ACW_First"
-				(path "/f90a1fa2-4579-4163-be1b-3b1c72ac9515/b1ee6347-5b28-490c-a137-9ca76f07a51b/b1b93fb9-9075-42e9-b467-1451a7a42c90"
+				(path "/f90a1fa2-4579-4163-be1b-3b1c72ac9515/b1ee6347-5b28-490c-a137-9ca76f07a51b/ed3cf17e-89b7-4b35-8f01-664318c40924"
 					(reference "R128")
 					(unit 1)
@@
 		(instances
 			(project "ACW_First"
-				(path "/f90a1fa2-4579-4163-be1b-3b1c72ac9515/b1ee6347-5b28-490c-a137-9ca76f07a51b/b1b93fb9-9075-42e9-b467-1451a7a42c90"
+				(path "/f90a1fa2-4579-4163-be1b-3b1c72ac9515/b1ee6347-5b28-490c-a137-9ca76f07a51b/ed3cf17e-89b7-4b35-8f01-664318c40924"
 					(reference "#PWR0148")
 					(unit 1)
@@
 		(instances
 			(project "ACW_First"
-				(path "/f90a1fa2-4579-4163-be1b-3b1c72ac9515/b1ee6347-5b28-490c-a137-9ca76f07a51b/b1b93fb9-9075-42e9-b467-1451a7a42c90"
+				(path "/f90a1fa2-4579-4163-be1b-3b1c72ac9515/b1ee6347-5b28-490c-a137-9ca76f07a51b/ed3cf17e-89b7-4b35-8f01-664318c40924"
 					(reference "#PWR0147")
 					(unit 1)
@@
 		(instances
 			(project "ACW_First"
-				(path "/f90a1fa2-4579-4163-be1b-3b1c72ac9515/b1ee6347-5b28-490c-a137-9ca76f07a51b/b1b93fb9-9075-42e9-b467-1451a7a42c90"
+				(path "/f90a1fa2-4579-4163-be1b-3b1c72ac9515/b1ee6347-5b28-490c-a137-9ca76f07a51b/ed3cf17e-89b7-4b35-8f01-664318c40924"
 					(reference "U108")
 					(unit 1)
@@
 		(instances
 			(project "ACW_First"
-				(path "/f90a1fa2-4579-4163-be1b-3b1c72ac9515/b1ee6347-5b28-490c-a137-9ca76f07a51b/b1b93fb9-9075-42e9-b467-1451a7a42c90"
+				(path "/f90a1fa2-4579-4163-be1b-3b1c72ac9515/b1ee6347-5b28-490c-a137-9ca76f07a51b/ed3cf17e-89b7-4b35-8f01-664318c40924"
 					(reference "#PWR0150")
 					(unit 1)
@@
 		(instances
 			(project "ACW_First"
-				(path "/f90a1fa2-4579-4163-be1b-3b1c72ac9515/b1ee6347-5b28-490c-a137-9ca76f07a51b/b1b93fb9-9075-42e9-b467-1451a7a42c90"
+				(path "/f90a1fa2-4579-4163-be1b-3b1c72ac9515/b1ee6347-5b28-490c-a137-9ca76f07a51b/ed3cf17e-89b7-4b35-8f01-664318c40924"
 					(reference "C115")
 					(unit 1)
@@
 		(instances
 			(project "ACW_First"
-				(path "/f90a1fa2-4579-4163-be1b-3b1c72ac9515/b1ee6347-5b28-490c-a137-9ca76f07a51b/b1b93fb9-9075-42e9-b467-1451a7a42c90"
+				(path "/f90a1fa2-4579-4163-be1b-3b1c72ac9515/b1ee6347-5b28-490c-a137-9ca76f07a51b/ed3cf17e-89b7-4b35-8f01-664318c40924"
 					(reference "PS101")
 					(unit 1)
@@
 		(instances
 			(project "ACW_First"
-				(path "/f90a1fa2-4579-4163-be1b-3b1c72ac9515/b1ee6347-5b28-490c-a137-9ca76f07a51b/b1b93fb9-9075-42e9-b467-1451a7a42c90"
+				(path "/f90a1fa2-4579-4163-be1b-3b1c72ac9515/b1ee6347-5b28-490c-a137-9ca76f07a51b/ed3cf17e-89b7-4b35-8f01-664318c40924"
 					(reference "R126")
-					(unit 1)
-				)
-			)
-		)
-	)
-	(symbol
-		(lib_id "power:GND")
-		(at 67.31 64.77 0)
-		(unit 1)
-		(body_style 1)
-		(exclude_from_sim no)
-		(in_bom yes)
-		(on_board yes)
-		(in_pos_files yes)
-		(dnp no)
-		(fields_autoplaced yes)
-		(property "Reference" "#PWR0141"
-			(at 67.31 71.12 0)
-			(hide yes)
-			(show_name no)
-			(do_not_autoplace no)
-			(effects
-				(font
-					(size 1.27 1.27)
-				)
-			)
-		)
-		(property "Value" "GND"
-			(at 67.31 69.85 0)
-			(show_name no)
-			(do_not_autoplace no)
-			(effects
-				(font
-					(size 1.27 1.27)
-				)
-			)
-		)
-		(property "Footprint" ""
-			(at 67.31 64.77 0)
-			(hide yes)
-			(show_name no)
-			(do_not_autoplace no)
-			(effects
-				(font
-					(size 1.27 1.27)
-				)
-			)
-		)
-		(property "Datasheet" ""
-			(at 67.31 64.77 0)
-			(hide yes)
-			(show_name no)
-			(do_not_autoplace no)
-			(effects
-				(font
-					(size 1.27 1.27)
-				)
-			)
-		)
-		(property "Description" ""
-			(at 67.31 64.77 0)
-			(show_name no)
-			(do_not_autoplace no)
-			(effects
-				(font
-					(size 1.27 1.27)
-				)
-			)
-		)
-		(pin "1"
-		)
-		(instances
-			(project "ACW_First"
-				(path "/f90a1fa2-4579-4163-be1b-3b1c72ac9515/b1ee6347-5b28-490c-a137-9ca76f07a51b/b1b93fb9-9075-42e9-b467-1451a7a42c90"
-					(reference "#PWR0141")
 					(unit 1)
 				)
@@
 		(instances
 			(project "ACW_First"
-				(path "/f90a1fa2-4579-4163-be1b-3b1c72ac9515/b1ee6347-5b28-490c-a137-9ca76f07a51b/b1b93fb9-9075-42e9-b467-1451a7a42c90"
+				(path "/f90a1fa2-4579-4163-be1b-3b1c72ac9515/b1ee6347-5b28-490c-a137-9ca76f07a51b/ed3cf17e-89b7-4b35-8f01-664318c40924"
 					(reference "U107")
 					(unit 1)
@@
 		(instances
 			(project "ACW_First"
-				(path "/f90a1fa2-4579-4163-be1b-3b1c72ac9515/b1ee6347-5b28-490c-a137-9ca76f07a51b/b1b93fb9-9075-42e9-b467-1451a7a42c90"
+				(path "/f90a1fa2-4579-4163-be1b-3b1c72ac9515/b1ee6347-5b28-490c-a137-9ca76f07a51b/ed3cf17e-89b7-4b35-8f01-664318c40924"
 					(reference "#PWR0149")
 					(unit 1)
@@
 		(instances
 			(project "ACW_First"
-				(path "/f90a1fa2-4579-4163-be1b-3b1c72ac9515/b1ee6347-5b28-490c-a137-9ca76f07a51b/b1b93fb9-9075-42e9-b467-1451a7a42c90"
+				(path "/f90a1fa2-4579-4163-be1b-3b1c72ac9515/b1ee6347-5b28-490c-a137-9ca76f07a51b/ed3cf17e-89b7-4b35-8f01-664318c40924"
 					(reference "R125")
 					(unit 1)
@@
 		(instances
 			(project "ACW_First"
-				(path "/f90a1fa2-4579-4163-be1b-3b1c72ac9515/b1ee6347-5b28-490c-a137-9ca76f07a51b/b1b93fb9-9075-42e9-b467-1451a7a42c90"
+				(path "/f90a1fa2-4579-4163-be1b-3b1c72ac9515/b1ee6347-5b28-490c-a137-9ca76f07a51b/ed3cf17e-89b7-4b35-8f01-664318c40924"
 					(reference "C116")
 					(unit 1)
@@
 		(instances
 			(project "ACW_First"
-				(path "/f90a1fa2-4579-4163-be1b-3b1c72ac9515/b1ee6347-5b28-490c-a137-9ca76f07a51b/b1b93fb9-9075-42e9-b467-1451a7a42c90"
+				(path "/f90a1fa2-4579-4163-be1b-3b1c72ac9515/b1ee6347-5b28-490c-a137-9ca76f07a51b/ed3cf17e-89b7-4b35-8f01-664318c40924"
 					(reference "R124")
 					(unit 1)
@@
 		(instances
 			(project "ACW_First"
-				(path "/f90a1fa2-4579-4163-be1b-3b1c72ac9515/b1ee6347-5b28-490c-a137-9ca76f07a51b/b1b93fb9-9075-42e9-b467-1451a7a42c90"
+				(path "/f90a1fa2-4579-4163-be1b-3b1c72ac9515/b1ee6347-5b28-490c-a137-9ca76f07a51b/ed3cf17e-89b7-4b35-8f01-664318c40924"
 					(reference "R127")
 					(unit 1)
@@
 		(instances
 			(project "ACW_First"
-				(path "/f90a1fa2-4579-4163-be1b-3b1c72ac9515/b1ee6347-5b28-490c-a137-9ca76f07a51b/b1b93fb9-9075-42e9-b467-1451a7a42c90"
+				(path "/f90a1fa2-4579-4163-be1b-3b1c72ac9515/b1ee6347-5b28-490c-a137-9ca76f07a51b/ed3cf17e-89b7-4b35-8f01-664318c40924"
 					(reference "R129")
-					(unit 1)
-				)
-			)
-		)
-	)
-	(symbol
-		(lib_id "power:+12V")
-		(at 66.04 45.72 90)
-		(unit 1)
-		(body_style 1)
-		(exclude_from_sim no)
-		(in_bom yes)
-		(on_board yes)
-		(in_pos_files yes)
-		(dnp no)
-		(fields_autoplaced yes)
-		(property "Reference" "#PWR0140"
-			(at 69.85 45.72 0)
-			(hide yes)
-			(show_name no)
-			(do_not_autoplace no)
-			(effects
-				(font
-					(size 1.27 1.27)
-				)
-			)
-		)
-		(property "Value" "+12V"
-			(at 62.23 45.7199 90)
-			(show_name no)
-			(do_not_autoplace no)
-			(effects
-				(font
-					(size 1.27 1.27)
-				)
-				(justify left)
-			)
-		)
-		(property "Footprint" ""
-			(at 66.04 45.72 0)
-			(hide yes)
-			(show_name no)
-			(do_not_autoplace no)
-			(effects
-				(font
-					(size 1.27 1.27)
-				)
-			)
-		)
-		(property "Datasheet" ""
-			(at 66.04 45.72 0)
-			(hide yes)
-			(show_name no)
-			(do_not_autoplace no)
-			(effects
-				(font
-					(size 1.27 1.27)
-				)
-			)
-		)
-		(property "Description" "Power symbol creates a global label with name \"+12V\""
-			(at 66.04 45.72 0)
-			(hide yes)
-			(show_name no)
-			(do_not_autoplace no)
-			(effects
-				(font
-					(size 1.27 1.27)
-				)
-			)
-		)
-		(pin "1"
-		)
-		(instances
-			(project "ACW_First"
-				(path "/f90a1fa2-4579-4163-be1b-3b1c72ac9515/b1ee6347-5b28-490c-a137-9ca76f07a51b/b1b93fb9-9075-42e9-b467-1451a7a42c90"
-					(reference "#PWR0140")
 					(unit 1)
 				)
@@
 		(instances
 			(project "ACW_First"
-				(path "/f90a1fa2-4579-4163-be1b-3b1c72ac9515/b1ee6347-5b28-490c-a137-9ca76f07a51b/b1b93fb9-9075-42e9-b467-1451a7a42c90"
+				(path "/f90a1fa2-4579-4163-be1b-3b1c72ac9515/b1ee6347-5b28-490c-a137-9ca76f07a51b/ed3cf17e-89b7-4b35-8f01-664318c40924"
 					(reference "#PWR0151")
 					(unit 1)

Commit message: okok
Connections:
- net -12VDC is gone; now on net GND: PS101.2 (-VIN)
Changed lines of the file:
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@@
-	(wire
-		(pts
-			(xy 67.31 64.77) (xy 67.31 55.88)
-		)
-		(stroke
-			(width 0)
-			(type default)
-		)
-	)
 	(wire
 		(pts
@@
 	(wire
 		(pts
+			(xy 66.04 55.88) (xy 72.39 55.88)
+		)
+		(stroke
+			(width 0)
+			(type default)
+		)
+	)
+	(wire
+		(pts
 			(xy 105.41 95.25) (xy 115.57 95.25)
 		)
@@
 	(wire
 		(pts
-			(xy 67.31 55.88) (xy 72.39 55.88)
-		)
-		(stroke
-			(width 0)
-			(type default)
-		)
-	)
-	(wire
-		(pts
 			(xy 66.04 45.72) (xy 72.39 45.72)
 		)
@@
 	(wire
 		(pts
+			(xy 66.04 62.23) (xy 66.04 55.88)
+		)
+		(stroke
+			(width 0)
+			(type default)
+		)
+	)
+	(wire
+		(pts
 			(xy 140.97 95.25) (xy 147.32 95.25)
 		)
@@
 			(width 0)
 			(type default)
-		)
-	)
-	(global_label "-12VDC"
-		(shape input)
-		(at 67.31 64.77 270)
-		(fields_autoplaced yes)
-		(effects
-			(font
-				(size 1.27 1.27)
-			)
-			(justify right)
-		)
-		(property "Intersheetrefs" "${INTERSHEET_REFS}"
-			(at 67.31 75.3752 90)
-			(hide yes)
-			(show_name no)
-			(do_not_autoplace no)
-			(effects
-				(font
-					(size 1.27 1.27)
-				)
-				(justify right)
-			)
 		)
 	)
@@
 					(unit 1)
 				)
+			)
+		)
+	)
+	(symbol
+		(lib_name "GND_2")
+		(lib_id "power:GND")
+		(at 66.04 62.23 0)
+		(unit 1)
+		(body_style 1)
+		(exclude_from_sim no)
+		(in_bom yes)
+		(on_board yes)
+		(in_pos_files yes)
+		(dnp no)
+		(fields_autoplaced yes)
+		(property "Reference" "#PWR010"
+			(at 66.04 68.58 0)
+			(hide yes)
+			(show_name no)
+			(do_not_autoplace no)
+			(effects
+				(font
+					(size 1.27 1.27)
+				)
+			)
+		)
+		(property "Value" "GND"
+			(at 66.04 67.31 0)
+			(show_name no)
+			(do_not_autoplace no)
+			(effects
+				(font
+					(size 1.27 1.27)
+				)
+			)
+		)
+		(property "Footprint" ""
+			(at 66.04 62.23 0)
+			(hide yes)
+			(show_name no)
+			(do_not_autoplace no)
+			(effects
+				(font
+					(size 1.27 1.27)
+				)
+			)
+		)
+		(property "Datasheet" ""
+			(at 66.04 62.23 0)
+			(hide yes)
+			(show_name no)
+			(do_not_autoplace no)
+			(effects
+				(font
+					(size 1.27 1.27)
+				)
+			)
+		)
+		(property "Description" "Power symbol creates a global label with name \"GND\" , ground"
+			(at 66.04 62.23 0)
+			(hide yes)
+			(show_name no)
+			(do_not_autoplace no)
+			(effects
+				(font
+					(size 1.27 1.27)
+				)
+			)
+		)
+		(pin "1"
+		)
+		(instances
+			(project "ACW_First"
+				(path "/f90a1fa2-4579-4163-be1b-3b1c72ac9515/b1ee6347-5b28-490c-a137-9ca76f07a51b/ed3cf17e-89b7-4b35-8f01-664318c40924"
+					(reference "#PWR010")
+					(unit 1)
+				)

Commit message: fix
Parts:
- renumbered C115 to C12, C116 to C13, PS101 to PS1, R124 to R20, R125 to R21, R126 to R22, R127 to R23, R128 to R24, R129 to R25, U107 to U5, U108 to U6
Changed lines of the file:
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@@
 		(dnp no)
 		(fields_autoplaced yes)
-		(property "Reference" "R128"
+		(property "Reference" "R24"
 			(at 151.13 88.9 90)
 			(show_name no)
@@
 			(project "ACW_First"
 				(path "/f90a1fa2-4579-4163-be1b-3b1c72ac9515/b1ee6347-5b28-490c-a137-9ca76f07a51b/ed3cf17e-89b7-4b35-8f01-664318c40924"
-					(reference "R128")
+					(reference "R24")
 					(unit 1)
 				)
@@
 		(dnp no)
 		(fields_autoplaced yes)
-		(property "Reference" "#PWR0148"
+		(property "Reference" "#PWR033"
 			(at 106.68 69.85 0)
 			(hide yes)
@@
 			(project "ACW_First"
 				(path "/f90a1fa2-4579-4163-be1b-3b1c72ac9515/b1ee6347-5b28-490c-a137-9ca76f07a51b/ed3cf17e-89b7-4b35-8f01-664318c40924"
-					(reference "#PWR0148")
+					(reference "#PWR033")
 					(unit 1)
 				)
@@
 		(dnp no)
 		(fields_autoplaced yes)
-		(property "Reference" "#PWR0147"
+		(property "Reference" "#PWR032"
 			(at 85.09 105.41 0)
 			(hide yes)
@@
 			(project "ACW_First"
 				(path "/f90a1fa2-4579-4163-be1b-3b1c72ac9515/b1ee6347-5b28-490c-a137-9ca76f07a51b/ed3cf17e-89b7-4b35-8f01-664318c40924"
-					(reference "#PWR0147")
+					(reference "#PWR032")
 					(unit 1)
 				)
@@
 		(dnp no)
 		(fields_autoplaced yes)
-		(property "Reference" "U108"
+		(property "Reference" "U6"
 			(at 199.39 82.55 0)
 			(show_name no)
@@
 			(project "ACW_First"
 				(path "/f90a1fa2-4579-4163-be1b-3b1c72ac9515/b1ee6347-5b28-490c-a137-9ca76f07a51b/ed3cf17e-89b7-4b35-8f01-664318c40924"
-					(reference "U108")
+					(reference "U6")
 					(unit 1)
 				)
@@
 		(dnp no)
 		(fields_autoplaced yes)
-		(property "Reference" "#PWR0150"
+		(property "Reference" "#PWR035"
 			(at 166.37 160.02 0)
 			(hide yes)
@@
 			(project "ACW_First"
 				(path "/f90a1fa2-4579-4163-be1b-3b1c72ac9515/b1ee6347-5b28-490c-a137-9ca76f07a51b/ed3cf17e-89b7-4b35-8f01-664318c40924"
-					(reference "#PWR0150")
+					(reference "#PWR035")
 					(unit 1)
 				)
@@
 		(dnp no)
 		(fields_autoplaced yes)
-		(property "Reference" "C115"
+		(property "Reference" "C12"
 			(at 170.18 147.3199 0)
 			(show_name no)
@@
 			(project "ACW_First"
 				(path "/f90a1fa2-4579-4163-be1b-3b1c72ac9515/b1ee6347-5b28-490c-a137-9ca76f07a51b/ed3cf17e-89b7-4b35-8f01-664318c40924"
-					(reference "C115")
+					(reference "C12")
 					(unit 1)
 				)
@@
 		(dnp no)
 		(fields_autoplaced yes)
-		(property "Reference" "#PWR010"
+		(property "Reference" "#PWR031"
 			(at 66.04 68.58 0)
 			(hide yes)
@@
 			(project "ACW_First"
 				(path "/f90a1fa2-4579-4163-be1b-3b1c72ac9515/b1ee6347-5b28-490c-a137-9ca76f07a51b/ed3cf17e-89b7-4b35-8f01-664318c40924"
-					(reference "#PWR010")
+					(reference "#PWR031")
 					(unit 1)
 				)
@@
 		(dnp no)
 		(fields_autoplaced yes)
-		(property "Reference" "PS101"
+		(property "Reference" "PS1"
 			(at 87.63 39.37 0)
 			(show_name no)
@@
 			(project "ACW_First"
 				(path "/f90a1fa2-4579-4163-be1b-3b1c72ac9515/b1ee6347-5b28-490c-a137-9ca76f07a51b/ed3cf17e-89b7-4b35-8f01-664318c40924"
-					(reference "PS101")
+					(reference "PS1")
 					(unit 1)
 				)
@@
 		(dnp no)
 		(fields_autoplaced yes)
-		(property "Reference" "R126"
+		(property "Reference" "R22"
 			(at 118.11 106.6799 0)
 			(show_name no)
@@
 			(project "ACW_First"
 				(path "/f90a1fa2-4579-4163-be1b-3b1c72ac9515/b1ee6347-5b28-490c-a137-9ca76f07a51b/ed3cf17e-89b7-4b35-8f01-664318c40924"
-					(reference "R126")
+					(reference "R22")
 					(unit 1)
 				)
@@
 		(dnp no)
 		(fields_autoplaced yes)
-		(property "Reference" "U107"
+		(property "Reference" "U5"
 			(at 97.79 83.82 0)
 			(show_name no)
@@
 			(project "ACW_First"
 				(path "/f90a1fa2-4579-4163-be1b-3b1c72ac9515/b1ee6347-5b28-490c-a137-9ca76f07a51b/ed3cf17e-89b7-4b35-8f01-664318c40924"
-					(reference "U107")
+					(reference "U5")
 					(unit 1)
 				)
@@
 		(dnp no)
 		(fields_autoplaced yes)
-		(property "Reference" "#PWR0149"
+		(property "Reference" "#PWR034"
 			(at 115.57 121.92 0)
 			(hide yes)
@@
 			(project "ACW_First"
 				(path "/f90a1fa2-4579-4163-be1b-3b1c72ac9515/b1ee6347-5b28-490c-a137-9ca76f07a51b/ed3cf17e-89b7-4b35-8f01-664318c40924"
-					(reference "#PWR0149")
+					(reference "#PWR034")
 					(unit 1)
 				)
@@
 		(dnp no)
 		(fields_autoplaced yes)
-		(property "Reference" "R125"
+		(property "Reference" "R21"
 			(at 118.11 76.1999 0)
 			(show_name no)
@@
 			(project "ACW_First"
 				(path "/f90a1fa2-4579-4163-be1b-3b1c72ac9515/b1ee6347-5b28-490c-a137-9ca76f07a51b/ed3cf17e-89b7-4b35-8f01-664318c40924"
-					(reference "R125")
+					(reference "R21")
 					(unit 1)
 				)
@@
 		(in_pos_files yes)
 		(dnp no)
-		(property "Reference" "C116"
+		(property "Reference" "C13"
 			(at 186.69 135.89 90)
 			(show_name no)
@@
 			(project "ACW_First"
 				(path "/f90a1fa2-4579-4163-be1b-3b1c72ac9515/b1ee6347-5b28-490c-a137-9ca76f07a51b/ed3cf17e-89b7-4b35-8f01-664318c40924"
-					(reference "C116")
+					(reference "C13")
 					(unit 1)
 				)
@@
 		(dnp no)
 		(fields_autoplaced yes)
-		(property "Reference" "R124"
+		(property "Reference" "R20"
 			(at 72.39 83.82 90)
 			(show_name no)
@@
 			(project "ACW_First"
 				(path "/f90a1fa2-4579-4163-be1b-3b1c72ac9515/b1ee6347-5b28-490c-a137-9ca76f07a51b/ed3cf17e-89b7-4b35-8f01-664318c40924"
-					(reference "R124")
+					(reference "R20")
 					(unit 1)
 				)
@@
 		(dnp no)
 		(fields_autoplaced yes)
-		(property "Reference" "R127"
+		(property "Reference" "R23"
 			(at 137.16 88.9 90)
 			(show_name no)
@@
 			(project "ACW_First"
 				(path "/f90a1fa2-4579-4163-be1b-3b1c72ac9515/b1ee6347-5b28-490c-a137-9ca76f07a51b/ed3cf17e-89b7-4b35-8f01-664318c40924"
-					(reference "R127")
+					(reference "R23")
 					(unit 1)
 				)
@@
 		(in_pos_files yes)
 		(dnp no)
-		(property "Reference" "R129"
+		(property "Reference" "R25"
 			(at 237.49 120.6499 0)
 			(show_name no)
@@
 			(project "ACW_First"
 				(path "/f90a1fa2-4579-4163-be1b-3b1c72ac9515/b1ee6347-5b28-490c-a137-9ca76f07a51b/ed3cf17e-89b7-4b35-8f01-664318c40924"
-					(reference "R129")
+					(reference "R25")
 					(unit 1)
 				)
@@
 		(dnp no)
 		(fields_autoplaced yes)
-		(property "Reference" "#PWR0151"
+		(property "Reference" "#PWR036"
 			(at 234.95 147.32 0)
 			(hide yes)
@@
 			(project "ACW_First"
 				(path "/f90a1fa2-4579-4163-be1b-3b1c72ac9515/b1ee6347-5b28-490c-a137-9ca76f07a51b/ed3cf17e-89b7-4b35-8f01-664318c40924"
-					(reference "#PWR0151")
-					(unit 1)
-				)
+					(reference "#PWR036")
+					(unit 1)
+				)

Commit message: okok
Parts:
- U15: renamed from U5; footprint Custom_Library:SOP254P975X460-4N -> Custom_Footprints:SOP-4_L6.4-W4.6-P2.54-LS10.2-TL
- renumbered C12 to C53, C13 to C54, PS1 to PS2, R20 to R62, R21 to R64, R22 to R65, R25 to R66, R23 to R67, R24 to R68, U6 to U16
Changed lines of the file:
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@@
 		(dnp no)
 		(fields_autoplaced yes)
-		(property "Reference" "R24"
+		(property "Reference" "R68"
 			(at 151.13 88.9 90)
 			(show_name no)
@@
 			(project "ACW_First"
 				(path "/f90a1fa2-4579-4163-be1b-3b1c72ac9515/b1ee6347-5b28-490c-a137-9ca76f07a51b/ed3cf17e-89b7-4b35-8f01-664318c40924"
-					(reference "R24")
+					(reference "R68")
 					(unit 1)
 				)
@@
 		(dnp no)
 		(fields_autoplaced yes)
-		(property "Reference" "U6"
+		(property "Reference" "U16"
 			(at 199.39 82.55 0)
 			(show_name no)
@@
 			(project "ACW_First"
 				(path "/f90a1fa2-4579-4163-be1b-3b1c72ac9515/b1ee6347-5b28-490c-a137-9ca76f07a51b/ed3cf17e-89b7-4b35-8f01-664318c40924"
-					(reference "U6")
+					(reference "U16")
 					(unit 1)
 				)
@@
 		(dnp no)
 		(fields_autoplaced yes)
-		(property "Reference" "C12"
+		(property "Reference" "C53"
 			(at 170.18 147.3199 0)
 			(show_name no)
@@
 			(project "ACW_First"
 				(path "/f90a1fa2-4579-4163-be1b-3b1c72ac9515/b1ee6347-5b28-490c-a137-9ca76f07a51b/ed3cf17e-89b7-4b35-8f01-664318c40924"
-					(reference "C12")
+					(reference "C53")
 					(unit 1)
 				)
@@
 		(dnp no)
 		(fields_autoplaced yes)
-		(property "Reference" "PS1"
+		(property "Reference" "PS2"
 			(at 87.63 39.37 0)
 			(show_name no)
@@
 			(project "ACW_First"
 				(path "/f90a1fa2-4579-4163-be1b-3b1c72ac9515/b1ee6347-5b28-490c-a137-9ca76f07a51b/ed3cf17e-89b7-4b35-8f01-664318c40924"
-					(reference "PS1")
+					(reference "PS2")
 					(unit 1)
 				)
@@
 		(dnp no)
 		(fields_autoplaced yes)
-		(property "Reference" "R22"
+		(property "Reference" "R65"
 			(at 118.11 106.6799 0)
 			(show_name no)
@@
 			(project "ACW_First"
 				(path "/f90a1fa2-4579-4163-be1b-3b1c72ac9515/b1ee6347-5b28-490c-a137-9ca76f07a51b/ed3cf17e-89b7-4b35-8f01-664318c40924"
-					(reference "R22")
+					(reference "R65")
 					(unit 1)
 				)
@@
 		(dnp no)
 		(fields_autoplaced yes)
-		(property "Reference" "U5"
+		(property "Reference" "U15"
 			(at 97.79 83.82 0)
 			(show_name no)
@@
 			)
 		)
-		(property "Footprint" "Custom_Library:SOP254P975X460-4N"
+		(property "Footprint" "Custom_Footprints:SOP-4_L6.4-W4.6-P2.54-LS10.2-TL"
 			(at 92.71 97.79 0)
 			(hide yes)
@@
 			(project "ACW_First"
 				(path "/f90a1fa2-4579-4163-be1b-3b1c72ac9515/b1ee6347-5b28-490c-a137-9ca76f07a51b/ed3cf17e-89b7-4b35-8f01-664318c40924"
-					(reference "U5")
+					(reference "U15")
 					(unit 1)
 				)
@@
 		(dnp no)
 		(fields_autoplaced yes)
-		(property "Reference" "R21"
+		(property "Reference" "R64"
 			(at 118.11 76.1999 0)
 			(show_name no)
@@
 			(project "ACW_First"
 				(path "/f90a1fa2-4579-4163-be1b-3b1c72ac9515/b1ee6347-5b28-490c-a137-9ca76f07a51b/ed3cf17e-89b7-4b35-8f01-664318c40924"
-					(reference "R21")
+					(reference "R64")
 					(unit 1)
 				)
@@
 		(in_pos_files yes)
 		(dnp no)
-		(property "Reference" "C13"
+		(property "Reference" "C54"
 			(at 186.69 135.89 90)
 			(show_name no)
@@
 			(project "ACW_First"
 				(path "/f90a1fa2-4579-4163-be1b-3b1c72ac9515/b1ee6347-5b28-490c-a137-9ca76f07a51b/ed3cf17e-89b7-4b35-8f01-664318c40924"
-					(reference "C13")
+					(reference "C54")
 					(unit 1)
 				)
@@
 		(dnp no)
 		(fields_autoplaced yes)
-		(property "Reference" "R20"
+		(property "Reference" "R62"
 			(at 72.39 83.82 90)
 			(show_name no)
@@
 			(project "ACW_First"
 				(path "/f90a1fa2-4579-4163-be1b-3b1c72ac9515/b1ee6347-5b28-490c-a137-9ca76f07a51b/ed3cf17e-89b7-4b35-8f01-664318c40924"
-					(reference "R20")
+					(reference "R62")
 					(unit 1)
 				)
@@
 		(dnp no)
 		(fields_autoplaced yes)
-		(property "Reference" "R23"
+		(property "Reference" "R67"
 			(at 137.16 88.9 90)
 			(show_name no)
@@
 			(project "ACW_First"
 				(path "/f90a1fa2-4579-4163-be1b-3b1c72ac9515/b1ee6347-5b28-490c-a137-9ca76f07a51b/ed3cf17e-89b7-4b35-8f01-664318c40924"
-					(reference "R23")
+					(reference "R67")
 					(unit 1)
 				)
@@
 		(in_pos_files yes)
 		(dnp no)
-		(property "Reference" "R25"
+		(property "Reference" "R66"
 			(at 237.49 120.6499 0)
 			(show_name no)
@@
 			(project "ACW_First"
 				(path "/f90a1fa2-4579-4163-be1b-3b1c72ac9515/b1ee6347-5b28-490c-a137-9ca76f07a51b/ed3cf17e-89b7-4b35-8f01-664318c40924"
-					(reference "R25")
+					(reference "R66")
 					(unit 1)
 				)
