File: ACW_First/PZEM.kicad_sch (KiCad schematic)
At the start: 44 parts, among them U5 HT7133-1_C15060, U6 V9881D, U7 CT817C, U8 CT817C

Commit message: okok
Connections:
- net at C34.1, C37.2, R31.2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: now also U6.2 (IAP); no longer U6.23 (VDD5)
- net at C26.2, C27.2, R27.2: now also U6.22 (VDCIN); no longer U6.3 (IAN)
- net at U7.2 (CATHODE): now also U6.9 (P0.2/WAKEUP3/TMS); no longer U6.16 (P2.5/TXD2)
- net at C40.1, R36.1: now also U6.6 (MODE1); no longer U6.19 (RSTn)
- net at C25.2, C27.1, R26.2: now also U6.23 (VDD5); no longer U6.2 (IAP)
- net at C35.1, C38.2: now also U6.12 (VSS); no longer U6.13 (DVCC)
- net at C36.1, C39.2, R36.2: now also U6.11 (P1.3/RXD5/INT0/CFx/SP/PLLDIV/WAKEUP2); no longer U6.14 (LDO33)
- net at C28.1, R28.1, R29.2: now also U6.24 (REF); no longer U6.1 (UP)
- net at R37.2, U8.4 (COLLECTOR): now also U6.8 (P0.1/TDI); no longer U6.17 (P2.4/RXD2)
- net at C30.1: now also U6.1 (UP); no longer U6.24 (REF)
- net at Y1.1: now also U6.5 (IBP); no longer U6.20 (CTI)
- net at Y1.2: now also U6.4 (IBN); no longer U6.21 (CTO)
- net at C33.2, R32.2, R33.1: now also U6.3 (IAN); no longer U6.22 (VDCIN)
- net at U8.3 (EMITTER): now also U6.7 (P0.0/TDO); no longer U6.18 (P2.0/T2/OSC)
- net at R34.1: now also U6.19 (RSTn); no longer U6.6 (MODE1)
- net CT renamed CT2
- net CT2: now also U6.13 (DVCC); no longer R25.2, R26.1, U6.12 (VSS)
- new net: U6.20 (CTI), U6.21 (CTO)
- new net CT1: R25.2, R26.1
Other:
- moved on the sheet: C29, R25
Changed lines of the file:
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@@
 		)
 	)
-	(hierarchical_label "CT"
+	(hierarchical_label "CT1"
 		(shape input)
 		(at 20.32 59.69 180)
@@
 		)
 	)
-	(hierarchical_label "CT"
+	(hierarchical_label "CT2"
 		(shape input)
 		(at 20.32 63.5 180)
@@
 	(symbol
 		(lib_id "Device:C")
-		(at 31.75 74.93 180)
+		(at 31.75 74.93 0)
+		(mirror x)
 		(unit 1)
 		(body_style 1)
@@
 		(dnp no)
 		(property "Reference" "C29"
-			(at 29.21 74.168 0)
+			(at 34.29 74.168 0)
 			(show_name no)
 			(do_not_autoplace no)
@@
 		)
 		(property "Value" "0.47µF/275VAC"
-			(at 29.21 75.692 0)
+			(at 34.29 75.692 0)
 			(show_name no)
 			(do_not_autoplace no)
@@
 		)
 		(property "Footprint" "Capacitor_THT:C_Rect_L18.0mm_W11.0mm_P15.00mm_FKS3_FKP3"
-			(at 30.7848 71.12 0)
+			(at 32.7152 71.12 0)
 			(hide yes)
 			(show_name no)
@@
 		(lib_id "Device:R")
 		(at 31.75 86.36 0)
+		(mirror y)
 		(unit 1)
 		(body_style 1)
@@
 		(dnp no)
 		(property "Reference" "R35"
-			(at 29.972 86.36 90)
+			(at 33.528 86.36 90)
 			(show_name no)
 			(do_not_autoplace no)
@@
 		)
 		(property "Value" "100Ω/2W"
-			(at 33.528 86.36 90)
+			(at 29.972 86.36 90)
 			(show_name no)
 			(do_not_autoplace no)
@@
 		)
 		(property "Footprint" "Resistor_THT:R_Axial_DIN0516_L15.5mm_D5.0mm_P25.40mm_Horizontal"
-			(at 29.972 86.36 90)
+			(at 33.528 86.36 90)
 			(hide yes)
 			(show_name no)
@@
 	(symbol
 		(lib_id "Device:R")
-		(at 36.83 45.72 180)
+		(at 36.83 45.72 0)
+		(mirror x)
 		(unit 1)
 		(body_style 1)
@@
 		(dnp no)
 		(property "Reference" "R25"
-			(at 35.052 45.72 90)
+			(at 38.608 45.72 90)
 			(show_name no)
 			(do_not_autoplace no)
@@
 		)
 		(property "Value" "0.001Ω/2W"
-			(at 38.862 45.72 90)
+			(at 34.798 45.72 90)
 			(show_name no)
 			(do_not_autoplace no)
@@
 		)
 		(property "Footprint" "Resistor_SMD:R_2512_6332Metric"
-			(at 38.608 45.72 90)
+			(at 35.052 45.72 90)
 			(hide yes)
 			(show_name no)
@@
 		(lib_id "V9881D:V9881D")
 		(at 154.94 71.12 0)
+		(mirror y)
 		(unit 1)
 		(body_style 1)
@@
 		(in_pos_files yes)
 		(dnp no)
-		(fields_autoplaced yes)
 		(property "Reference" "U6"
 			(at 154.94 49.53 0)

Commit message: okok
Parts:
- Y1: footprint Crystal:Crystal_C26-LF_D2.1mm_L6.5mm_Horizontal -> Crystal:Crystal_SMD_5032-4Pin_5.0x3.2mm
Changed lines of the file:
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@@
 			)
 		)
-		(property "Footprint" "Crystal:Crystal_C26-LF_D2.1mm_L6.5mm_Horizontal"
+		(property "Footprint" "Crystal:Crystal_SMD_5032-4Pin_5.0x3.2mm"
 			(at 204.47 67.31 0)
 			(hide yes)

Commit message: add firstlevel & secondlevevl pcb
Other:
- moved on the sheet: C39
Changed lines of the file:
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@@
 	(wire
 		(pts
+			(xy 151.13 111.76) (xy 151.13 119.38)
+		)
+		(stroke
+			(width 0)
+			(type default)
+		)
+	)
+	(wire
+		(pts
 			(xy 25.4 67.31) (xy 25.4 87.63)
 		)
@@
 	(wire
 		(pts
-			(xy 151.13 119.38) (xy 151.13 111.76)
-		)
-		(stroke
-			(width 0)
-			(type default)
-		)
-	)
-	(wire
-		(pts
 			(xy 97.79 63.5) (xy 97.79 85.09)
 		)
@@
 	(symbol
 		(lib_id "Device:C")
-		(at 171.45 107.95 180)
+		(at 171.45 107.95 0)
+		(mirror x)
 		(unit 1)
 		(body_style 1)
@@
 		(dnp no)
 		(property "Reference" "C39"
-			(at 169.164 107.188 0)
+			(at 173.736 107.188 0)
 			(show_name no)
 			(do_not_autoplace no)
@@
 		)
 		(property "Value" "100nF"
-			(at 169.164 108.712 0)
+			(at 173.736 108.712 0)
 			(show_name no)
 			(do_not_autoplace no)
@@
 		)
 		(property "Footprint" "Capacitor_SMD:C_0603_1608Metric"
-			(at 170.4848 104.14 0)
+			(at 172.4152 104.14 0)
 			(hide yes)
 			(show_name no)

Commit message: okokok
Changed lines of the file:
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@@
 	)
 	(hierarchical_label "N"
-		(shape input)
+		(shape output)
 		(at 21.59 67.31 180)
 		(effects
@@
 	)
 	(hierarchical_label "L"
-		(shape input)
+		(shape output)
 		(at 21.59 71.12 180)
 		(effects

Commit message: okok
Parts:
- removed R29: 750Ω, Resistor_SMD:R_0603_1608Metric, symbol Device:R
Connections:
- net at C34.1, C37.2, R31.2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: now also R38.2; no longer R38.1
- net at U7.1 (ANODE): now also R38.1; no longer R38.2
Other:
- moved on the sheet: D12, R38
Changed lines of the file:
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@@
 	)
 	(junction
-		(at 62.23 71.12)
-		(diameter 0)
-		(color 0 0 0 0)
-	)
-	(junction
 		(at 77.47 119.38)
 		(diameter 0)
@@
 	)
 	(junction
-		(at 69.85 71.12)
-		(diameter 0)
-		(color 0 0 0 0)
-	)
-	(junction
 		(at 121.92 119.38)
 		(diameter 0)
@@
 	(wire
 		(pts
-			(xy 69.85 71.12) (xy 69.85 77.47)
-		)
-		(stroke
-			(width 0)
-			(type default)
-		)
-	)
-	(wire
-		(pts
 			(xy 31.75 78.74) (xy 39.37 78.74)
 		)
@@
 	(wire
 		(pts
-			(xy 69.85 63.5) (xy 69.85 71.12)
+			(xy 69.85 63.5) (xy 69.85 77.47)
 		)
 		(stroke
@@
 	(symbol
 		(lib_id "Device:LED_Small")
-		(at 238.76 123.19 270)
+		(at 238.76 123.19 90)
+		(mirror x)
 		(unit 1)
 		(body_style 1)
@@
 		(dnp no)
 		(property "Reference" "D12"
-			(at 242.316 123.19 0)
+			(at 235.204 123.19 0)
 			(show_name no)
 			(do_not_autoplace no)
@@
 		)
 		(property "Value" "LED"
-			(at 241.3 123.19 0)
+			(at 236.22 123.19 0)
 			(show_name no)
 			(do_not_autoplace no)
@@
 	(symbol
 		(lib_id "Device:R")
-		(at 232.41 60.96 90)
+		(at 232.41 60.96 270)
+		(mirror x)
 		(unit 1)
 		(body_style 1)
@@
 					(unit 1)
 				)
-			)
-		)
-	)
-	(symbol
-		(lib_id "Device:R")
-		(at 66.04 71.12 270)
-		(unit 1)
-		(body_style 1)
-		(exclude_from_sim no)
-		(in_bom yes)
-		(on_board yes)
-		(in_pos_files yes)
-		(dnp no)
-		(property "Reference" "R29"
-			(at 66.04 69.342 90)
-			(show_name no)
-			(do_not_autoplace no)
-			(effects
-				(font
-					(size 0.889 0.889)
-				)
-			)
-		)
-		(property "Value" "750Ω"
-			(at 66.04 72.898 90)
-			(show_name no)
-			(do_not_autoplace no)
-			(effects
-				(font
-					(size 0.762 0.762)
-				)
-			)
-		)
-		(property "Footprint" "Resistor_SMD:R_0603_1608Metric"
-			(at 66.04 69.342 90)
-			(hide yes)
-			(show_name no)
-			(do_not_autoplace no)
-			(effects
-				(font
-					(size 1.27 1.27)
-				)
-			)
-		)
-		(property "Datasheet" ""
-			(at 66.04 71.12 0)
-			(hide yes)
-			(show_name no)
-			(do_not_autoplace no)
-			(effects
-				(font
-					(size 1.27 1.27)
-				)
-			)
-		)
-		(property "Description" "Resistor"
-			(at 66.04 71.12 0)
-			(hide yes)
-			(show_name no)
-			(do_not_autoplace no)
-			(effects
-				(font
-					(size 1.27 1.27)
-				)
-			)
-		)
-		(pin "1"
-		)
-		(pin "2"
-		)
-		(instances
-			(project "ACW_First"
-				(path "/f90a1fa2-4579-4163-be1b-3b1c72ac9515/12eda807-bac2-4cc9-8a54-0cbb858c2020"
-					(reference "R29")
-					(unit 1)
-				)

Commit message: fix
Parts:
- renumbered C29 to C41, C31 to C42, C25 to C43, C26 to C44, C32 to C45, C27 to C46, C28 to C47, C33 to C48, C37 to C49, C34 to C50, C35 to C51, C38 to C52, C36 to C53, C39 to C54, C30 to C55, C40 to C56, D10 to D11, D11 to D12, D12 to D13, D13 to D14, R35 to R53, R25 to R54, R30 to R55, R26 to R56, R27 to R57, R28 to R58, R32 to R59, R33 to R60, R31 to R61, R34 to R62, R36 to R63, R38 to R64, R37 to R65, R39 to R66, R40 to R67, R41 to R68, R42 to R69, U5 to U13, U6 to U14, U8 to U15, U7 to U16, Y1 to Y2

Commit message: okok
Parts:
- added R42: 100Ω, Resistor_SMD:R_0603_1608Metric, symbol Device:R
- renumbered C41 to C2, C45 to C3, C50 to C32, C49 to C33, C51 to C34, C52 to C35, C54 to C36, C53 to C37, C55 to C38, C56 to C39, C46 to C40, C47 to C41, C48 to C42, C42 to C43, C43 to C45, D13 to D1, D14 to D2, D12 to D4, R61 to R3, R69 to R32, R67 to R33, R68 to R34, R66 to R35, R63 to R37, R65 to R38, R64 to R39, R62 to R4, R58 to R43, R55 to R44, R60 to R45, R59 to R46, R57 to R47, R56 to R48, R54 to R49, R53 to R5, U14 to U10, U13 to U11, U15 to U7, U16 to U8
Connections:
- net CT2: now also R42.2
- net at C41.1, R43.1, U10.24 (REF): now also R42.1
Other:
- moved on the sheet: C41
