File: ACW_First/Power.kicad_sch (KiCad schematic)
At the start: 66 parts, among them U10 MP1584EN, U11 MP1584EN, U9 MP1584EN

Commit message: okokok
Parts:
- added J3: 3.8VDC, Connector_PinHeader_2.54mm:PinHeader_1x02_P2.54mm_Vertical, symbol Connector:Conn_01x02_Pin
- added J4: 5VDC, Connector_PinHeader_2.54mm:PinHeader_1x02_P2.54mm_Vertical, symbol Connector:Conn_01x02_Pin
- added J5: 12VDC, Connector_PinHeader_2.54mm:PinHeader_1x02_P2.54mm_Vertical, symbol Connector:Conn_01x02_Pin
Connections:
- net 3.8VDC: no longer C61.1, C62.1, C63.2, L6.2, R61.2, TP8.1
- net 5VDC: now also J4.2 (Pin_2)
- net GND: now also J3.1 (Pin_1), J4.1 (Pin_1), J5.1 (Pin_1)
- net 12VDC: no longer names the net of C47.1, L4.2, R49.2, TP6.1
- net 12VDC: now also J5.2 (Pin_2)
- new net: C61.1, C62.1, C63.2, J3.2 (Pin_2), L6.2, R61.2, TP8.1
Other:
- moved on the sheet: C55, TP6, TP7

Commit message: revisi
Changed lines of the file:
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@@
-		)
-	)
-	(label "-24VDC"
-		(at 243.84 104.14 0)
-		(effects
-			(font
-				(size 1.27 1.27)
-			)
-			(justify left bottom)
 		)
 	)
@@
 		)
 	)
-	(label "24VDC"
-		(at 243.84 109.22 0)
-		(effects
-			(font
-				(size 1.27 1.27)
-			)
-			(justify left bottom)
-		)
-	)
 	(label "COMP INPUT"
 		(at 228.6 69.85 180)
@@
 		)
 	)
+	(hierarchical_label "-24VDC"
+		(shape output)
+		(at 243.84 104.14 0)
+		(effects
+			(font
+				(size 1.27 1.27)
+			)
+			(justify left)
+		)
+	)
 	(hierarchical_label "5VDC"
-		(shape input)
+		(shape output)
 		(at 33.02 73.66 180)
 		(effects
@@
 	)
 	(hierarchical_label "24VDC"
-		(shape input)
+		(shape output)
 		(at 185.42 69.85 180)
 		(effects
@@
 	)
 	(hierarchical_label "24VDC"
-		(shape input)
+		(shape output)
 		(at 49.53 160.02 180)
 		(effects
@@
 		)
 	)
+	(hierarchical_label "24VDC"
+		(shape output)
+		(at 243.84 109.22 0)
+		(effects
+			(font
+				(size 1.27 1.27)
+			)
+			(justify left)
+		)
+	)

Commit message: okok
Parts:
- removed J3: 3.8VDC, Connector_PinHeader_2.54mm:PinHeader_1x02_P2.54mm_Vertical, symbol Connector:Conn_01x02_Pin
- removed J4: 5VDC, Connector_PinHeader_2.54mm:PinHeader_1x02_P2.54mm_Vertical, symbol Connector:Conn_01x02_Pin
- removed J5: 12VDC, Connector_PinHeader_2.54mm:PinHeader_1x02_P2.54mm_Vertical, symbol Connector:Conn_01x02_Pin
Connections:
- net 3.8VDC: now also C61.1, C62.1, C63.2, L6.2, R61.2, TP8.1
- net at C52.1: now also D18.1 (K), L5.1, U10.1 (SW); no longer U10.8 (BST)
- net 12VDC: now reaches C47.1, L4.2, R49.2, TP6.1
- removed net 1.65V: R44.2, R45.1, R50.2, R51.1, R56.2, R57.1, U10.2 (EN), U11.2 (EN), U9.2 (EN)
- removed net COMP INPUT: C44.1, C46.1, C51.1, C53.1, C58.1, C60.1, U10.3 (COMP), U11.3 (COMP), U9.3 (COMP)
- new net: C52.2, U10.8 (BST)
- new net 1.65V for 12VDC: R44.2, R45.1, U9.2 (EN)
- new net 1.65V for 3.8VDC: R56.2, R57.1, U11.2 (EN)
- new net 1.65V for 5VDC: R50.2, R51.1, U10.2 (EN)
- new net COMP INPUT for 12VDC: C44.1, C46.1, U9.3 (COMP)
- new net COMP INPUT for 3.8VDC: C58.1, C60.1, U11.3 (COMP)
- new net COMP INPUT for 5VDC: C51.1, C53.1, U10.3 (COMP)
Other:
- moved on the sheet: C52, C56, C57, C58, C59, C60, C61, C62, C63, D14, D19, D20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

Commit message: fix
Parts:
- renumbered C56 to C14, C48 to C15, C57 to C16, C49 to C17, C50 to C18, C58 to C19, C59 to C20, C60 to C21, C51 to C22, C52 to C23, C61 to C24, C53 to C25, C62 to C26, C63 to C27, C54 to C28, C55 to C29, C41 to C30, C42 to C31, C43 to C32, C44 to C33, C45 to C34, C46 to C35, C47 to C36, D14 to D10, D19 to D4, D17 to D5, D20 to D6, D18 to D7, D15 to D8, D16 to D9, F6 to F2, F5 to F3, L6 to L1, L5 to L2, L4 to L3, PS1 to PS2, R56 to R26, R57 to R27, R50 to R28, R58 to R29, R51 to R30, R52 to R31, R59 to R32, R60 to R33, R53 to R34, R61 to R35, R54 to R36, R55 to R37, R44 to R38, R45 to R39, R46 to R40, R47 to R41, R48 to R42, R49 to R43, R43 to R44, RV3 to RV2, TH2 to TH1, TP8 to TP1, TP7 to TP2, TP6 to TP3, TP1 to TP4, TP2 to TP5, U11 to U7, U10 to U8

Commit message: okok
Parts:
- L3: renamed from L2; footprint Inductor_SMD:L_Bourns-SRR1005 -> Inductor_SMD:L_7.3x7.3_H4.5
- renumbered C24 to C10, C31 to C12, C34 to C13, C17 to C14, C23 to C15, C18 to C16, C20 to C17, C32 to C18, C25 to C21, C35 to C22, C22 to C23, C19 to C24, C16 to C25, C33 to C26, C28 to C27, C14 to C28, C36 to C29, C21 to C30, C29 to C31, C27 to C4, C26 to C5, C15 to C8, C30 to C9, D4 to D10, D6 to D12, D9 to D13, D7 to D14, D10 to D3, D5 to D8, D8 to D9, F4 to F1, F2 to F4, L3 to L2, PS2 to PS1, R39 to R11, R38 to R12, R31 to R17, R40 to R18, R44 to R2, R41 to R21, R34 to R22, R37 to R23, R42 to R24, R43 to R25, R36 to R26, R32 to R27, R28 to R6, R35 to R60, R33 to R61, R29 to R63, R26 to R69, R27 to R70, R30 to R8, RV2 to RV1, TP4 to TP1, TP5 to TP2, TP1 to TP3, TP3 to TP4, TP2 to TP5, U8 to U2, U9 to U3, U7 to U4
Other:
- moved on the sheet: D3, F1, PS1, R2, RV1, TH1, TP1, TP2
