File: ACW_First/RTC_Circuit.kicad_sch (KiCad schematic)
At the start: 11 parts, among them U105 DS3231M, U106 AT24C512-SSHM

Commit message: fix
Parts:
- renumbered BT101 to BT1, C112 to C38, C113 to C39, C114 to C40, R119 to R48, R120 to R49, R121 to R50, R122 to R51, R123 to R52, U105 to U11, U106 to U12
Changed lines of the file:
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@@
 		(dnp no)
 		(fields_autoplaced yes)
-		(property "Reference" "#PWR0134"
+		(property "Reference" "#PWR072"
 			(at 110.49 144.78 0)
 			(hide yes)
@@
 			(project "ACW_First"
 				(path "/f90a1fa2-4579-4163-be1b-3b1c72ac9515/b1ee6347-5b28-490c-a137-9ca76f07a51b/310cfdba-f14c-429b-bae2-5d48e453e8a4"
-					(reference "#PWR0134")
+					(reference "#PWR072")
 					(unit 1)
 				)
@@
 		(dnp no)
 		(fields_autoplaced yes)
-		(property "Reference" "U106"
+		(property "Reference" "U12"
 			(at 126.4794 46.99 0)
 			(show_name no)
@@
 			(project "ACW_First"
 				(path "/f90a1fa2-4579-4163-be1b-3b1c72ac9515/b1ee6347-5b28-490c-a137-9ca76f07a51b/310cfdba-f14c-429b-bae2-5d48e453e8a4"
-					(reference "U106")
+					(reference "U12")
 					(unit 1)
 				)
@@
 		(dnp no)
 		(fields_autoplaced yes)
-		(property "Reference" "U105"
+		(property "Reference" "U11"
 			(at 125.2094 130.81 0)
 			(show_name no)
@@
 			(project "ACW_First"
 				(path "/f90a1fa2-4579-4163-be1b-3b1c72ac9515/b1ee6347-5b28-490c-a137-9ca76f07a51b/310cfdba-f14c-429b-bae2-5d48e453e8a4"
-					(reference "U105")
+					(reference "U11")
 					(unit 1)
 				)
@@
 		(dnp no)
 		(fields_autoplaced yes)
-		(property "Reference" "R121"
+		(property "Reference" "R50"
 			(at 97.79 64.7699 0)
 			(show_name no)
@@
 			(project "ACW_First"
 				(path "/f90a1fa2-4579-4163-be1b-3b1c72ac9515/b1ee6347-5b28-490c-a137-9ca76f07a51b/310cfdba-f14c-429b-bae2-5d48e453e8a4"
-					(reference "R121")
+					(reference "R50")
 					(unit 1)
 				)
@@
 		(in_pos_files yes)
 		(dnp no)
-		(property "Reference" "C113"
+		(property "Reference" "C39"
 			(at 142.24 41.91 0)
 			(show_name no)
@@
 			(project "ACW_First"
 				(path "/f90a1fa2-4579-4163-be1b-3b1c72ac9515/b1ee6347-5b28-490c-a137-9ca76f07a51b/310cfdba-f14c-429b-bae2-5d48e453e8a4"
-					(reference "C113")
+					(reference "C39")
 					(unit 1)
 				)
@@
 		(in_pos_files yes)
 		(dnp no)
-		(property "Reference" "C112"
+		(property "Reference" "C38"
 			(at 78.74 109.22 0)
 			(show_name no)
@@
 			(project "ACW_First"
 				(path "/f90a1fa2-4579-4163-be1b-3b1c72ac9515/b1ee6347-5b28-490c-a137-9ca76f07a51b/310cfdba-f14c-429b-bae2-5d48e453e8a4"
-					(reference "C112")
+					(reference "C38")
 					(unit 1)
 				)
@@
 		(dnp no)
 		(fields_autoplaced yes)
-		(property "Reference" "R123"
+		(property "Reference" "R52"
 			(at 163.83 40.6399 0)
 			(show_name no)
@@
 			(project "ACW_First"
 				(path "/f90a1fa2-4579-4163-be1b-3b1c72ac9515/b1ee6347-5b28-490c-a137-9ca76f07a51b/310cfdba-f14c-429b-bae2-5d48e453e8a4"
-					(reference "R123")
+					(reference "R52")
 					(unit 1)
 				)
@@
 		(in_pos_files yes)
 		(dnp no)
-		(property "Reference" "R122"
+		(property "Reference" "R51"
 			(at 155.448 45.974 0)
 			(show_name no)
@@
 			(project "ACW_First"
 				(path "/f90a1fa2-4579-4163-be1b-3b1c72ac9515/b1ee6347-5b28-490c-a137-9ca76f07a51b/310cfdba-f14c-429b-bae2-5d48e453e8a4"
-					(reference "R122")
+					(reference "R51")
 					(unit 1)
 				)
@@
 		(in_pos_files yes)
 		(dnp no)
-		(property "Reference" "R119"
+		(property "Reference" "R48"
 			(at 76.2 64.77 0)
 			(show_name no)
@@
 			(project "ACW_First"
 				(path "/f90a1fa2-4579-4163-be1b-3b1c72ac9515/b1ee6347-5b28-490c-a137-9ca76f07a51b/310cfdba-f14c-429b-bae2-5d48e453e8a4"
-					(reference "R119")
+					(reference "R48")
 					(unit 1)
 				)
@@
 		(dnp no)
 		(fields_autoplaced yes)
-		(property "Reference" "#PWR0133"
+		(property "Reference" "#PWR071"
 			(at 87.63 81.28 0)
 			(hide yes)
@@
 			(project "ACW_First"
 				(path "/f90a1fa2-4579-4163-be1b-3b1c72ac9515/b1ee6347-5b28-490c-a137-9ca76f07a51b/310cfdba-f14c-429b-bae2-5d48e453e8a4"
-					(reference "#PWR0133")
+					(reference "#PWR071")
 					(unit 1)
 				)
@@
 		(dnp no)
 		(fields_autoplaced yes)
-		(property "Reference" "#PWR0137"
+		(property "Reference" "#PWR073"
 			(at 124.46 76.2 0)
 			(hide yes)
@@
 			(project "ACW_First"
 				(path "/f90a1fa2-4579-4163-be1b-3b1c72ac9515/b1ee6347-5b28-490c-a137-9ca76f07a51b/310cfdba-f14c-429b-bae2-5d48e453e8a4"
-					(reference "#PWR0137")
+					(reference "#PWR073")
 					(unit 1)
 				)
@@
 		(dnp no)
 		(fields_autoplaced yes)
-		(property "Reference" "BT101"
+		(property "Reference" "BT1"
 			(at 191.1985 92.71 90)
 			(show_name no)
@@
 			(project "ACW_First"
 				(path "/f90a1fa2-4579-4163-be1b-3b1c72ac9515/b1ee6347-5b28-490c-a137-9ca76f07a51b/310cfdba-f14c-429b-bae2-5d48e453e8a4"
-					(reference "BT101")
+					(reference "BT1")
 					(unit 1)
 				)
@@
 		(dnp no)
 		(fields_autoplaced yes)
-		(property "Reference" "#PWR0139"
+		(property "Reference" "#PWR075"
 			(at 208.28 72.39 0)
 			(hide yes)
@@
 			(project "ACW_First"
 				(path "/f90a1fa2-4579-4163-be1b-3b1c72ac9515/b1ee6347-5b28-490c-a137-9ca76f07a51b/310cfdba-f14c-429b-bae2-5d48e453e8a4"
-					(reference "#PWR0139")
+					(reference "#PWR075")
 					(unit 1)
 				)
@@
 		(dnp no)
 		(fields_autoplaced yes)
-		(property "Reference" "#PWR0138"
+		(property "Reference" "#PWR074"
 			(at 172.72 93.98 0)
 			(hide yes)
@@
 			(project "ACW_First"
 				(path "/f90a1fa2-4579-4163-be1b-3b1c72ac9515/b1ee6347-5b28-490c-a137-9ca76f07a51b/310cfdba-f14c-429b-bae2-5d48e453e8a4"
-					(reference "#PWR0138")
+					(reference "#PWR074")
 					(unit 1)
 				)
@@
 		(dnp no)
 		(fields_autoplaced yes)
-		(property "Reference" "R120"
+		(property "Reference" "R49"
 			(at 90.17 64.7699 0)
 			(show_name no)
@@
 			(project "ACW_First"
 				(path "/f90a1fa2-4579-4163-be1b-3b1c72ac9515/b1ee6347-5b28-490c-a137-9ca76f07a51b/310cfdba-f14c-429b-bae2-5d48e453e8a4"
-					(reference "R120")
+					(reference "R49")
 					(unit 1)
 				)
@@
 		(in_pos_files yes)
 		(dnp no)
-		(property "Reference" "C114"
+		(property "Reference" "C40"
 			(at 153.67 120.65 0)
 			(show_name no)
@@
 			(project "ACW_First"
 				(path "/f90a1fa2-4579-4163-be1b-3b1c72ac9515/b1ee6347-5b28-490c-a137-9ca76f07a51b/310cfdba-f14c-429b-bae2-5d48e453e8a4"
-					(reference "C114")
-					(unit 1)
-				)
+					(reference "C40")
+					(unit 1)
+				)

Commit message: okok
Parts:
- renumbered C40 to C46, C39 to C47, C38 to C48, R50 to R51, R51 to R53, R48 to R55, R52 to R56, R49 to R57, U11 to U12, U12 to U13
Changed lines of the file:
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@@
+		(dnp no)
+		(fields_autoplaced yes)
+		(property "Reference" "U13"
+			(at 126.4794 46.99 0)
+			(show_name no)
+			(do_not_autoplace no)
+			(effects
+				(font
+					(size 1.27 1.27)
+				)
+				(justify left)
+			)
+		)
+		(property "Value" "AT24C512-SSHM"
+			(at 126.4794 49.53 0)
+			(show_name no)
+			(do_not_autoplace no)
+			(effects
+				(font
+					(size 1.27 1.27)
+				)
+				(justify left)
+			)
+		)
+		(property "Footprint" "Custom_Library:SOIC127P600X175-8N"
+			(at 124.46 57.15 0)
+			(hide yes)
+			(show_name no)
+			(do_not_autoplace no)
+			(effects
+				(font
+					(size 1.27 1.27)
+				)
+			)
+		)
+		(property "Datasheet" "http://ww1.microchip.com/downloads/en/DeviceDoc/Atmel-8869-SEEPROM-AT24CS32-Datasheet.pdf"
+			(at 124.46 57.15 0)
+			(hide yes)
+			(show_name no)
+			(do_not_autoplace no)
+			(effects
+				(font
+					(size 1.27 1.27)
+				)
+			)
+		)
+		(property "Description" ""
+			(at 124.46 57.15 0)
+			(show_name no)
+			(do_not_autoplace no)
+			(effects
+				(font
+					(size 1.27 1.27)
+				)
+			)
+		)
+		(pin "1"
+		)
+		(pin "2"
+		)
+		(pin "3"
+		)
+		(pin "4"
+		)
+		(pin "5"
+		)
+		(pin "6"
+		)
+		(pin "7"
+		)
+		(pin "8"
+		)
+		(instances
+			(project "ACW_First"
+				(path "/f90a1fa2-4579-4163-be1b-3b1c72ac9515/b1ee6347-5b28-490c-a137-9ca76f07a51b/310cfdba-f14c-429b-bae2-5d48e453e8a4"
+					(reference "U13")
+					(unit 1)
+				)
+			)
+		)
+	)
+	(symbol
+		(lib_id "Timer_RTC:DS3231M")
+		(at 123.19 120.65 0)
+		(unit 1)
+		(body_style 1)
+		(exclude_from_sim no)
+		(in_bom yes)
+		(on_board yes)
+		(in_pos_files yes)
 		(dnp no)
 		(fields_autoplaced yes)
 		(property "Reference" "U12"
-			(at 126.4794 46.99 0)
-			(show_name no)
-			(do_not_autoplace no)
-			(effects
-				(font
-					(size 1.27 1.27)
-				)
-				(justify left)
-			)
-		)
-		(property "Value" "AT24C512-SSHM"
-			(at 126.4794 49.53 0)
-			(show_name no)
-			(do_not_autoplace no)
-			(effects
-				(font
-					(size 1.27 1.27)
-				)
-				(justify left)
-			)
-		)
-		(property "Footprint" "Custom_Library:SOIC127P600X175-8N"
-			(at 124.46 57.15 0)
-			(hide yes)
-			(show_name no)
-			(do_not_autoplace no)
-			(effects
-				(font
-					(size 1.27 1.27)
-				)
-			)
-		)
-		(property "Datasheet" "http://ww1.microchip.com/downloads/en/DeviceDoc/Atmel-8869-SEEPROM-AT24CS32-Datasheet.pdf"
-			(at 124.46 57.15 0)
-			(hide yes)
-			(show_name no)
-			(do_not_autoplace no)
-			(effects
-				(font
-					(size 1.27 1.27)
-				)
-			)
-		)
-		(property "Description" ""
-			(at 124.46 57.15 0)
-			(show_name no)
-			(do_not_autoplace no)
-			(effects
-				(font
-					(size 1.27 1.27)
-				)
-			)
-		)
-		(pin "1"
-		)
-		(pin "2"
-		)
-		(pin "3"
-		)
-		(pin "4"
-		)
-		(pin "5"
-		)
-		(pin "6"
-		)
-		(pin "7"
-		)
-		(pin "8"
-		)
-		(instances
-			(project "ACW_First"
-				(path "/f90a1fa2-4579-4163-be1b-3b1c72ac9515/b1ee6347-5b28-490c-a137-9ca76f07a51b/310cfdba-f14c-429b-bae2-5d48e453e8a4"
-					(reference "U12")
-					(unit 1)
-				)
-			)
-		)
-	)
-	(symbol
-		(lib_id "Timer_RTC:DS3231M")
-		(at 123.19 120.65 0)
-		(unit 1)
-		(body_style 1)
-		(exclude_from_sim no)
-		(in_bom yes)
-		(on_board yes)
-		(in_pos_files yes)
-		(dnp no)
-		(fields_autoplaced yes)
-		(property "Reference" "U11"
 			(at 125.2094 130.81 0)
 			(show_name no)
@@
 			(project "ACW_First"
 				(path "/f90a1fa2-4579-4163-be1b-3b1c72ac9515/b1ee6347-5b28-490c-a137-9ca76f07a51b/310cfdba-f14c-429b-bae2-5d48e453e8a4"
-					(reference "U11")
+					(reference "U12")
 					(unit 1)
 				)
@@
 		(dnp no)
 		(fields_autoplaced yes)
-		(property "Reference" "R50"
+		(property "Reference" "R51"
 			(at 97.79 64.7699 0)
 			(show_name no)
@@
 			(project "ACW_First"
 				(path "/f90a1fa2-4579-4163-be1b-3b1c72ac9515/b1ee6347-5b28-490c-a137-9ca76f07a51b/310cfdba-f14c-429b-bae2-5d48e453e8a4"
-					(reference "R50")
+					(reference "R51")
 					(unit 1)
 				)
@@
 		(in_pos_files yes)
 		(dnp no)
-		(property "Reference" "C39"
+		(property "Reference" "C47"
 			(at 142.24 41.91 0)
 			(show_name no)
@@
 			(project "ACW_First"
 				(path "/f90a1fa2-4579-4163-be1b-3b1c72ac9515/b1ee6347-5b28-490c-a137-9ca76f07a51b/310cfdba-f14c-429b-bae2-5d48e453e8a4"
-					(reference "C39")
+					(reference "C47")
 					(unit 1)
 				)
@@
 		(in_pos_files yes)
 		(dnp no)
-		(property "Reference" "C38"
+		(property "Reference" "C48"
 			(at 78.74 109.22 0)
 			(show_name no)
@@
 			(project "ACW_First"
 				(path "/f90a1fa2-4579-4163-be1b-3b1c72ac9515/b1ee6347-5b28-490c-a137-9ca76f07a51b/310cfdba-f14c-429b-bae2-5d48e453e8a4"
-					(reference "C38")
+					(reference "C48")
 					(unit 1)
 				)
@@
 		(dnp no)
 		(fields_autoplaced yes)
-		(property "Reference" "R52"
+		(property "Reference" "R56"
 			(at 163.83 40.6399 0)
 			(show_name no)
@@
 			(project "ACW_First"
 				(path "/f90a1fa2-4579-4163-be1b-3b1c72ac9515/b1ee6347-5b28-490c-a137-9ca76f07a51b/310cfdba-f14c-429b-bae2-5d48e453e8a4"
-					(reference "R52")
+					(reference "R56")
 					(unit 1)
 				)
@@
 		(in_pos_files yes)
 		(dnp no)
-		(property "Reference" "R51"
+		(property "Reference" "R53"
 			(at 155.448 45.974 0)
 			(show_name no)
@@
 			(project "ACW_First"
 				(path "/f90a1fa2-4579-4163-be1b-3b1c72ac9515/b1ee6347-5b28-490c-a137-9ca76f07a51b/310cfdba-f14c-429b-bae2-5d48e453e8a4"
-					(reference "R51")
+					(reference "R53")
 					(unit 1)
 				)
@@
 		(in_pos_files yes)
 		(dnp no)
-		(property "Reference" "R48"
+		(property "Reference" "R55"
 			(at 76.2 64.77 0)
 			(show_name no)
@@
 			(project "ACW_First"
 				(path "/f90a1fa2-4579-4163-be1b-3b1c72ac9515/b1ee6347-5b28-490c-a137-9ca76f07a51b/310cfdba-f14c-429b-bae2-5d48e453e8a4"
-					(reference "R48")
+					(reference "R55")
 					(unit 1)
 				)
@@
 		(dnp no)
 		(fields_autoplaced yes)
-		(property "Reference" "R49"
+		(property "Reference" "R57"
 			(at 90.17 64.7699 0)
 			(show_name no)
@@
 			(project "ACW_First"
 				(path "/f90a1fa2-4579-4163-be1b-3b1c72ac9515/b1ee6347-5b28-490c-a137-9ca76f07a51b/310cfdba-f14c-429b-bae2-5d48e453e8a4"
-					(reference "R49")
+					(reference "R57")
 					(unit 1)
 				)
@@
 		(in_pos_files yes)
 		(dnp no)
-		(property "Reference" "C40"
+		(property "Reference" "C46"
 			(at 153.67 120.65 0)
 			(show_name no)
@@
 			(project "ACW_First"
 				(path "/f90a1fa2-4579-4163-be1b-3b1c72ac9515/b1ee6347-5b28-490c-a137-9ca76f07a51b/310cfdba-f14c-429b-bae2-5d48e453e8a4"
-					(reference "C40")
-					(unit 1)
-				)
+					(reference "C46")
+					(unit 1)
+				)
