File: ACW_First/Relay.kicad_sch (KiCad schematic)
At the start: 13 parts, among them K1 SRD-05VDC-SL-C, Q1 S8050, U4 PC817

Commit message: okok
Parts:
- Q1: footprint Package_TO_SOT_THT:TO-92_Inline -> Package_TO_SOT_SMD:SOT-23
- U4: footprint Package_DIP:DIP-4_W7.62mm -> Custom_Library:SOP254P975X460-4N
Connections:
- net GND: now also U4.3; no longer U4.2
- net at R20.2: now also U4.4; no longer U4.1
- net at R21.1: now also U4.2; no longer U4.3
- net at C24.1, F3.2, RV2.1: no longer K1.NO
- net 5 VDC renamed 5V
- net 5V: now also U4.1; no longer U4.4
- net LI renamed COM
- net LO renamed NO
- net N: no longer names the net of R24.1, RV2.2
- net N: now also K1.NO
Other:
- moved on the sheet: R24, RV2
Changed lines of the file:
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@@
-	)
-	(junction
-		(at 176.53 71.12)
-		(diameter 0)
-		(color 0 0 0 0)
 	)
 	(junction
@@
 	)
 	(junction
+		(at 177.8 66.04)
+		(diameter 0)
+		(color 0 0 0 0)
+	)
+	(junction
 		(at 143.51 64.77)
 		(diameter 0)
@@
 	)
 	(junction
-		(at 176.53 66.04)
-		(diameter 0)
-		(color 0 0 0 0)
-	)
-	(junction
-		(at 176.53 83.82)
+		(at 177.8 81.28)
 		(diameter 0)
 		(color 0 0 0 0)
@@
 	(wire
 		(pts
-			(xy 176.53 66.04) (xy 176.53 71.12)
-		)
-		(stroke
-			(width 0)
-			(type default)
-		)
-	)
-	(wire
-		(pts
-			(xy 187.96 81.28) (xy 190.5 81.28)
+			(xy 189.23 81.28) (xy 191.77 81.28)
 		)
 		(stroke
@@
 	(wire
 		(pts
+			(xy 177.8 66.04) (xy 180.34 66.04)
+		)
+		(stroke
+			(width 0)
+			(type default)
+		)
+	)
+	(wire
+		(pts
 			(xy 143.51 85.09) (xy 149.86 85.09)
 		)
@@
 	(wire
 		(pts
-			(xy 180.34 66.04) (xy 176.53 66.04)
-		)
-		(stroke
-			(width 0)
-			(type default)
-		)
-	)
-	(wire
-		(pts
-			(xy 176.53 72.39) (xy 176.53 71.12)
+			(xy 170.18 66.04) (xy 177.8 66.04)
+		)
+		(stroke
+			(width 0)
+			(type default)
+		)
+	)
+	(wire
+		(pts
+			(xy 177.8 66.04) (xy 177.8 69.85)
 		)
 		(stroke
@@
 	(wire
 		(pts
-			(xy 176.53 83.82) (xy 176.53 82.55)
-		)
-		(stroke
-			(width 0)
-			(type default)
-		)
-	)
-	(wire
-		(pts
 			(xy 123.19 92.71) (xy 123.19 95.25)
 		)
@@
 	(wire
 		(pts
-			(xy 143.51 62.23) (xy 143.51 64.77)
+			(xy 143.51 59.69) (xy 143.51 64.77)
+		)
+		(stroke
+			(width 0)
+			(type default)
+		)
+	)
+	(wire
+		(pts
+			(xy 177.8 81.28) (xy 177.8 80.01)
+		)
+		(stroke
+			(width 0)
+			(type default)
+		)
+	)
+	(wire
+		(pts
+			(xy 181.61 81.28) (xy 177.8 81.28)
 		)
 		(stroke
@@
 	(wire
 		(pts
-			(xy 176.53 83.82) (xy 180.34 83.82)
-		)
-		(stroke
-			(width 0)
-			(type default)
-		)
-	)
-	(wire
-		(pts
 			(xy 132.08 64.77) (xy 132.08 71.12)
 		)
@@
 		)
 	)
-	(wire
-		(pts
-			(xy 165.1 71.12) (xy 176.53 71.12)
-		)
-		(stroke
-			(width 0)
-			(type default)
-		)
-	)
 	(polyline
 		(pts
@@
 	(wire
 		(pts
-			(xy 187.96 66.04) (xy 190.5 66.04)
+			(xy 173.99 81.28) (xy 177.8 81.28)
+		)
+		(stroke
+			(width 0)
+			(type default)
+		)
+	)
+	(wire
+		(pts
+			(xy 187.96 66.04) (xy 191.77 66.04)
 		)
 		(stroke
@@
 	(wire
 		(pts
-			(xy 176.53 66.04) (xy 170.18 66.04)
-		)
-		(stroke
-			(width 0)
-			(type default)
-		)
-	)
-	(wire
-		(pts
 			(xy 128.27 64.77) (xy 132.08 64.77)
 		)
@@
 	(wire
 		(pts
-			(xy 180.34 83.82) (xy 180.34 81.28)
-		)
-		(stroke
-			(width 0)
-			(type default)
-		)
-	)
-	(wire
-		(pts
 			(xy 88.9 92.71) (xy 107.95 92.71)
 		)
@@
 	(wire
 		(pts
-			(xy 190.5 81.28) (xy 190.5 66.04)
+			(xy 191.77 81.28) (xy 191.77 66.04)
 		)
 		(stroke
@@
 	(wire
 		(pts
+			(xy 165.1 71.12) (xy 173.99 71.12)
+		)
+		(stroke
+			(width 0)
+			(type default)
+		)
+	)
+	(wire
+		(pts
 			(xy 143.51 81.28) (xy 143.51 85.09)
 		)
@@
 	(wire
 		(pts
-			(xy 176.53 86.36) (xy 176.53 83.82)
+			(xy 173.99 71.12) (xy 173.99 81.28)
 		)
 		(stroke
@@
 		)
 	)
-	(global_label "5 VDC"
-		(shape input)
-		(at 143.51 62.23 90)
-		(fields_autoplaced yes)
-		(effects
-			(font
-				(size 1.27 1.27)
-			)
-			(justify left)
-		)
-		(property "Intersheetrefs" "${INTERSHEET_REFS}"
-			(at 143.51 53.4391 90)
-			(hide yes)
-			(show_name no)
-			(do_not_autoplace no)
-			(effects
-				(font
-					(size 1.27 1.27)
-				)
-				(justify left)
-			)
-		)
-	)
-	(hierarchical_label "N"
-		(shape input)
-		(at 176.53 86.36 270)
-		(effects
-			(font
-				(size 1.27 1.27)
-			)
-			(justify right)
-		)
-	)
-	(hierarchical_label "LO"
+	(hierarchical_label "NO"
 		(shape output)
 		(at 170.18 55.88 90)
@@
 		)
 	)
-	(hierarchical_label "LI"
+	(hierarchical_label "COM"
 		(shape input)
 		(at 167.64 73.66 0)
@@
 			)
 			(justify right)
+		)
+	)
+	(hierarchical_label "5V"
+		(shape input)
+		(at 143.51 59.69 90)
+		(effects
+			(font
+				(size 1.27 1.27)
+			)
+			(justify left)
 		)
 	)
@@
 		(lib_id "Isolator:PC817")
 		(at 115.57 90.17 0)
+		(mirror y)
 		(unit 1)
 		(body_style 1)
@@
 		(in_pos_files yes)
 		(dnp no)
-		(fields_autoplaced yes)
 		(property "Reference" "U4"
 			(at 115.57 81.28 0)
@@
 			)
 		)
-		(property "Footprint" "Package_DIP:DIP-4_W7.62mm"
-			(at 110.49 95.25 0)
+		(property "Footprint" "Custom_Library:SOP254P975X460-4N"
+			(at 120.65 95.25 0)
 			(hide yes)
 			(show_name no)
@@
 	(symbol
 		(lib_id "10D471K:10D471K-C8760")
-		(at 176.53 77.47 270)
+		(at 177.8 74.93 270)
 		(unit 1)
 		(body_style 1)
@@
 		(dnp no)
 		(property "Reference" "RV2"
-			(at 177.8 77.724 90)
+			(at 179.07 75.184 90)
 			(show_name no)
 			(do_not_autoplace no)
@@
 		)
 		(property "Value" "10D471K"
-			(at 170.18 78.994 90)
+			(at 171.45 76.454 90)
 			(show_name no)
 			(do_not_autoplace no)
@@
 		)
 		(property "Footprint" "Custom_Footprints:RES-TH_L12.5-W6.7-P7.50-D1.2"
-			(at 168.91 77.47 0)
+			(at 170.18 74.93 0)
 			(hide yes)
 			(show_name no)
@@
 		)
 		(property "Datasheet" "https://lcsc.com/product-detail/Varistors_10D471K_C8760.html"
-			(at 166.37 77.47 0)
+			(at 167.64 74.93 0)
 			(hide yes)
 			(show_name no)
@@
 		)
 		(property "Description" "10D471K"
-			(at 176.53 77.47 0)
+			(at 177.8 74.93 0)
 			(hide yes)
 			(show_name no)
@@
 		)
 		(property "Manufacturer" "RUILON(瑞隆源)"
-			(at 163.83 77.47 0)
+			(at 165.1 74.93 0)
 			(hide yes)
 			(show_name no)
@@
 		)
 		(property "MPN" "10D471K"
-			(at 161.29 77.47 0)
+			(at 162.56 74.93 0)
 			(hide yes)
 			(show_name no)
@@
 		)
 		(property "LCSC Part" "C8760"
-			(at 158.75 77.47 0)
+			(at 160.02 74.93 0)
 			(hide yes)
 			(show_name no)
@@
 			)
 		)
-		(property "Footprint" "Package_TO_SOT_THT:TO-92_Inline"
+		(property "Footprint" "Package_TO_SOT_SMD:SOT-23"
 			(at 148.59 97.155 0)
 			(hide yes)
@@
 	(symbol
 		(lib_id "Device:R")
-		(at 184.15 81.28 90)
+		(at 185.42 81.28 90)
 		(unit 1)
 		(body_style 1)
@@
 		(dnp no)
 		(property "Reference" "R24"
-			(at 184.15 78.232 90)
+			(at 185.42 78.232 90)
 			(show_name no)
 			(do_not_autoplace no)
@@
 		)
 		(property "Value" "120Ω 2W"
-			(at 184.15 79.502 90)
+			(at 185.42 79.502 90)
 			(show_name no)
 			(do_not_autoplace no)
@@
 		)
 		(property "Footprint" "Resistor_THT:R_Axial_DIN0414_L11.9mm_D4.5mm_P15.24mm_Horizontal"
-			(at 184.15 83.058 90)
+			(at 185.42 83.058 90)
 			(hide yes)
 			(show_name no)
@@
 		)
 		(property "Datasheet" ""
-			(at 184.15 81.28 0)
+			(at 185.42 81.28 0)
 			(hide yes)
 			(show_name no)
@@
 		)
 		(property "Description" "Resistor"
-			(at 184.15 81.28 0)
-			(hide yes)
-			(show_name no)
+			(at 185.42 81.28 0)
+			(hide yes)
+			(show_name no)

Commit message: okok
Parts:
- F3: footprint Fuse:Fuseholder_Clip-5x20mm_Littelfuse_100_Inline_P20.50x4.60mm_D1.30mm_Horizontal -> Fuse:Fuseholder_Cylinder-5x20mm_Schurter_0031_8201_Horizontal_Open
Changed lines of the file:
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@@
 			)
 		)
-		(property "Footprint" "Fuse:Fuseholder_Clip-5x20mm_Littelfuse_100_Inline_P20.50x4.60mm_D1.30mm_Horizontal"
+		(property "Footprint" "Fuse:Fuseholder_Cylinder-5x20mm_Schurter_0031_8201_Horizontal_Open"
 			(at 168.402 60.96 90)
 			(hide yes)

Commit message: okok
Connections:
- net at C24.1, F3.2, RV2.1: now also K1.NO
- net at R24.1, RV2.2: no longer K1.NO
Other:
- moved on the sheet: F3
Changed lines of the file:
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@@
+	)
+	(junction
+		(at 172.72 66.04)
+		(diameter 0)
+		(color 0 0 0 0)
 	)
 	(junction
@@
 	)
 	(junction
-		(at 177.8 66.04)
-		(diameter 0)
-		(color 0 0 0 0)
-	)
-	(junction
 		(at 143.51 64.77)
 		(diameter 0)
@@
 	)
 	(junction
-		(at 177.8 81.28)
-		(diameter 0)
-		(color 0 0 0 0)
-	)
-	(junction
 		(at 143.51 85.09)
 		(diameter 0)
 		(color 0 0 0 0)
 	)
+	(junction
+		(at 177.8 66.04)
+		(diameter 0)
+		(color 0 0 0 0)
+	)
 	(no_connect
 		(at 165.1 78.74)
@@
 	(wire
 		(pts
-			(xy 170.18 66.04) (xy 177.8 66.04)
-		)
-		(stroke
-			(width 0)
-			(type default)
-		)
-	)
-	(wire
-		(pts
 			(xy 177.8 66.04) (xy 177.8 69.85)
 		)
@@
 	(wire
 		(pts
+			(xy 172.72 71.12) (xy 172.72 66.04)
+		)
+		(stroke
+			(width 0)
+			(type default)
+		)
+	)
+	(wire
+		(pts
 			(xy 143.51 59.69) (xy 143.51 64.77)
 		)
@@
 		)
 	)
+	(wire
+		(pts
+			(xy 172.72 66.04) (xy 177.8 66.04)
+		)
+		(stroke
+			(width 0)
+			(type default)
+		)
+	)
 	(polyline
 		(pts
@@
 	(wire
 		(pts
-			(xy 173.99 81.28) (xy 177.8 81.28)
-		)
-		(stroke
-			(width 0)
-			(type default)
-		)
-	)
-	(wire
-		(pts
 			(xy 187.96 66.04) (xy 191.77 66.04)
 		)
@@
 	(wire
 		(pts
-			(xy 170.18 64.77) (xy 170.18 66.04)
-		)
-		(stroke
-			(width 0)
-			(type default)
-		)
-	)
-	(wire
-		(pts
 			(xy 128.27 64.77) (xy 132.08 64.77)
 		)
@@
 	(wire
 		(pts
+			(xy 172.72 64.77) (xy 172.72 66.04)
+		)
+		(stroke
+			(width 0)
+			(type default)
+		)
+	)
+	(wire
+		(pts
 			(xy 88.9 92.71) (xy 107.95 92.71)
 		)
@@
 	(wire
 		(pts
-			(xy 170.18 55.88) (xy 170.18 57.15)
+			(xy 172.72 55.88) (xy 172.72 57.15)
 		)
 		(stroke
@@
 	(wire
 		(pts
-			(xy 165.1 71.12) (xy 173.99 71.12)
+			(xy 165.1 71.12) (xy 172.72 71.12)
 		)
 		(stroke
@@
 		(pts
 			(xy 132.08 78.74) (xy 132.08 85.09)
-		)
-		(stroke
-			(width 0)
-			(type default)
-		)
-	)
-	(wire
-		(pts
-			(xy 173.99 71.12) (xy 173.99 81.28)
 		)
 		(stroke
@@
 	(hierarchical_label "NO"
 		(shape output)
-		(at 170.18 55.88 90)
+		(at 172.72 55.88 90)
 		(effects
 			(font
@@
 	(symbol
 		(lib_id "Device:Fuse")
-		(at 170.18 60.96 0)
+		(at 172.72 60.96 0)
 		(unit 1)
 		(body_style 1)
@@
 		(dnp no)
 		(property "Reference" "F3"
-			(at 166.624 59.69 0)
+			(at 169.164 59.69 0)
 			(show_name no)
 			(do_not_autoplace no)
@@
 		)
 		(property "Value" "Fuse"
-			(at 164.846 61.214 0)
+			(at 167.386 61.214 0)
 			(show_name no)
 			(do_not_autoplace no)
@@
 		)
 		(property "Footprint" "Fuse:Fuseholder_Cylinder-5x20mm_Schurter_0031_8201_Horizontal_Open"
-			(at 168.402 60.96 90)
+			(at 170.942 60.96 90)
 			(hide yes)
 			(show_name no)
@@
 		)
 		(property "Datasheet" ""
-			(at 170.18 60.96 0)
+			(at 172.72 60.96 0)
 			(hide yes)
 			(show_name no)
@@
 		)
 		(property "Description" "Fuse"
-			(at 170.18 60.96 0)
-			(hide yes)
-			(show_name no)
+			(at 172.72 60.96 0)
+			(hide yes)
+			(show_name no)

Commit message: okokok
Connections:
- net 5V: now also U4.3; no longer U4.1
- net GND: now also U4.1; no longer U4.3
- net at U4.2: now also R20.2; no longer R21.1
- net at U4.4: now also R21.1; no longer R20.2
- net NeutralInput: now reaches R24.1, RV2.2
Changed lines of the file:
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@@
+	)
+	(junction
+		(at 177.8 81.28)
+		(diameter 0)
+		(color 0 0 0 0)
 	)
 	(junction
@@
 	(wire
 		(pts
+			(xy 173.99 81.28) (xy 177.8 81.28)
+		)
+		(stroke
+			(width 0)
+			(type default)
+		)
+	)
+	(wire
+		(pts
 			(xy 189.23 81.28) (xy 191.77 81.28)
 		)
@@
 		(pts
 			(xy 132.08 64.77) (xy 143.51 64.77)
+		)
+		(stroke
+			(width 0)
+			(type default)
+		)
+	)
+	(wire
+		(pts
+			(xy 173.99 87.63) (xy 173.99 81.28)
 		)
 		(stroke
@@
 			)
 			(justify left)
+		)
+	)
+	(hierarchical_label "NeutralInput"
+		(shape input)
+		(at 173.99 87.63 270)
+		(effects
+			(font
+				(size 1.27 1.27)
+			)
+			(justify right)
 		)
 	)
@@
 		(lib_id "Isolator:PC817")
 		(at 115.57 90.17 0)
-		(mirror y)
+		(mirror x)
 		(unit 1)
 		(body_style 1)
@@
 		(dnp no)
 		(property "Reference" "U4"
-			(at 115.57 81.28 0)
+			(at 115.57 99.06 0)
 			(show_name no)
 			(do_not_autoplace no)
@@
 		)
 		(property "Value" "PC817"
-			(at 115.57 83.82 0)
+			(at 115.57 96.52 0)
 			(show_name no)
 			(do_not_autoplace no)
@@
 		)
 		(property "Footprint" "Custom_Library:SOP254P975X460-4N"
-			(at 120.65 95.25 0)
+			(at 110.49 85.09 0)
 			(hide yes)
 			(show_name no)

Commit message: revisi
Parts:
- removed U4: PC817, Custom_Library:SOP254P975X460-4N, symbol Isolator:PC817
- added U1: PC817, Custom_Library:SOP254P975X460-4N, symbol Isolator:PC817
Connections:
- net 5V: now also U1.4
- net GND: now also U1.2
- net at R20.2: now also U1.1
- net at R21.1: now also U1.3
Changed lines of the file:
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@@
-	)
-	(symbol
-		(lib_id "Isolator:PC817")
-		(at 115.57 90.17 0)
-		(mirror x)
-		(unit 1)
-		(body_style 1)
-		(exclude_from_sim no)
-		(in_bom yes)
-		(on_board yes)
-		(in_pos_files yes)
-		(dnp no)
-		(property "Reference" "U4"
-			(at 115.57 99.06 0)
-			(show_name no)
-			(do_not_autoplace no)
-			(effects
-				(font
-					(size 1.27 1.27)
-				)
-			)
-		)
-		(property "Value" "PC817"
-			(at 115.57 96.52 0)
-			(show_name no)
-			(do_not_autoplace no)
-			(effects
-				(font
-					(size 1.27 1.27)
-				)
-			)
-		)
-		(property "Footprint" "Custom_Library:SOP254P975X460-4N"
-			(at 110.49 85.09 0)
-			(hide yes)
-			(show_name no)
-			(do_not_autoplace no)
-			(effects
-				(font
-					(size 1.27 1.27)
-					(italic yes)
-				)
-				(justify left)
-			)
-		)
-		(property "Datasheet" "http://www.soselectronic.cz/a_info/resource/d/pc817.pdf"
-			(at 115.57 90.17 0)
-			(hide yes)
-			(show_name no)
-			(do_not_autoplace no)
-			(effects
-				(font
-					(size 1.27 1.27)
-				)
-				(justify left)
-			)
-		)
-		(property "Description" "DC Optocoupler, Vce 35V, CTR 50-300%, DIP-4"
-			(at 115.57 90.17 0)
-			(hide yes)
-			(show_name no)
-			(do_not_autoplace no)
-			(effects
-				(font
-					(size 1.27 1.27)
-				)
-			)
-		)
-		(pin "1"
-		)
-		(pin "4"
-		)
-		(pin "3"
-		)
-		(pin "2"
-		)
-		(instances
-			(project "ACW_First"
-				(path "/f90a1fa2-4579-4163-be1b-3b1c72ac9515/1cc8220c-d861-4212-897b-561f3cc307ea"
-					(reference "U4")
-					(unit 1)
-				)
-			)
-		)
 	)
 	(symbol
@@
 					(unit 1)
 				)
+			)
+		)
+	)
+	(symbol
+		(lib_id "Isolator:PC817")
+		(at 115.57 90.17 0)
+		(unit 1)
+		(body_style 1)
+		(exclude_from_sim no)
+		(in_bom yes)
+		(on_board yes)
+		(in_pos_files yes)
+		(dnp no)
+		(fields_autoplaced yes)
+		(property "Reference" "U1"
+			(at 115.57 81.28 0)
+			(show_name no)
+			(do_not_autoplace no)
+			(effects
+				(font
+					(size 1.27 1.27)
+				)
+			)
+		)
+		(property "Value" "PC817"
+			(at 115.57 83.82 0)
+			(show_name no)
+			(do_not_autoplace no)
+			(effects
+				(font
+					(size 1.27 1.27)
+				)
+			)
+		)
+		(property "Footprint" "Custom_Library:SOP254P975X460-4N"
+			(at 110.49 95.25 0)
+			(hide yes)
+			(show_name no)
+			(do_not_autoplace no)
+			(effects
+				(font
+					(size 1.27 1.27)
+					(italic yes)
+				)
+				(justify left)
+			)
+		)
+		(property "Datasheet" "http://www.soselectronic.cz/a_info/resource/d/pc817.pdf"
+			(at 115.57 90.17 0)
+			(hide yes)
+			(show_name no)
+			(do_not_autoplace no)
+			(effects
+				(font
+					(size 1.27 1.27)
+				)
+				(justify left)
+			)
+		)
+		(property "Description" "DC Optocoupler, Vce 35V, CTR 50-300%, DIP-4"
+			(at 115.57 90.17 0)
+			(hide yes)
+			(show_name no)
+			(do_not_autoplace no)
+			(effects
+				(font
+					(size 1.27 1.27)
+				)
+			)
+		)
+		(pin "4"
+		)
+		(pin "3"
+		)
+		(pin "2"
+		)
+		(pin "1"
+		)
+		(instances
+			(project "ACW_First"
+				(path "/f90a1fa2-4579-4163-be1b-3b1c72ac9515/1cc8220c-d861-4212-897b-561f3cc307ea"
+					(reference "U1")
+					(unit 1)
+				)

Commit message: okok
Parts:
- removed D6: LED_Red, LED_SMD:LED_0805_2012Metric, symbol Device:LED_Small
- removed R23: 1KΩ, Resistor_SMD:R_0603_1608Metric, symbol Device:R
- U1: footprint Custom_Library:SOP254P975X460-4N -> Custom_Footprints:SOP-4_L6.4-W4.6-P2.54-LS10.2-TL
Other:
- note removed: "1.2V - 1.8V"
- moved on the sheet: D9

Commit message: fix
Parts:
- renumbered C24 to C1, D9 to D1, F3 to F1, R20 to R1, R21 to R2, R22 to R3, R24 to R4, RV2 to RV1
Changed lines of the file:
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@@
 		(in_pos_files yes)
 		(dnp no)
-		(property "Reference" "F3"
+		(property "Reference" "F1"
 			(at 169.164 59.69 0)
 			(show_name no)
@@
 			(project "ACW_First"
 				(path "/f90a1fa2-4579-4163-be1b-3b1c72ac9515/1cc8220c-d861-4212-897b-561f3cc307ea"
-					(reference "F3")
+					(reference "F1")
 					(unit 1)
 				)
@@
 		(in_pos_files yes)
 		(dnp no)
-		(property "Reference" "RV2"
+		(property "Reference" "RV1"
 			(at 179.07 75.184 90)
 			(show_name no)
@@
 			(project "ACW_First"
 				(path "/f90a1fa2-4579-4163-be1b-3b1c72ac9515/1cc8220c-d861-4212-897b-561f3cc307ea"
-					(reference "RV2")
+					(reference "RV1")
 					(unit 1)
 				)
@@
 		(in_pos_files yes)
 		(dnp no)
-		(property "Reference" "#PWR037"
+		(property "Reference" "#PWR08"
 			(at 146.05 118.11 0)
 			(hide yes)
@@
 			(project "ACW_First"
 				(path "/f90a1fa2-4579-4163-be1b-3b1c72ac9515/1cc8220c-d861-4212-897b-561f3cc307ea"
-					(reference "#PWR037")
+					(reference "#PWR08")
 					(unit 1)
 				)
@@
 		(in_pos_files yes)
 		(dnp no)
-		(property "Reference" "R22"
+		(property "Reference" "R3"
 			(at 132.842 107.95 90)
 			(show_name no)
@@
 			(project "ACW_First"
 				(path "/f90a1fa2-4579-4163-be1b-3b1c72ac9515/1cc8220c-d861-4212-897b-561f3cc307ea"
-					(reference "R22")
+					(reference "R3")
 					(unit 1)
 				)
@@
 		(in_pos_files yes)
 		(dnp no)
-		(property "Reference" "D9"
+		(property "Reference" "D1"
 			(at 145.034 74.168 90)
 			(show_name no)
@@
 			(project "ACW_First"
 				(path "/f90a1fa2-4579-4163-be1b-3b1c72ac9515/1cc8220c-d861-4212-897b-561f3cc307ea"
-					(reference "D9")
+					(reference "D1")
 					(unit 1)
 				)
@@
 		(in_pos_files yes)
 		(dnp no)
-		(property "Reference" "C24"
+		(property "Reference" "C1"
 			(at 184.15 61.722 90)
 			(show_name no)
@@
 			(project "ACW_First"
 				(path "/f90a1fa2-4579-4163-be1b-3b1c72ac9515/1cc8220c-d861-4212-897b-561f3cc307ea"
-					(reference "C24")
+					(reference "C1")
 					(unit 1)
 				)
@@
 		(in_pos_files yes)
 		(dnp no)
-		(property "Reference" "R21"
+		(property "Reference" "R2"
 			(at 129.54 92.202 90)
 			(show_name no)
@@
 			(project "ACW_First"
 				(path "/f90a1fa2-4579-4163-be1b-3b1c72ac9515/1cc8220c-d861-4212-897b-561f3cc307ea"
-					(reference "R21")
+					(reference "R2")
 					(unit 1)
 				)
@@
 		(in_pos_files yes)
 		(dnp no)
-		(property "Reference" "#PWR036"
+		(property "Reference" "#PWR07"
 			(at 88.9 101.6 0)
 			(hide yes)
@@
 			(project "ACW_First"
 				(path "/f90a1fa2-4579-4163-be1b-3b1c72ac9515/1cc8220c-d861-4212-897b-561f3cc307ea"
-					(reference "#PWR036")
+					(reference "#PWR07")
 					(unit 1)
 				)
@@
 		(in_pos_files yes)
 		(dnp no)
-		(property "Reference" "R20"
+		(property "Reference" "R1"
 			(at 99.06 84.582 90)
 			(show_name no)
@@
 			(project "ACW_First"
 				(path "/f90a1fa2-4579-4163-be1b-3b1c72ac9515/1cc8220c-d861-4212-897b-561f3cc307ea"
-					(reference "R20")
+					(reference "R1")
 					(unit 1)
 				)
@@
 		(in_pos_files yes)
 		(dnp no)
-		(property "Reference" "R24"
+		(property "Reference" "R4"
 			(at 185.42 78.232 90)
 			(show_name no)
@@
 			(project "ACW_First"
 				(path "/f90a1fa2-4579-4163-be1b-3b1c72ac9515/1cc8220c-d861-4212-897b-561f3cc307ea"
-					(reference "R24")
-					(unit 1)
-				)
+					(reference "R4")
+					(unit 1)
+				)

Commit message: okok
Parts:
- renumbered D1 to D5, F1 to F2, R4 to R1, R1 to R36, R2 to R40, R3 to R41, RV1 to RV2, U1 to U9
Changed lines of the file:
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@@
 		(in_pos_files yes)
 		(dnp no)
-		(property "Reference" "F1"
+		(property "Reference" "F2"
 			(at 169.164 59.69 0)
 			(show_name no)
@@
 			(project "ACW_First"
 				(path "/f90a1fa2-4579-4163-be1b-3b1c72ac9515/1cc8220c-d861-4212-897b-561f3cc307ea"
-					(reference "F1")
+					(reference "F2")
 					(unit 1)
 				)
@@
 		(in_pos_files yes)
 		(dnp no)
-		(property "Reference" "RV1"
+		(property "Reference" "RV2"
 			(at 179.07 75.184 90)
 			(show_name no)
@@
 			(project "ACW_First"
 				(path "/f90a1fa2-4579-4163-be1b-3b1c72ac9515/1cc8220c-d861-4212-897b-561f3cc307ea"
-					(reference "RV1")
+					(reference "RV2")
 					(unit 1)
 				)
@@
 		(in_pos_files yes)
 		(dnp no)
-		(property "Reference" "R3"
+		(property "Reference" "R41"
 			(at 132.842 107.95 90)
 			(show_name no)
@@
 			(project "ACW_First"
 				(path "/f90a1fa2-4579-4163-be1b-3b1c72ac9515/1cc8220c-d861-4212-897b-561f3cc307ea"
-					(reference "R3")
+					(reference "R41")
 					(unit 1)
 				)
@@
 		(in_pos_files yes)
 		(dnp no)
-		(property "Reference" "D1"
+		(property "Reference" "D5"
 			(at 145.034 74.168 90)
 			(show_name no)
@@
 			(project "ACW_First"
 				(path "/f90a1fa2-4579-4163-be1b-3b1c72ac9515/1cc8220c-d861-4212-897b-561f3cc307ea"
-					(reference "D1")
+					(reference "D5")
 					(unit 1)
 				)
@@
 		(in_pos_files yes)
 		(dnp no)
-		(property "Reference" "R2"
+		(property "Reference" "R40"
 			(at 129.54 92.202 90)
 			(show_name no)
@@
 			(project "ACW_First"
 				(path "/f90a1fa2-4579-4163-be1b-3b1c72ac9515/1cc8220c-d861-4212-897b-561f3cc307ea"
-					(reference "R2")
+					(reference "R40")
 					(unit 1)
 				)
@@
 		(dnp no)
 		(fields_autoplaced yes)
-		(property "Reference" "U1"
+		(property "Reference" "U9"
 			(at 115.57 81.28 0)
 			(show_name no)
@@
 			(project "ACW_First"
 				(path "/f90a1fa2-4579-4163-be1b-3b1c72ac9515/1cc8220c-d861-4212-897b-561f3cc307ea"
-					(reference "U1")
+					(reference "U9")
 					(unit 1)
 				)
@@
 		(in_pos_files yes)
 		(dnp no)
-		(property "Reference" "R1"
+		(property "Reference" "R36"
 			(at 99.06 84.582 90)
 			(show_name no)
@@
 			(project "ACW_First"
 				(path "/f90a1fa2-4579-4163-be1b-3b1c72ac9515/1cc8220c-d861-4212-897b-561f3cc307ea"
-					(reference "R1")
+					(reference "R36")
 					(unit 1)
 				)
@@
 		(in_pos_files yes)
 		(dnp no)
-		(property "Reference" "R4"
+		(property "Reference" "R1"
 			(at 185.42 78.232 90)
 			(show_name no)
@@
 			(project "ACW_First"
 				(path "/f90a1fa2-4579-4163-be1b-3b1c72ac9515/1cc8220c-d861-4212-897b-561f3cc307ea"
-					(reference "R4")
-					(unit 1)
-				)
+					(reference "R1")
+					(unit 1)
+				)
